File: Hardware/biruta.kicad_sch (KiCad schematic)
At the start: 1 part, among them J32 R-RJ11R06P-A800

Commit message: Sensores metereologicos -IA que fez
Parts:
- added C50: 10n, Capacitor_SMD:C_0603_1608Metric, symbol Device:C
- added D50: PESD5V0S1UL, Diode_SMD:D_SOD-882, symbol Device:D_Zener
- added D51: BAS70-04, Package_TO_SOT_SMD:SOT-23, symbol Sensores_Meteo:BAS70-04
- added R50, R51: 10k, Resistor_SMD:R_0603_1608Metric, symbol Device:R
- added R52: 1k, Resistor_SMD:R_0603_1608Metric, symbol Device:R
- added TP50: WIND_DIR_RAW, TestPoint:TestPoint_Pad_D1.5mm, symbol Connector:TestPoint
- added TP51: WIND_DIR_ADC, TestPoint:TestPoint_Pad_D1.5mm, symbol Connector:TestPoint
- added TP52: VREF_SENSOR, TestPoint:TestPoint_Pad_D1.5mm, symbol Connector:TestPoint
- added TP53: GND, TestPoint:TestPoint_Pad_D1.5mm, symbol Connector:TestPoint
- J32: Function (none) -> RJ11 individual; contatos centrais; LCSC (none) -> C189750; Manufacturer (none) -> Ckmtw; Rating (none) -> 6P6C; p3=return; p4=signal; THT
Connections:
- net GND: now also C50.2, D50.2 (A), D51.1 (A), TP53.1
- net WIND_DIR_ADC: now also C50.1, R52.2, TP51.1; no longer J32.4
- new net: D51.3 (COM), R51.2, R52.1
- new net +3V3: D51.2 (K)
- new net VREF_SENSOR: R50.1, TP52.1
- new net WIND_DIR_RAW: D50.1 (K), J32.4, R50.2, R51.1, TP50.1
Other:
- note added: "1 CONECTOR / DIVISOR"
- note added: "2 LIMITACAO / CLAMP"
- note added: "3 FILTRO / ADC"
- note added: "MISOL WH-SP-WD: rede resistiva passiva; 8 chaves / ate 16 codigos; cabo ~2 m."
- note added: "R50=10k 1%; ADC ideal=4095*R_sensor/(10000+R_sensor). R51/R52 estao APOS o divisor: nao entram na relacao DC ideal. Rfonte maxima ~20,23k; tau maxima ~202 us; validar tempo ADC (144 ciclos)."
- note added: "VREF_SENSOR vem de U5 CN10_7 (AVDD). Nao unir ao 3V3 digital por etiqueta. C50 junto ao PA0; retorno GND curto. Medir offsets por fuga e temperatura. A LUT ativa do firmware tem 16 entradas; 8 e o numero de amostras por leitura."
- note removed: "J32: Ckmtw R-RJ11R06P-A800 / LCSC C189750. Assumido: sensor usa os contatos centrais 3 e 4; confirmar no cabo real. A proteção e o condicionamento serão inseridos entre J32 e WIND_DIR_ADC."
- company: (none) -> TCC - Estacao meteorologica
- title: (none) -> BIRUTA - divisor ratiometrico e protecao ADC
- moved on the sheet: J32
