File: Hardware/mcu.kicad_sch (KiCad schematic)
At the start: 0 parts

Commit message: hardware: inicia PCB V2
Parts:
- added U5: NUCLEO-F446RE, myLibrary:MODULE_NUCLEO-F446RE, symbol Nucleo_F446:NUCLEO-F446RE
Connections:
- new net +5V: U5.CN7_18 (CN7_+5V)
- new net CN10_GND: U5.CN10_20 (CN10_GND), U5.CN10_9 (CN10_GND), U5.CN7_19 (CN7_GND), U5.CN7_20 (CN7_GND), U5.CN7_22 (CN7_GND), U5.CN7_8 (CN7_GND)
- new net PA0: U5.CN7_28 (PA0)
- new net PA1: U5.CN7_30 (PA1)
- new net PA11: U5.CN10_14 (PA11)
- new net PA12: U5.CN10_12 (PA12)
- new net PA5: U5.CN10_11 (PA5)
- new net PA6: U5.CN10_13 (PA6)
- new net PA7: U5.CN10_15 (PA7)
- new net PA8: U5.CN10_23 (PA8)
- new net PB12: U5.CN10_16 (PB12)
- new net PB13: U5.CN10_30 (PB13)
- new net PB14: U5.CN10_28 (PB14)
- new net PB15: U5.CN10_26 (PB15)
- new net PB6: U5.CN10_17 (PB6)
- new net PB7: U5.CN7_21 (PB7)
- new net PC4: U5.CN10_34 (PC4)
- new net PC5: U5.CN10_6 (PC5)
- new net PC7: U5.CN10_19 (PC7)
- no-connect marks 0 -> 44

Commit message: Sensores metereologicos -IA que fez
Parts:
- U5: symbol Nucleo_F446:NUCLEO-F446RE -> Hardware_MCU:NUCLEO-F446RE_Morpho
Connections:
- net CN10_GND is gone; now on net GND: U5.CN10_20 (CN10_GND), U5.CN10_9 (CN10_GND), U5.CN7_19 (CN7_GND), U5.CN7_20 (CN7_GND), U5.CN7_22 (CN7_GND), U5.CN7_8 (CN7_GND)
- net GND: now reaches U5.CN10_32 (AGND)
- net VREF_SENSOR: now reaches U5.CN10_7 (AVDD)
- net PA0 renamed WIND_DIR_ADC
- net PA1 renamed RAIN_PULSE
- net PC7 renamed WIND_SPEED_PULSE
- no-connect marks 44 -> 42
Other:
- note added: "METEO: PA1=chuva; PC7=velocidade; PA0=ADC. VREF_SENSOR: AVDD/VREF+ da Nucleo. Futura MCU discreta: ligar a mesma fonte da referencia ADC."
Changed lines of the file:
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@@
-	)
-	(no_connect
-		(at 186.69 50.8)
 	)
 	(no_connect
@@
 	)
 	(no_connect
-		(at 186.69 121.92)
-	)
-	(no_connect
 		(at 88.9 119.38)
 	)
@@
 		)
 	)
-	(global_label "PA1"
-		(shape input)
-		(at 85.09 76.2 180)
+	(hierarchical_label "RAIN_PULSE" (shape input) (at 85.09 76.2 0) (effects (font (size 1.0 1.0)) (justify right)))
+	(global_label "PA6"
+		(shape input)
+		(at 148.59 66.04 180)
 		(fields_autoplaced yes)
 		(effects
@@
 		)
 		(property "Intersheetrefs" "${INTERSHEET_REFS}"
-			(at 78.5367 76.2 0)
+			(at 142.0367 66.04 0)
 			(effects
 				(font
@@
 		)
 	)
-	(global_label "PA6"
-		(shape input)
-		(at 148.59 66.04 180)
+	(global_label "PB15"
+		(shape input)
+		(at 148.59 116.84 180)
 		(fields_autoplaced yes)
 		(effects
@@
 		)
 		(property "Intersheetrefs" "${INTERSHEET_REFS}"
-			(at 142.0367 66.04 0)
+			(at 140.6458 116.84 0)
 			(effects
 				(font
@@
 		)
 	)
-	(global_label "PB15"
-		(shape input)
-		(at 148.59 116.84 180)
+	(global_label "PB14"
+		(shape input)
+		(at 148.59 114.3 180)
 		(fields_autoplaced yes)
 		(effects
@@
 		)
 		(property "Intersheetrefs" "${INTERSHEET_REFS}"
-			(at 140.6458 116.84 0)
+			(at 140.6458 114.3 0)
 			(effects
 				(font
@@
 		)
 	)
-	(global_label "PB14"
-		(shape input)
-		(at 148.59 114.3 180)
+	(global_label "PB12"
+		(shape input)
+		(at 148.59 109.22 180)
 		(fields_autoplaced yes)
 		(effects
@@
 		)
 		(property "Intersheetrefs" "${INTERSHEET_REFS}"
-			(at 140.6458 114.3 0)
+			(at 140.6458 109.22 0)
 			(effects
 				(font
@@
 		)
 	)
-	(global_label "PB12"
-		(shape input)
-		(at 148.59 109.22 180)
+	(global_label "PA7"
+		(shape input)
+		(at 148.59 68.58 180)
 		(fields_autoplaced yes)
 		(effects
@@
 		)
 		(property "Intersheetrefs" "${INTERSHEET_REFS}"
-			(at 140.6458 109.22 0)
+			(at 142.0367 68.58 0)
 			(effects
 				(font
@@
 		)
 	)
-	(global_label "PA7"
-		(shape input)
-		(at 148.59 68.58 180)
+	(global_label "PC5"
+		(shape input)
+		(at 189.23 60.96 0)
+		(fields_autoplaced yes)
+		(effects
+			(font
+				(size 1.27 1.27)
+			)
+			(justify left)
+		)
+		(property "Intersheetrefs" "${INTERSHEET_REFS}"
+			(at 195.9647 60.96 0)
+			(effects
+				(font
+					(size 1.27 1.27)
+				)
+				(justify left)
+				(hide yes)
+			)
+		)
+	)
+	(global_label "PA8"
+		(shape input)
+		(at 148.59 71.12 180)
 		(fields_autoplaced yes)
 		(effects
@@
 		)
 		(property "Intersheetrefs" "${INTERSHEET_REFS}"
-			(at 142.0367 68.58 0)
+			(at 142.0367 71.12 0)
 			(effects
 				(font
@@
 		)
 	)
-	(global_label "PC5"
-		(shape input)
-		(at 189.23 60.96 0)
+	(global_label "PA11"
+		(shape input)
+		(at 148.59 78.74 180)
+		(fields_autoplaced yes)
+		(effects
+			(font
+				(size 1.27 1.27)
+			)
+			(justify right)
+		)
+		(property "Intersheetrefs" "${INTERSHEET_REFS}"
+			(at 140.8272 78.74 0)
+			(effects
+				(font
+					(size 1.27 1.27)
+				)
+				(justify right)
+				(hide yes)
+			)
+		)
+	)
+	(global_label "GND"
+		(shape input)
+		(at 137.16 127 0)
 		(fields_autoplaced yes)
 		(effects
@@
 		)
 		(property "Intersheetrefs" "${INTERSHEET_REFS}"
-			(at 195.9647 60.96 0)
+			(at 143.7132 127 0)
 			(effects
 				(font
@@
 		)
 	)
-	(global_label "PA8"
-		(shape input)
-		(at 148.59 71.12 180)
+	(hierarchical_label "WIND_SPEED_PULSE" (shape input) (at 189.23 66.04 180) (effects (font (size 1.0 1.0)) (justify left)))
+	(hierarchical_label "WIND_DIR_ADC" (shape input) (at 85.09 73.66 0) (effects (font (size 1.0 1.0)) (justify right)))
+	(global_label "PB13"
+		(shape input)
+		(at 148.59 111.76 180)
 		(fields_autoplaced yes)
 		(effects
@@
 		)
 		(property "Intersheetrefs" "${INTERSHEET_REFS}"
-			(at 142.0367 71.12 0)
+			(at 140.6458 111.76 0)
 			(effects
 				(font
@@
 		)
 	)
-	(global_label "PA11"
-		(shape input)
-		(at 148.59 78.74 180)
+	(global_label "PB7"
+		(shape input)
+		(at 85.09 93.98 180)
 		(fields_autoplaced yes)
 		(effects
@@
 		)
 		(property "Intersheetrefs" "${INTERSHEET_REFS}"
-			(at 140.8272 78.74 0)
+			(at 78.3553 93.98 0)
 			(effects
 				(font
@@
 		)
 	)
-	(global_label "Gnd"
-		(shape input)
-		(at 137.16 127 0)
+	(global_label "+5V"
+		(shape input)
+		(at 137.16 50.8 0)
 		(fields_autoplaced yes)
 		(effects
@@
 		)
 		(property "Intersheetrefs" "${INTERSHEET_REFS}"
-			(at 143.7132 127 0)
+			(at 144.0157 50.8 0)
 			(effects
 				(font
@@
 		)
 	)
-	(global_label "PC7"
-		(shape input)
-		(at 189.23 66.04 0)
+	(global_label "PA5"
+		(shape input)
+		(at 148.59 63.5 180)
+		(fields_autoplaced yes)
+		(effects
+			(font
+				(size 1.27 1.27)
+			)
+			(justify right)
+		)
+		(property "Intersheetrefs" "${INTERSHEET_REFS}"
+			(at 142.0367 63.5 0)
+			(effects
+				(font
+					(size 1.27 1.27)
+				)
+				(justify right)
+				(hide yes)
+			)
+		)
+	)
+	(global_label "GND"
+		(shape input)
+		(at 186.69 124.46 0)
 		(fields_autoplaced yes)
 		(effects
@@
 		)
 		(property "Intersheetrefs" "${INTERSHEET_REFS}"
-			(at 195.9647 66.04 0)
+			(at 193.2432 124.46 0)
 			(effects
 				(font
@@
 		)
 	)
-	(global_label "PA0"
-		(shape input)
-		(at 85.09 73.66 180)
+	(global_label "PA12"
+		(shape input)
+		(at 148.59 81.28 180)
 		(fields_autoplaced yes)
 		(effects
@@
 		)
 		(property "Intersheetrefs" "${INTERSHEET_REFS}"
-			(at 78.5367 73.66 0)
+			(at 140.8272 81.28 0)
 			(effects
 				(font
@@
 		)
 	)
-	(global_label "PB13"
-		(shape input)
-		(at 148.59 111.76 180)
-		(fields_autoplaced yes)
-		(effects
-			(font
-				(size 1.27 1.27)
-			)
-			(justify right)
-		)
-		(property "Intersheetrefs" "${INTERSHEET_REFS}"
-			(at 140.6458 111.76 0)
-			(effects
-				(font
-					(size 1.27 1.27)
-				)
-				(justify right)
-				(hide yes)
-			)
-		)
-	)
-	(global_label "PB7"
-		(shape input)
-		(at 85.09 93.98 180)
-		(fields_autoplaced yes)
-		(effects
-			(font
-				(size 1.27 1.27)
-			)
-			(justify right)
-		)
-		(property "Intersheetrefs" "${INTERSHEET_REFS}"
-			(at 78.3553 93.98 0)
-			(effects
-				(font
-					(size 1.27 1.27)
-				)
-				(justify right)
-				(hide yes)
-			)
-		)
-	)
-	(global_label "+5V"
-		(shape input)
-		(at 137.16 50.8 0)
-		(fields_autoplaced yes)
-		(effects
-			(font
-				(size 1.27 1.27)
-			)
-			(justify left)
-		)
-		(property "Intersheetrefs" "${INTERSHEET_REFS}"
-			(at 144.0157 50.8 0)
-			(effects
-				(font
-					(size 1.27 1.27)
-				)
-				(justify left)
-				(hide yes)
-			)
-		)
-	)
-	(global_label "PA5"
-		(shape input)
-		(at 148.59 63.5 180)
-		(fields_autoplaced yes)
-		(effects
-			(font
-				(size 1.27 1.27)
-			)
-			(justify right)
-		)
-		(property "Intersheetrefs" "${INTERSHEET_REFS}"
-			(at 142.0367 63.5 0)
-			(effects
-				(font
-					(size 1.27 1.27)
-				)
-				(justify right)
-				(hide yes)
-			)
-		)
-	)
-	(global_label "Gnd"
-		(shape input)
-		(at 186.69 124.46 0)
-		(fields_autoplaced yes)
-		(effects
-			(font
-				(size 1.27 1.27)
-			)
-			(justify left)
-		)
-		(property "Intersheetrefs" "${INTERSHEET_REFS}"
-			(at 193.2432 124.46 0)
-			(effects
-				(font
-					(size 1.27 1.27)
-				)
-				(justify left)
-				(hide yes)
-			)
-		)
-	)
-	(global_label "PA12"
-		(shape input)
-		(at 148.59 81.28 180)
-		(fields_autoplaced yes)
-		(effects
-			(font
-				(size 1.27 1.27)
-			)
-			(justify right)
-		)
-		(property "Intersheetrefs" "${INTERSHEET_REFS}"
-			(at 140.8272 81.28 0)
-			(effects
-				(font
-					(size 1.27 1.27)
-				)
-				(justify right)
-				(hide yes)
-			)
-		)
-	)
 	(symbol
-		(lib_id "Nucleo_F446:NUCLEO-F446RE")
+		(lib_id "Hardware_MCU:NUCLEO-F446RE_Morpho")
 		(at 111.76 86.36 0)
 		(unit 1)
@@
 	)
 	(symbol
-		(lib_id "Nucleo_F446:NUCLEO-F446RE")
+		(lib_id "Hardware_MCU:NUCLEO-F446RE_Morpho")
 		(at 168.91 86.36 0)
 		(unit 2)
@@
 		)
 	)
+(wire (pts (xy 186.69 50.8) (xy 210.82 50.8)) (stroke (width 0) (type default)))
+(hierarchical_label "VREF_SENSOR" (shape output) (at 210.82 50.8 180) (effects (font (size 1.0 1.0)) (justify left)))
+(wire (pts (xy 186.69 121.92) (xy 201.93 121.92)) (stroke (width 0) (type default)))
+(global_label "GND" (shape passive) (at 201.93 121.92 0) (effects (font (size 1.0 1.0)) (justify left)))
+(text "METEO: PA1=chuva; PC7=velocidade; PA0=ADC.
+VREF_SENSOR: AVDD/VREF+ da Nucleo.
+Futura MCU discreta: ligar a mesma fonte da referencia ADC." (at 45.72 152.4 0) (effects (font (size 1.27 1.27)) (justify left top)))
 )

Commit message: design sensores pronto
Connections:
- net PB6 renamed BH_SCK
- net PB7 renamed BH_SDA
Other:
- note removed: "METEO: PA1=chuva; PC7=velocidade; PA0=ADC. VREF_SENSOR: AVDD/VREF+ da Nucleo. Futura MCU discreta: ligar a mesma fonte da referencia ADC."
- moved on the sheet: U5A
