File: Hardware/meteorologia.kicad_sch (KiCad schematic)
At the start: 0 parts

Commit message: Sensores metereologicos -IA que fez
Other:
- sheet BIRUTA ports: added VREF_SENSOR; removed none
Changed lines of the file:
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@@
 	(hierarchical_label "RAIN_PULSE"
 		(shape output)
-		(at 101.6 38.1 0)
+		(at 101.6 38.1 180)
 		(effects
 			(font
@@
 	(hierarchical_label "WIND_SPEED_PULSE"
 		(shape output)
-		(at 101.6 69.85 0)
+		(at 101.6 69.85 180)
 		(effects
 			(font
@@
 	)
 	(hierarchical_label "WIND_DIR_ADC"
-		(shape output)
-		(at 101.6 101.6 0)
+		(shape passive)
+		(at 101.6 101.6 180)
 		(effects
 			(font
@@
 			)
 		)
-		(pin "WIND_DIR_ADC" output
+		(pin "WIND_DIR_ADC" passive
 			(at 73.66 101.6 0)
 			(effects
@@
 			)
 		)
-	)
+	(pin "VREF_SENSOR" input (at 30.48 101.6 180) (effects (font (size 1.27 1.27)) )))
 	(sheet_instances
 		(path "/"
@@
 	)
 	(embedded_fonts no)
+(hierarchical_label "VREF_SENSOR" (shape input) (at 15.24 101.6 0) (effects (font (size 1.0 1.0)) (justify right)))
+(wire (pts (xy 15.24 101.6) (xy 30.48 101.6)) (stroke (width 0) (type default)))
 )
