File: Hardware/pluviometro.kicad_sch (KiCad schematic)
At the start: 1 part, among them J30 R-RJ11R06P-A800

Commit message: Sensores metereologicos -IA que fez
Parts:
- added C30, C31: 100n, Capacitor_SMD:C_0603_1608Metric, symbol Device:C
- added D30: PESD5V0S1UL, Diode_SMD:D_SOD-882, symbol Device:D_Zener
- added D31: BAS70-04, Package_TO_SOT_SMD:SOT-23, symbol Sensores_Meteo:BAS70-04
- added R30: 10k, Resistor_SMD:R_0603_1608Metric, symbol Device:R
- added R31: 4k7, Resistor_SMD:R_0603_1608Metric, symbol Device:R
- added TP30: PLUVIOMETRO_RAW, TestPoint:TestPoint_Pad_D1.5mm, symbol Connector:TestPoint
- added TP31: PLUVIOMETRO_FILT, TestPoint:TestPoint_Pad_D1.5mm, symbol Connector:TestPoint
- added TP32: RAIN_PULSE, TestPoint:TestPoint_Pad_D1.5mm, symbol Connector:TestPoint
- added TP33: GND, TestPoint:TestPoint_Pad_D1.5mm, symbol Connector:TestPoint
- added U30: SN74LVC1G17DBVR, Package_TO_SOT_SMD:SOT-23-5, symbol 74xGxx:74LVC1G17
- J30: Function (none) -> RJ11 individual; contatos centrais; LCSC (none) -> C189750; Manufacturer (none) -> Ckmtw; Rating (none) -> 6P6C; p3=return; p4=signal; THT
Connections:
- net GND: now also C30.2, C31.2, D30.2 (A), D31.1 (A), TP33.1, U30.3 (GND)
- net RAIN_PULSE: now also TP32.1, U30.4; no longer J30.4
- new net: C30.1, D31.3 (COM), R31.2, TP31.1, U30.2
- new net +3V3: C31.1, D31.2 (K), R30.1, U30.5 (VCC)
- new net PLUVIOMETRO_RAW: D30.1 (K), J30.4, R30.2, R31.1, TP30.1
Other:
- note added: "1 CONECTOR / ESD"
- note added: "2 FILTRO / CLAMP"
- note added: "3 SCHMITT / MCU"
- note added: "ESD junto ao RJ11; clamp e C junto ao buffer. Plano GND continuo. Protecao transitoria a validar em bancada; sem isolamento e sem qualificacao contra raios."
- note added: "MISOL: contato reed passivo; cabo externo ~2 m; entrada individual 6P6C p3/p4."
- note added: "Pull-up no lado do cabo evita divisor 4k7/10k na entrada Schmitt. Tau abertura=1,47 ms; fechamento=0,47 ms. Debounce atual: 200 ms."
- note removed: "J30: Ckmtw R-RJ11R06P-A800 / LCSC C189750. Assumido: sensor usa os contatos centrais 3 e 4; confirmar no cabo real. A proteção e o condicionamento serão inseridos entre J30 e RAIN_PULSE."
- company: (none) -> TCC - Estacao meteorologica
- title: (none) -> PLUVIOMETRO - protecao e condicionamento
- moved on the sheet: J30
