File: Hardware/alimentacao.kicad_sch (KiCad schematic)
At the start: 4 parts, among them J10 Conn_GND, J13 Conn_+5V, J9 Conn_+3v3

Commit message: hardware: inicia PCB V2
Changed lines of the file:
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@@
-	(wire
-		(pts
-			(xy 62.23 73.66) (xy 67.31 73.66)
-		)
-		(stroke
-			(width 0)
-			(type default)
-		)
-	)
 	(wire
 		(pts
@@
 	(wire
 		(pts
+			(xy 57.15 68.58) (xy 67.31 68.58)
+		)
+		(stroke
+			(width 0)
+			(type default)
+		)
+	)
+	(wire
+		(pts
 			(xy 76.2 53.34) (xy 78.74 53.34)
 		)
@@
 	(wire
 		(pts
-			(xy 62.23 68.58) (xy 67.31 68.58)
-		)
-		(stroke
-			(width 0)
-			(type default)
-		)
-	)
-	(wire
-		(pts
 			(xy 100.33 60.96) (xy 100.33 64.77)
 		)
@@
 		(pts
 			(xy 73.66 53.34) (xy 76.2 53.34)
+		)
+		(stroke
+			(width 0)
+			(type default)
+		)
+	)
+	(wire
+		(pts
+			(xy 57.15 73.66) (xy 67.31 73.66)
 		)
 		(stroke
@@
 		)
 	)
-	(hierarchical_label "+12V"
-		(shape input)
-		(at 62.23 68.58 180)
-		(effects
-			(font
-				(size 1.27 1.27)
-			)
-			(justify right)
-		)
-	)
 	(hierarchical_label "Gnd"
 		(shape output)
@@
 			)
 			(justify left)
-		)
-	)
-	(hierarchical_label "GND"
-		(shape input)
-		(at 62.23 73.66 180)
-		(effects
-			(font
-				(size 1.27 1.27)
-			)
-			(justify right)
 		)
 	)
@@
 					(unit 1)
 				)
+			)
+		)
+	)
+	(symbol
+		(lib_id "power:+12V")
+		(at 57.15 68.58 0)
+		(unit 1)
+		(exclude_from_sim no)
+		(in_bom yes)
+		(on_board yes)
+		(dnp no)
+		(fields_autoplaced yes)
+		(property "Reference" "#PWR01"
+			(at 57.15 72.39 0)
+			(effects
+				(font
+					(size 1.27 1.27)
+				)
+				(hide yes)
+			)
+		)
+		(property "Value" "+12V"
+			(at 57.15 63.5 0)
+			(effects
+				(font
+					(size 1.27 1.27)
+				)
+			)
+		)
+		(property "Footprint" ""
+			(at 57.15 68.58 0)
+			(effects
+				(font
+					(size 1.27 1.27)
+				)
+				(hide yes)
+			)
+		)
+		(property "Datasheet" ""
+			(at 57.15 68.58 0)
+			(effects
+				(font
+					(size 1.27 1.27)
+				)
+				(hide yes)
+			)
+		)
+		(property "Description" "Power symbol creates a global label with name \"+12V\""
+			(at 57.15 68.58 0)
+			(effects
+				(font
+					(size 1.27 1.27)
+				)
+				(hide yes)
+			)
+		)
+		(pin "1"
+		)
+		(instances
+			(project ""
+				(path "/0c305a6e-f9cd-49a1-b146-c2956e5469b6/19a3c20f-53ab-4562-aabc-58e6e99571a0"
+					(reference "#PWR01")
+					(unit 1)
+				)
+			)
+		)
+	)
+	(symbol
+		(lib_id "power:GND")
+		(at 57.15 73.66 0)
+		(unit 1)
+		(exclude_from_sim no)
+		(in_bom yes)
+		(on_board yes)
+		(dnp no)
+		(fields_autoplaced yes)
+		(property "Reference" "#PWR08"
+			(at 57.15 80.01 0)
+			(effects
+				(font
+					(size 1.27 1.27)
+				)
+				(hide yes)
+			)
+		)
+		(property "Value" "GND"
+			(at 57.15 78.74 0)
+			(effects
+				(font
+					(size 1.27 1.27)
+				)
+			)
+		)
+		(property "Footprint" ""
+			(at 57.15 73.66 0)
+			(effects
+				(font
+					(size 1.27 1.27)
+				)
+				(hide yes)
+			)
+		)
+		(property "Datasheet" ""
+			(at 57.15 73.66 0)
+			(effects
+				(font
+					(size 1.27 1.27)
+				)
+				(hide yes)
+			)
+		)
+		(property "Description" "Power symbol creates a global label with name \"GND\" , ground"
+			(at 57.15 73.66 0)
+			(effects
+				(font
+					(size 1.27 1.27)
+				)
+				(hide yes)
+			)
+		)
+		(pin "1"
+		)
+		(instances
+			(project ""
+				(path "/0c305a6e-f9cd-49a1-b146-c2956e5469b6/19a3c20f-53ab-4562-aabc-58e6e99571a0"
+					(reference "#PWR08")
+					(unit 1)
+				)

Commit message: Sensores metereologicos -IA que fez
Connections:
- net Gnd is gone; now on net GND: J10.1 (Pin_1), J10.10 (Pin_10), J10.2 (Pin_2), J10.3 (Pin_3), J10.4 (Pin_4), J10.5 (Pin_5), J10.6 (Pin_6), J10.7 (Pin_7), J10.8 (Pin_8), J10.9 (Pin_9), PS1.OUT-
Changed lines of the file:
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@@
 		)
 	)
-	(hierarchical_label "Gnd"
+	(hierarchical_label "GND"
 		(shape output)
 		(at 101.6 73.66 0)

Commit message: hardware: implementa alimentacao e adiciona bibliotecas locais - ajuda gpt
Parts:
- removed J10: Conn_GND, Connector_PinSocket_2.54mm:PinSocket_1x10_P2.54mm_Vertical, symbol Connector:Conn_01x10_Socket
- removed J13: Conn_+5V, Connector_PinSocket_2.54mm:PinSocket_1x10_P2.54mm_Vertical, symbol Connector:Conn_01x10_Socket
- removed J9: Conn_+3v3, Connector_PinSocket_2.54mm:PinSocket_1x10_P2.54mm_Vertical, symbol Connector:Conn_01x10_Socket
- removed PS1: Lm2596, myLibrary:LM2596_modulo, symbol LM2596_modulo:MC00100
- added C60: 47u / 35V, Capacitor_SMD:CP_Elec_6.3x5.8, symbol Device:C_Polarized
- added C61, C62: 10u / 50V, Capacitor_SMD:C_1206_3216Metric, symbol Device:C
- added C63, C64: 100n / 50V, Capacitor_SMD:C_0603_1608Metric, symbol Device:C
- added C65, C66, C69: 22u / 25V, Capacitor_SMD:C_1206_3216Metric, symbol Device:C
- added C67, C68: 10u / 25V, Capacitor_SMD:C_0805_2012Metric, symbol Device:C
- added C70: 6p8 / 50V, Capacitor_SMD:C_0603_1608Metric, symbol Device:C
- added D60: SMBJ16CA, Diode_SMD:D_SMB, symbol Device:D_TVS
- added D61: BZT52C10 / 10V, Diode_SMD:D_SOD-123, symbol Device:D_Zener
- added F60: 1.5A / 32V lento, Fuse:Fuse_1206_3216Metric, symbol Device:Fuse
- added J60: P4 / DC-005-2.0, Hardware_Power:DC-IN-TH_DC-005-2.0_C22459640, symbol Hardware_Power:DC-005-2.0_C22459640
- added J61: J_PWR / JST-XH, Connector_JST:JST_XH_B2B-XH-A_1x02_P2.50mm_Vertical, symbol Connector_Generic:Conn_01x02
- added JP60: SEL_FONTE, Jumper:SolderJumper-3_P2.0mm_Open_TrianglePad1.0x1.5mm_NumberLabels, symbol Jumper:SolderJumper_3_Open
- added L60: 4u7 / MWSA0603S, Inductor_SMD:L_Sunlord_MWSA0603S, symbol Device:L
- added L61: 2u2 / MWSA0402S, Inductor_SMD:L_Sunlord_MWSA0402S, symbol Device:L
- added Q60: DMP6023LE-13, Hardware_Power:SOT-223-4_L6.5-W3.5-P2.30-LS7.0-BR, symbol Hardware_Power:DMP6023LE-13
- added R60, R63: 100k / 1%, Resistor_SMD:R_0603_1608Metric, symbol Device:R
- added R61: 300k / 1%, Resistor_SMD:R_0603_1608Metric, symbol Device:R
- added R62: 150k / 1%, Resistor_SMD:R_0603_1608Metric, symbol Device:R
- added TP60: VIN_MAIN, TestPoint:TestPoint_Pad_D1.5mm, symbol Connector:TestPoint
- added TP61: +5V, TestPoint:TestPoint_Pad_D1.5mm, symbol Connector:TestPoint
- added TP62: +3V3, TestPoint:TestPoint_Pad_D1.5mm, symbol Connector:TestPoint
- added TP63: GND, TestPoint:TestPoint_Pad_D1.5mm, symbol Connector:TestPoint
- added U60: AP63205WU-7, Package_TO_SOT_SMD:TSOT-23-6, symbol Regulator_Switching:AP63205WU
- added U61: TLV62569DBVR, Package_TO_SOT_SMD:SOT-23-5, symbol Regulator_Switching:TLV62569DBV
Connections:
- net +3V3: now also C68.1, C69.1, C70.1, L61.2, R61.1, TP62.1
- net +5V: now also C65.1, C66.1, C67.1, L60.2, TP61.1, U60.1 (FB), U61.1 (EN), U61.4 (VIN)
- net GND: now also C60.2, C61.2, C62.2, C63.2, C65.2, C66.2, C67.2, C68.2, C69.2, D60.1 (A1), J60.2, J61.2 (Pin_2), R60.2, R63.2, TP63.1, U60.4 (GND), U61.2 (GND)
- new net: F60.1, JP60.2 (C)
- new net: D60.2 (A2), F60.2, Q60.2 (D), Q60.4 (D)
- new net: C64.1, U60.6 (BST)
- new net: C64.2, L60.1, U60.5 (SW)
- new net: R61.2, R62.1
- new net: D61.2 (A), Q60.1 (G), R60.1
- new net: L61.1, U61.3 (SW)
- new net ENERGIA_POS: J61.1 (Pin_1), JP60.1 (A)
- new net FB_3V3: C70.2, R62.2, R63.1, U61.5 (FB)
- new net P4_POS: J60.1, JP60.3 (B)
- new net VIN_MAIN: C60.1, C61.1, C62.1, C63.1, D61.1 (K), Q60.3 (S), TP60.1, U60.2 (EN), U60.3 (IN)
Other:
- note added: "1 ENTRADAS / SELECAO / PROTECAO"
- note added: "2 BUCK 5 V | CI 2 A / VALIDAR TERMICA"
- note added: "3 BUCK 3,3 V | SEM MCU PARA PARTIDA"
- note added: "ALIMENTACAO DA PCB PRINCIPAL | entrada nominal 12 V, nao regulada | faixa de projeto 10 a 16 Vcc"
- note added: "C68=10uF +30,5uF existentes =40,5uF; C69 DNP. Alvo3V3 <=1A; validar carga/termica. Sem LED permanente. NAO unir3V3 ao regulador3V3 da Nucleo; evitar retorno porUSB."
- note added: "FB: medir apos L60"
- note added: "JP60 aberto: placa desligada. Fechar SOMENTE 1-2 (J_PWR) ou 2-3 (P4). Nunca fechar os tres pads. Desenergizar antes de alterar. GNDs sao comuns."
- note added: "L60=4,7uH; C65+C66=44uF nominais; FB ligado APOS L60. C61/C62/C63 fisicamente junto a U60, apesar de desenhados acima. Alvo inicial: 5V externo <=0,5A + carga do buck3V3; validar termica."
- note added: "Nao conectar bateria sem LVD/fusivel externo. Nao ha OR automatico nesta PCB. TVS nao protege contra sobretensao sustentada nem raio direto."
- note added: "Placa externa: solar / VRLA / carregador / LVD. J61 requer fusivel e limitacao de corrente externos. PCB: protecao + bucks."
- note added: "REFERENCIAS: Diodes AP63205 DS41326 Fig.21/Tab.3; TI TLV62569 SLVSDG1C sec.8.2/10. LAYOUT: malhas VIN-CIN-GND curtas; SW minimo; FB longe deSW; planoGND continuo. Detalhes, BOM/LCSC e limites: docs/alimentacao/README.md"
- company: (none) -> TCC - Estacao meteorologica
- title: (none) -> PCB PRINCIPAL - alimentacao local protegida
