File: Hardware/esquematico_V4.kicad_pcb (KiCad board)
At the start: 2 copper layers, 200 x 100 mm, 50 parts, among them J1 Conn_SPI, J10 Conn_GND, J11 Conn_01x02_Socket, J12 Conn_SPI, J13 Conn_+5V, J14 Conn_01x02_Socket, J15 Conn_01x02_Socket, J16 Conn_01x02_Socket, J17 Conn_01x02_Socket, J18 Conn_01x02_Socket, J19 Conn_01x02_Socket, J2 Conn_DHT, J20 Conn_01x02_Socket, J21 Conn_01x02_Socket, J22 Conn_01x02_Socket, J23 RJ45, J24 RJ45, J25 RJ45, J3 Conn_SPI, J4 Conn_cartao_SD, J5 Conn_BH1750, J6 Conn_BMP, J7 Conn_Lora_4, J8 Conn_02x06_Row_Letter_Last, J9 Conn_+3v3, U1 DHT22, U2 module_bh1750, U3 module_bme280, U4 Lora_Sx1276, U6 MicroSD Card Adapter, U7 NUCLEO-F446RE

Commit message: hardware: inicia PCB V2
Parts:
- added C4: 100n, Capacitor_THT:C_Disc_D3.8mm_W2.6mm_P2.50mm, F.Cu at (94.0, 124.5)
- added C5: 100n, Capacitor_THT:C_Disc_D3.8mm_W2.6mm_P2.50mm, F.Cu at (172.7, 129.5)
- added J14: Conn_01x02_Socket, Connector_PinSocket_2.54mm:PinSocket_1x02_P2.54mm_Vertical, F.Cu at (134.6, 121.9)
- added J15: Conn_01x02_Socket, Connector_PinSocket_2.54mm:PinSocket_1x02_P2.54mm_Vertical, F.Cu at (170.2, 121.9)
- added J16: Conn_01x02_Socket, Connector_PinSocket_2.54mm:PinSocket_1x02_P2.54mm_Vertical, F.Cu at (88.9, 119.3)
- added R10: 10k, Resistor_THT:R_Axial_DIN0204_L3.6mm_D1.6mm_P7.62mm_Horizontal, F.Cu at (87.6, 132.0)
- added R11: 10k, Resistor_THT:R_Axial_DIN0204_L3.6mm_D1.6mm_P7.62mm_Horizontal, F.Cu at (166.4, 133.3)
- added R8: 10k, Resistor_THT:R_Axial_DIN0204_L3.6mm_D1.6mm_P7.62mm_Horizontal, F.Cu at (129.5, 119.4)
- moved J15 23.0 mm to (-155.7, 125.2)
- moved J24 3.32 mm to (127.6, 130.3)
Routing:
- net +3V3: track 45.1 -> 357.8 mm
- net GND: track 65.5 -> 170.6 mm
- net PA1: track 32.4 -> 64.3 mm
- net PC7: track 53.6 -> 69.9 mm
- net PA0: track 31.9 -> 41.3 mm
- net PA8: track 73.9 -> 65.0 mm

Commit message: hardware: adiciona sensores e cartao SD
Parts:
- added U8: BMP280, Package_LGA:Bosch_LGA-8_2x2.5mm_P0.65mm_ClockwisePinNumbering, F.Cu at (227.6, 57.6)
- added U9: BH1750FVI-TR, myLibrary:BH1750FVI-TR_sensor, F.Cu at (227.3, 50.8)
Connections:
- net +5V renamed VCC
- C4 pad 2: GND -> Gnd
- C5 pad 2: GND -> Gnd
- J10 pad 1: GND -> Gnd
- J10 pad 10: GND -> Gnd
- J10 pad 2: GND -> Gnd
- J10 pad 3: GND -> Gnd
- J10 pad 4: GND -> Gnd
- J10 pad 5: GND -> Gnd
- J10 pad 6: GND -> Gnd
- J10 pad 7: GND -> Gnd
- J10 pad 8: GND -> Gnd
- J10 pad 9: GND -> Gnd
- J14 pad 2: GND -> Gnd
- J2 pad 1: GND -> Gnd
- J4 pad 6: GND -> Gnd
- J5 pad 2: GND -> Gnd
- J5 pad 5: GND -> Gnd
- J6 pad 1: GND -> Gnd
- J6 pad 5: GND -> Gnd
- J8 pad 11: GND -> Gnd
- J8 pad 12: GND -> Gnd
- PS1 pad IN-: GND -> Gnd
- PS1 pad OUT-: GND -> Gnd
- R10 pad 1: GND -> Gnd
- R11 pad 1: GND -> Gnd
- U1 pad 4: GND -> Gnd
- U2 pad 1: GND -> Gnd
- U2 pad 4: GND -> Gnd
- U3 pad 2: GND -> Gnd
- U3 pad 6: GND -> Gnd
- U4 pad 16: GND -> Gnd
- U4 pad 2: GND -> Gnd
- U4 pad 9: GND -> Gnd
- U6 pad 1: GND -> Gnd
- U7 pad CN10_17: PB6 -> SCK
- U7 pad CN10_20: GND -> Gnd
- U7 pad CN10_9: GND -> Gnd
- U7 pad CN7_19: GND -> Gnd
- U7 pad CN7_20: GND -> Gnd
- U7 pad CN7_21: PB7 -> SDA
- U7 pad CN7_22: GND -> Gnd
- U7 pad CN7_34: PB0 -> unconnected-(U7A-PB0-PadCN7_34)
- U7 pad CN7_8: GND -> Gnd
Routing:
- net Gnd: track 0.00 -> 170.6 mm
- net GND: track 170.6 -> 0.00 mm

Commit message: Add subfolhas DHT22 e LORA
Parts:
- added J17: Micro_SD_Card, Connector_Card:microSD_HC_Molex_104031-0811, F.Cu at (103.0, 101.3)
- added U11: 74LVC125, Package_SO:TSSOP-14_4.4x5mm_P0.65mm, F.Cu at (81.3, 83.8)
- added U12: LORA1276-C1-915MHZ, LoRa1276_C1:COMM-SMD_LORA1276-C1-915MHZ, F.Cu at (56.8, 127.0)
- added U5: NUCLEO-F446RE, myLibrary:MODULE_NUCLEO-F446RE, F.Cu at (-163.8, 1.89)
- moved U4 180.4 mm to (76.1, 126.5)

Commit message: hardware: implementa alimentacao e adiciona bibliotecas locais - ajuda gpt
Parts:
- removed C1, C2, C3: 100n, Capacitor_THT:C_Disc_D3.8mm_W2.6mm_P2.50mm
- removed J1, J12, J3: Conn_SPI, Connector_PinSocket_2.54mm:PinSocket_1x03_P2.54mm_Vertical
- removed the J14 at (-183.2, 122.7)
- removed the J15 at (-155.7, 125.2)
- removed the J16 at (-174.0, 122.7)
- removed the J17 at (-169.4, 122.7)
- removed J18, J19, J20, J21, J22: Conn_01x02_Socket, Connector_PinSocket_2.54mm:PinSocket_1x02_P2.54mm_Vertical
- removed R1: 500, Resistor_THT:R_Axial_DIN0204_L3.6mm_D1.6mm_P7.62mm_Horizontal
- removed R2: 2000, Resistor_THT:R_Axial_DIN0204_L3.6mm_D1.6mm_P7.62mm_Horizontal
- removed R3: 5k, Resistor_THT:R_Axial_DIN0204_L3.6mm_D1.6mm_P7.62mm_Horizontal
- removed R4, R9: 10k, Resistor_THT:R_Axial_DIN0204_L3.6mm_D1.6mm_P7.62mm_Horizontal
- removed R5, R6: 1k, Resistor_THT:R_Axial_DIN0204_L3.6mm_D1.6mm_P7.62mm_Horizontal
- removed the R8 at (-95.5, 59.9)
- removed S1, S2, S3, S4, S5, S6: MISM7R1015, myLibrary:Reed_Switch
- added C30: 100n, Capacitor_SMD:C_0603_1608Metric, F.Cu at (-110.5, 88.0)
- added C31: 100n, Capacitor_SMD:C_0603_1608Metric, F.Cu at (-110.5, 90.5)
- added C40: 10n, Capacitor_SMD:C_0603_1608Metric, F.Cu at (-135.5, 88.0)
- added C41: 100n, Capacitor_SMD:C_0603_1608Metric, F.Cu at (-135.5, 90.5)
- added C50: 10n, Capacitor_SMD:C_0603_1608Metric, F.Cu at (-62.0, 69.8)
- added C60: 47u / 35V, Capacitor_SMD:CP_Elec_6.3x5.8, F.Cu at (-68.0, 16.5)
- added C61: 10u / 50V, Capacitor_SMD:C_1206_3216Metric, F.Cu at (-80.1, 14.1)
- added C62: 10u / 50V, Capacitor_SMD:C_1206_3216Metric, F.Cu at (-80.1, 17.4)
- added C63: 100n / 50V, Capacitor_SMD:C_0603_1608Metric, F.Cu at (-75.3, 13.7)
- added C64: 100n / 50V, Capacitor_SMD:C_0603_1608Metric, F.Cu at (-75.3, 16.2)
- added C65: 22u / 25V, Capacitor_SMD:C_1206_3216Metric, F.Cu at (-80.1, 20.8)
- added C66: 22u / 25V, Capacitor_SMD:C_1206_3216Metric, F.Cu at (-80.1, 24.1)
- added C67: 10u / 25V, Capacitor_SMD:C_0805_2012Metric, F.Cu at (-52.6, 7.72)
- added C68: 10u / 25V, Capacitor_SMD:C_0805_2012Metric, F.Cu at (-52.6, 10.7)
- added C69: 22u / 25V, Capacitor_SMD:C_1206_3216Metric, F.Cu at (-80.1, 27.5)
- added C70: 6p8 / 50V, Capacitor_SMD:C_0603_1608Metric, F.Cu at (-75.3, 18.7)
- added D30: PESD5V0S1UL, Diode_SMD:D_SOD-882, F.Cu at (-125.2, 102.1)
- added D31: BAS70-04, Package_TO_SOT_SMD:SOT-23, F.Cu at (-129.0, 103.2)
- added D40: PESD5V0S1UL, Diode_SMD:D_SOD-882, F.Cu at (-150.2, 102.1)
- added D41: BAS70-04, Package_TO_SOT_SMD:SOT-23, F.Cu at (-159.1, 108.3)
- added D50: PESD5V0S1UL, Diode_SMD:D_SOD-882, F.Cu at (-62.6, 79.7)
- added D51: BAS70-04, Package_TO_SOT_SMD:SOT-23, F.Cu at (-65.1, 85.0)
- added D60: SMBJ16CA, Diode_SMD:D_SMB, F.Cu at (-57.4, 3.44)
- added D61: BZT52C10 / 10V, Diode_SMD:D_SOD-123, F.Cu at (-66.8, 30.3)
- added F60: 1.5A / 32V lento, Fuse:Fuse_1206_3216Metric, F.Cu at (-80.1, 30.8)
- added J30: R-RJ11R06P-A800, Sensores_Meteo:RJ11-TH_PCB-6P6C-90, F.Cu at (-123.8, 90.8)
- added J31: R-RJ11R06P-A800, Sensores_Meteo:RJ11-TH_PCB-6P6C-90, F.Cu at (-148.8, 90.8)
- added J32: R-RJ11R06P-A800, Sensores_Meteo:RJ11-TH_PCB-6P6C-90, F.Cu at (-75.2, 72.6)
- added J60: P4 / DC-005-2.0, Hardware_Power:DC-IN-TH_DC-005-2.0_C22459640, F.Cu at (-71.5, 8.34)
- added J61: J_PWR / JST-XH, Connector_JST:JST_XH_B2B-XH-A_1x02_P2.50mm_Vertical, F.Cu at (-56.5, 23.9)
- added JP60: SEL_FONTE, Jumper:SolderJumper-3_P2.0mm_Open_TrianglePad1.0x1.5mm_NumberLabels, F.Cu at (-53.3, 33.0)
- added L60: 4u7 / MWSA0603S, Inductor_SMD:L_Sunlord_MWSA0603S, F.Cu at (-57.8, 16.5)
- added L61: 2u2 / MWSA0402S, Inductor_SMD:L_Sunlord_MWSA0402S, F.Cu at (-58.2, 9.09)
- added Q60: DMP6023LE-13, Hardware_Power:SOT-223-4_L6.5-W3.5-P2.30-LS7.0-BR, F.Cu at (-64.9, 24.6)
- added R30: 10k, Resistor_SMD:R_0603_1608Metric, F.Cu at (-110.5, 93.0)
- added R31: 4k7, Resistor_SMD:R_0603_1608Metric, F.Cu at (-110.5, 95.5)
- added R40: 10k, Resistor_SMD:R_0603_1608Metric, F.Cu at (-135.5, 93.0)
- added R41: 4k7, Resistor_SMD:R_0603_1608Metric, F.Cu at (-135.5, 95.5)
- added R50: 10k, Resistor_SMD:R_0603_1608Metric, F.Cu at (-62.0, 72.3)
- added R51: 10k, Resistor_SMD:R_0603_1608Metric, F.Cu at (-62.0, 74.8)
- added R52: 1k, Resistor_SMD:R_0603_1608Metric, F.Cu at (-62.0, 77.3)
- added R60: 100k / 1%, Resistor_SMD:R_0603_1608Metric, F.Cu at (-75.3, 21.2)
- added R61: 300k / 1%, Resistor_SMD:R_0603_1608Metric, F.Cu at (-75.3, 23.7)
- added R62: 150k / 1%, Resistor_SMD:R_0603_1608Metric, F.Cu at (-75.3, 26.2)
- added R63: 100k / 1%, Resistor_SMD:R_0603_1608Metric, F.Cu at (-75.3, 28.7)
- added TP30: PLUVIOMETRO_RAW, TestPoint:TestPoint_Pad_D1.5mm, F.Cu at (-114.3, 88.5)
- added TP31: PLUVIOMETRO_FILT, TestPoint:TestPoint_Pad_D1.5mm, F.Cu at (-114.3, 92.0)
- added TP32: RAIN_PULSE, TestPoint:TestPoint_Pad_D1.5mm, F.Cu at (-114.3, 95.6)
- added TP33: GND, TestPoint:TestPoint_Pad_D1.5mm, F.Cu at (-114.3, 99.1)
- added TP40: ANEMOMETRO_RAW, TestPoint:TestPoint_Pad_D1.5mm, F.Cu at (-139.3, 88.5)
- added TP41: ANEMOMETRO_FILT, TestPoint:TestPoint_Pad_D1.5mm, F.Cu at (-139.3, 92.0)
- added TP42: WIND_SPEED_PULSE, TestPoint:TestPoint_Pad_D1.5mm, F.Cu at (-139.3, 95.6)
- added TP43: GND, TestPoint:TestPoint_Pad_D1.5mm, F.Cu at (-139.3, 99.1)
- added TP50: WIND_DIR_RAW, TestPoint:TestPoint_Pad_D1.5mm, F.Cu at (-65.7, 70.3)
- added TP51: WIND_DIR_ADC, TestPoint:TestPoint_Pad_D1.5mm, F.Cu at (-65.7, 73.8)
- added TP52: VREF_SENSOR, TestPoint:TestPoint_Pad_D1.5mm, F.Cu at (-65.7, 77.4)
- added TP53: GND, TestPoint:TestPoint_Pad_D1.5mm, F.Cu at (-55.9, 81.0)
- added TP60: VIN_MAIN, TestPoint:TestPoint_Pad_D1.5mm, F.Cu at (-71.5, 22.3)
- added TP61: +5V, TestPoint:TestPoint_Pad_D1.5mm, F.Cu at (-71.5, 25.9)
- added TP62: +3V3, TestPoint:TestPoint_Pad_D1.5mm, F.Cu at (-71.5, 29.4)
- added TP63: GND, TestPoint:TestPoint_Pad_D1.5mm, F.Cu at (-71.5, 33.0)
- added U1: DHT22, myLibrary:XDCR_DHT22, F.Cu at (-74.4, 50.2)
- added U30: SN74LVC1G17DBVR, Package_TO_SOT_SMD:SOT-23-5, F.Cu at (-113.5, 103.3)
- added U40: SN74LVC1G17DBVR, Package_TO_SOT_SMD:SOT-23-5, F.Cu at (-143.6, 108.3)
- added U60: AP63205WU-7, Package_TO_SOT_SMD:TSOT-23-6, F.Cu at (-64.2, 3.06)
- added U61: TLV62569DBVR, Package_TO_SOT_SMD:SOT-23-5, F.Cu at (-64.2, 7.69)
- moved J11 76.9 mm to (-101.7, 89.0)
- moved U5 59.4 mm to (-120.7, 42.7)
- moved R7 36.1 mm to (-64.5, 38.3)
Connections:
- net ADDR renamed /BH1750/BH_ADDR
- net CSB renamed /BMP280/BMP_CSB
- net MCU_CS renamed /Cartao SD/SD_CS
- net MCU_MISO renamed /Cartao SD/SD_MISO
- net MCU_MOSI renamed /Cartao SD/MCU_MOSI
- net MCU_SCK renamed /Cartao SD/SD_SCK
- net SDO renamed /BMP280/BMP_SDO
- net SD_CARD_DETECT renamed /Cartao SD/SD_CD
- J17 pad 10: Gnd -> GND
- J17 pad 11: Gnd -> GND
- J17 pad 6: Gnd -> GND
- J4 pad 5: VCC -> +5V
- J4 pad 6: Gnd -> GND
- J5 pad 2: Gnd -> GND
- J5 pad 5: Gnd -> GND
- J6 pad 1: Gnd -> GND
- J6 pad 5: Gnd -> GND
- R7 pad 1: PA8 -> /DHT22/PA8
- R7 pad 2: VCC -> +5V
- U11 pad 1: Gnd -> GND
- U11 pad 10: Gnd -> GND
- U11 pad 13: Gnd -> GND
- U11 pad 14: VCC -> +5V
- U11 pad 4: Gnd -> GND
- U12 pad 1: unconnected-(U12-GND-Pad1) -> GND
- U12 pad 10: unconnected-(U12-GND-Pad10) -> GND
- U12 pad 13: unconnected-(U12-VCC-Pad13) -> +3V3
- U12 pad 14: unconnected-(U12-DIO0-Pad14) -> /LORA Module/Lora_DIO0
- U12 pad 15: unconnected-(U12-DIO1-Pad15) -> /LORA Module/Lora_DIO1
- U12 pad 16: unconnected-(U12-DIO2-Pad16) -> /LORA Module/Lora_DIO2
- U12 pad 2: unconnected-(U12-MISO-Pad2) -> /LORA Module/Lora_MISO
- U12 pad 3: unconnected-(U12-MOSI-Pad3) -> /LORA Module/Lora_MOSI
- U12 pad 4: unconnected-(U12-SCK-Pad4) -> /LORA Module/Lora_SCK
- U12 pad 5: unconnected-(U12-NSS-Pad5) -> /LORA Module/Lora_NSS
- U12 pad 6: unconnected-(U12-NRESET-Pad6) -> /LORA Module/Lora_RST
- U12 pad 8: unconnected-(U12-GND-Pad8) -> GND
- U12 pad 9: unconnected-(U12-ANT-Pad9) -> ANT_EXT
- U2 pad 1: Gnd -> GND
- U2 pad 4: Gnd -> GND
- U3 pad 2: Gnd -> GND
- U3 pad 6: Gnd -> GND
- U5 pad CN10_17: PB6 -> /mcu/BH_SCK
- U5 pad CN10_19: PC7 -> WIND_SPEED_PULSE
- U5 pad CN10_20: Gnd -> GND
- U5 pad CN10_32: unconnected-(U5B-AGND-PadCN10_32) -> GND
- U5 pad CN10_7: unconnected-(U5B-AVDD-PadCN10_7) -> VREF_SENSOR
- U5 pad CN10_9: Gnd -> GND
- U5 pad CN7_18: VCC -> +5V
- U5 pad CN7_19: Gnd -> GND
- U5 pad CN7_20: Gnd -> GND
- U5 pad CN7_21: PB7 -> /mcu/BH_SDA
- U5 pad CN7_22: Gnd -> GND
- U5 pad CN7_28: PA0 -> WIND_DIR_ADC
- U5 pad CN7_30: PA1 -> RAIN_PULSE
- U5 pad CN7_8: Gnd -> GND
- U6 pad 1: Gnd -> GND
- U6 pad 2: VCC -> +5V
- U8 pad 1: Gnd -> GND
- U8 pad 3: SDA -> /BMP280/BMP_SDA
- U8 pad 4: SCK -> /BMP280/BMP_SCK
- U8 pad 6: VDD -> +3V3
- U8 pad 7: Gnd -> GND
- U9 pad 3: Gnd -> GND
Routing:
- net Gnd: track 170.6 -> 137.8 mm
- net GND: track 0.00 -> 32.8 mm
