File: hardware/kicad/estacao-meteorologica/sheets/Lora_module.kicad_sch (KiCad schematic)
At the start: 5 parts, among them U12 LORA1276-C1-915MHZ

Commit message: refatoracao: atualizacoes de hardware e falta revisao LoRa
Changed lines of the file:
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@@
-		)
-	)
-	(global_label "PC4"
-		(shape input)
-		(at 85.09 95.25 180)
-		(fields_autoplaced yes)
-		(effects
-			(font
-				(size 1.27 1.27)
-			)
-			(justify right)
-		)
-		(property "Intersheetrefs" "${INTERSHEET_REFS}"
-			(at 78.3553 95.25 0)
-			(effects
-				(font
-					(size 1.27 1.27)
-				)
-				(justify right)
-				(hide yes)
-			)
-		)
-	)
-	(global_label "PB12"
-		(shape input)
-		(at 85.09 92.71 180)
-		(fields_autoplaced yes)
-		(effects
-			(font
-				(size 1.27 1.27)
-			)
-			(justify right)
-		)
-		(property "Intersheetrefs" "${INTERSHEET_REFS}"
-			(at 77.1458 92.71 0)
-			(effects
-				(font
-					(size 1.27 1.27)
-				)
-				(justify right)
-				(hide yes)
-			)
-		)
-	)
-	(global_label "PA12"
-		(shape input)
-		(at 187.96 85.09 0)
-		(fields_autoplaced yes)
-		(effects
-			(font
-				(size 1.27 1.27)
-			)
-			(justify left)
-		)
-		(property "Intersheetrefs" "${INTERSHEET_REFS}"
-			(at 195.7228 85.09 0)
-			(effects
-				(font
-					(size 1.27 1.27)
-				)
-				(justify left)
-				(hide yes)
-			)
-		)
-	)
-	(global_label "PA11"
-		(shape input)
-		(at 187.96 87.63 0)
-		(fields_autoplaced yes)
-		(effects
-			(font
-				(size 1.27 1.27)
-			)
-			(justify left)
-		)
-		(property "Intersheetrefs" "${INTERSHEET_REFS}"
-			(at 195.7228 87.63 0)
-			(effects
-				(font
-					(size 1.27 1.27)
-				)
-				(justify left)
-				(hide yes)
-			)
-		)
-	)
-	(global_label "PB15"
-		(shape input)
-		(at 85.09 87.63 180)
-		(fields_autoplaced yes)
-		(effects
-			(font
-				(size 1.27 1.27)
-			)
-			(justify right)
-		)
-		(property "Intersheetrefs" "${INTERSHEET_REFS}"
-			(at 77.1458 87.63 0)
-			(effects
-				(font
-					(size 1.27 1.27)
-				)
-				(justify right)
-				(hide yes)
-			)
-		)
-	)
-	(global_label "PB13"
-		(shape input)
-		(at 85.09 90.17 180)
-		(fields_autoplaced yes)
-		(effects
-			(font
-				(size 1.27 1.27)
-			)
-			(justify right)
-		)
-		(property "Intersheetrefs" "${INTERSHEET_REFS}"
-			(at 77.1458 90.17 0)
-			(effects
-				(font
-					(size 1.27 1.27)
-				)
-				(justify right)
-				(hide yes)
-			)
-		)
-	)
-	(global_label "DIO2"
-		(shape input)
-		(at 187.96 82.55 0)
-		(fields_autoplaced yes)
-		(effects
-			(font
-				(size 1.27 1.27)
-			)
-			(justify left)
-		)
-		(property "Intersheetrefs" "${INTERSHEET_REFS}"
-			(at 195.36 82.55 0)
-			(effects
-				(font
-					(size 1.27 1.27)
-				)
-				(justify left)
-				(hide yes)
-			)
 		)
 	)
@@
 				(hide yes)
 			)
-		)
-	)
-	(global_label "PB14"
-		(shape input)
-		(at 85.09 85.09 180)
-		(fields_autoplaced yes)
-		(effects
-			(font
-				(size 1.27 1.27)
-			)
-			(justify right)
-		)
-		(property "Intersheetrefs" "${INTERSHEET_REFS}"
-			(at 77.1458 85.09 0)
-			(effects
-				(font
-					(size 1.27 1.27)
-				)
-				(justify right)
-				(hide yes)
-			)

Commit message: refatoracao: lora + Verificacao projeto inteiro
Parts:
- added D70: PESD5V0R1BSFYL, Hardware_LoRa:SOD-962_L0.6-W0.3-BI, symbol Hardware_LoRa:PESD5V0R1BSFYL
- added FB70: 120R @100MHz / 2A, Inductor_SMD:L_0603_1608Metric, symbol Device:FerriteBead
- added J70: U.FL / 50 ohm, Hardware_LoRa:U.FL_Hirose_U.FL-R-SMT-1_Vertical, symbol Hardware_LoRa:U.FL-R-SMT-1_10
- C11: footprint (none) -> Capacitor_SMD:C_0603_1608Metric; LCSC (none) -> C14663; LCSC Part (none) -> C14663; MPN (none) -> CC0603KRX7R9BB104; Manufacturer (none) -> YAGEO; Modelo 3D (none) -> ${KICAD9_3DMODEL_DIR}/Capacitor_SMD.3dshapes/C_0603_1608Met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; Status_Ficha (none) -> Conferido no catalogo em 2026-09-24; verificar estoque ao c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
- C12: footprint (none) -> Capacitor_SMD:C_1206_3216Metric; LCSC (none) -> C13585; LCSC Part (none) -> C13585; MPN (none) -> CL31A106KBHNNNE; Manufacturer (none) -> Samsung Electro-Mechanics; Modelo 3D (none) -> ${KICAD9_3DMODEL_DIR}/Capacitor_SMD.3dshapes/C_1206_3216Met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; Status_Ficha (none) -> Conferido no catalogo em 2026-09-24; verificar estoque ao c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
- R14, R15: footprint (none) -> Resistor_SMD:R_0603_1608Metric; LCSC (none) -> C25804; LCSC Part (none) -> C25804; MPN (none) -> 0603WAF1002T5E; Manufacturer (none) -> UNI-ROYAL(Uniroyal Elec); Modelo 3D (none) -> ${KICAD9_3DMODEL_DIR}/Resistor_SMD.3dshapes/R_0603_1608Metr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; Status_Ficha (none) -> Conferido no catalogo em 2026-09-24; verificar estoque ao c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
- U12: footprint LoRa1276_C1:COMM-SMD_LORA1276-C1-915MHZ -> Hardware_LoRa:COMM-SMD_LORA1276-C1-915MHZ; symbol LoRa1276_C1:LORA1276-C1-915MHZ -> Hardware_LoRa:LORA1276-C1-915MHZ; LCSC (none) -> C3001531; Manufacturer G-NiceRF(思为无线) -> G-NiceRF; Modelo 3D (none) -> ${KIPRJMOD}/../../libraries/Hardware_LoRa/Hardware_LoRa.3ds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; Status_Ficha (none) -> Conferido no catalogo em 2026-09-24; verificar estoque ao c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
Connections:
- net +3V3: now also FB70.1; no longer C11.1, C12.1, R14.1, R15.1, U12.13 (VCC)
- net GND: now also D70.1 (A1), J70.2 (Ext)
- net ANT_EXT renamed RF_ANT_915
- net RF_ANT_915: now also D70.2 (A2), J70.1 (In)
- new net VCC_LORA: C11.1, C12.1, FB70.2, R14.1, R15.1, U12.13 (VCC)
Other:
- note added: "Antena/pigtail 915 MHz, 50 ohm, U.FL compativel (nao MHF4). Nao transmitir sem antena."
- note added: "D70: protecao ESD de baixa capacitancia; nao protege contra descarga atmosferica direta."
- note added: "DIO0 -> PA11; DIO1 -> PA12; DIO2 -> PB0 (EXTI0). DIO3/4/5 reservados, sem conexao."
- note added: "FB70 filtra a alimentacao local. C11/C12: 100 nF + 10 uF junto ao VCC do modulo."
- note added: "Firmware pendente: configurar PB0/DIO2 e revisar reset em open-drain/alta impedancia."
- note added: "LoRa 915 MHz | SPI 3,3 V | antena externa U.FL"
- note added: "NSS: pull-up mantem radio deselecionado na partida. NRESET ativo em LOW; liberar apos reset."
- note added: "PCB: RF_ANT_915 curta, impedancia 50 ohm; D70 junto ao U.FL e retorno GND curto com vias."
