File: hardware/kicad/estacao-meteorologica/sheets/meteorologia.kicad_sch (KiCad schematic)
At the start: 0 parts

Commit message: refatoracao: atualizacoes de hardware e falta revisao LoRa
Other:
- sheet BIRUTA ports: added AVREF_SENSOR; removed VREF_SENSOR
Changed lines of the file:
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@@
 	(text "Folha de integração dos sensores meteorológicos.\nCada subfolha contém o conector RJ11 e seu condicionamento dedicado."
 		(exclude_from_sim no)
-		(at 30.48 20.32 0)
+		(at 119.38 44.45 0)
 		(effects
 			(font
@@
 	(wire
 		(pts
-			(xy 73.66 38.1) (xy 101.6 38.1)
-		)
-		(stroke
-			(width 0)
-			(type default)
-		)
-	)
-	(wire
-		(pts
-			(xy 73.66 101.6) (xy 101.6 101.6)
-		)
-		(stroke
-			(width 0)
-			(type default)
-		)
-	)
-	(wire
-		(pts
-			(xy 15.24 101.6) (xy 30.48 101.6)
-		)
-		(stroke
-			(width 0)
-			(type default)
-		)
-	)
-	(wire
-		(pts
-			(xy 73.66 69.85) (xy 101.6 69.85)
+			(xy 109.22 124.46) (xy 119.38 124.46)
+		)
+		(stroke
+			(width 0)
+			(type default)
+		)
+	)
+	(wire
+		(pts
+			(xy 162.56 62.23) (xy 190.5 62.23)
+		)
+		(stroke
+			(width 0)
+			(type default)
+		)
+	)
+	(wire
+		(pts
+			(xy 162.56 123.19) (xy 190.5 123.19)
+		)
+		(stroke
+			(width 0)
+			(type default)
+		)
+	)
+	(wire
+		(pts
+			(xy 162.56 91.44) (xy 190.5 91.44)
 		)
 		(stroke
@@
 	(hierarchical_label "RAIN_PULSE"
 		(shape output)
-		(at 101.6 38.1 0)
+		(at 190.5 62.23 0)
 		(effects
 			(font
@@
 		)
 	)
-	(hierarchical_label "VREF_SENSOR"
+	(hierarchical_label "AVREF_SENSOR"
 		(shape input)
-		(at 15.24 101.6 180)
+		(at 109.22 124.46 180)
 		(effects
 			(font
@@
 	(hierarchical_label "WIND_DIR_ADC"
 		(shape passive)
-		(at 101.6 101.6 0)
+		(at 190.5 123.19 0)
 		(effects
 			(font
@@
 	(hierarchical_label "WIND_SPEED_PULSE"
 		(shape output)
-		(at 101.6 69.85 0)
+		(at 190.5 91.44 0)
 		(effects
 			(font
@@
 	)
 	(sheet
-		(at 30.48 93.98)
+		(at 119.38 115.57)
 		(size 43.18 15.24)
 		(exclude_from_sim no)
@@
 		)
 		(property "Sheetname" "BIRUTA"
-			(at 30.48 93.2684 0)
+			(at 119.38 114.8584 0)
 			(effects
 				(font
@@
 		)
 		(property "Sheetfile" "biruta.kicad_sch"
-			(at 30.48 109.9316 0)
+			(at 119.38 131.5216 0)
 			(effects
 				(font
@@
 		)
 		(pin "WIND_DIR_ADC" passive
-			(at 73.66 101.6 0)
+			(at 162.56 123.19 0)
 			(effects
 				(font
@@
 			)
 		)
-		(pin "VREF_SENSOR" input
-			(at 30.48 101.6 180)
-			(effects
-				(font
-					(size 1.27 1.27)
-				)
+		(pin "AVREF_SENSOR" input
+			(at 119.38 124.46 180)
+			(effects
+				(font
+					(size 1.27 1.27)
+				)
+				(justify left)
 			)
 		)
 		(instances
-			(project "esquematico_V4"
+			(project "estacao-meteorologica"
 				(path "/0c305a6e-f9cd-49a1-b146-c2956e5469b6/058dce74-971b-49d7-82f0-384e20be985c"
 					(page "12")
@@
 	)
 	(sheet
-		(at 30.48 62.23)
+		(at 119.38 83.82)
 		(size 43.18 15.24)
 		(exclude_from_sim no)
@@
 		)
 		(property "Sheetname" "ANEMOMETRO"
-			(at 30.48 61.5184 0)
+			(at 119.38 83.1084 0)
 			(effects
 				(font
@@
 		)
 		(property "Sheetfile" "anemometro.kicad_sch"
-			(at 30.48 78.1816 0)
+			(at 119.38 99.7716 0)
 			(effects
 				(font
@@
 		)
 		(pin "WIND_SPEED_PULSE" output
-			(at 73.66 69.85 0)
+			(at 162.56 91.44 0)
 			(effects
 				(font
@@
 		)
 		(instances
-			(project "esquematico_V4"
+			(project "estacao-meteorologica"
 				(path "/0c305a6e-f9cd-49a1-b146-c2956e5469b6/058dce74-971b-49d7-82f0-384e20be985c"
 					(page "11")
@@
 	)
 	(sheet
-		(at 30.48 30.48)
+		(at 119.38 54.61)
 		(size 43.18 15.24)
 		(exclude_from_sim no)
@@
 		)
 		(property "Sheetname" "PLUVIOMETRO"
-			(at 30.48 29.7684 0)
+			(at 119.38 53.8984 0)
 			(effects
 				(font
@@
 		)
 		(property "Sheetfile" "pluviometro.kicad_sch"
-			(at 30.48 46.4316 0)
+			(at 119.38 70.5616 0)
 			(effects
 				(font
@@
 		)
 		(pin "RAIN_PULSE" output
-			(at 73.66 38.1 0)
+			(at 162.56 62.23 0)
 			(effects
 				(font
@@
 		)
 		(instances
-			(project "esquematico_V4"
+			(project "estacao-meteorologica"
 				(path "/0c305a6e-f9cd-49a1-b146-c2956e5469b6/058dce74-971b-49d7-82f0-384e20be985c"
 					(page "10")

Commit message: Padronizacao de nomes e numero de componentes
Other:
- sheet ANEMOMETRO renamed ANEMÔMETRO
- sheet PLUVIOMETRO renamed PLUVIÔMETRO
Changed lines of the file:
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@@
 			(color 0 0 0 0.0000)
 		)
-		(property "Sheetname" "ANEMOMETRO"
+		(property "Sheetname" "ANEMÔMETRO"
 			(at 119.38 83.1084 0)
 			(effects
@@
 			(color 0 0 0 0.0000)
 		)
-		(property "Sheetname" "PLUVIOMETRO"
+		(property "Sheetname" "PLUVIÔMETRO"
 			(at 119.38 53.8984 0)
 			(effects
