File: hardware/kicad/estacao-meteorologica/sheets/bmp280.kicad_sch (KiCad schematic)
At the start: 5 parts, among them U8 BMP280

Commit message: Padronizacao de nomes e numero de componentes
Parts:
- C211: renamed from C1; value 100n -> 100 nF; Assembly (none) -> SMT; LCSC Part C14663 -> (none); Modelo 3D ${KICAD9_3DMODEL_DIR}/Capacitor_SMD.3dshapes/C_0603_1608Met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 -> (none); Rating 100 nF; X7R; 50 V; 0603 -> (none); Specification (none) -> 100 nF; X7R; 50 V; 0603; Status_Ficha Conferido no catalogo em 2026-09-24; verificar estoque ao c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 -> (none); Verification (none) -> Conferido no catalogo em 2026-09-24; verificar estoque ao c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
- C212: renamed from C2; value 100n -> 100 nF; Assembly (none) -> SMT; LCSC Part C14663 -> (none); Modelo 3D ${KICAD9_3DMODEL_DIR}/Capacitor_SMD.3dshapes/C_0603_1608Met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 -> (none); Rating 100 nF; X7R; 50 V; 0603 -> (none); Specification (none) -> 100 nF; X7R; 50 V; 0603; Status_Ficha Conferido no catalogo em 2026-09-24; verificar estoque ao c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 -> (none); Verification (none) -> Conferido no catalogo em 2026-09-24; verificar estoque ao c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
- R211: renamed from R3; value 10k -> 10 kΩ; Assembly (none) -> SMT; LCSC Part C25804 -> (none); Modelo 3D ${KICAD9_3DMODEL_DIR}/Resistor_SMD.3dshapes/R_0603_1608Metr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 -> (none); Rating 10 kOhm; 1%; 0,1 W; 75 V; 0603 -> (none); Specification (none) -> 10 kOhm; 1%; 0,1 W; 75 V; 0603; Status_Ficha Conferido no catalogo em 2026-09-24; verificar estoque ao c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 -> (none); Verification (none) -> Conferido no catalogo em 2026-09-24; verificar estoque ao c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
- R212: renamed from R4; value 10k -> 10 kΩ; Assembly (none) -> SMT; LCSC Part C25804 -> (none); Modelo 3D ${KICAD9_3DMODEL_DIR}/Resistor_SMD.3dshapes/R_0603_1608Metr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 -> (none); Rating 10 kOhm; 1%; 0,1 W; 75 V; 0603 -> (none); Specification (none) -> 10 kOhm; 1%; 0,1 W; 75 V; 0603; Status_Ficha Conferido no catalogo em 2026-09-24; verificar estoque ao c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 -> (none); Verification (none) -> Conferido no catalogo em 2026-09-24; verificar estoque ao c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
- U211: renamed from U8; Assembly (none) -> SMT; LCSC Part C83291 -> (none); Modelo 3D ${KICAD9_3DMODEL_DIR}/Package_LGA.3dshapes/Bosch_LGA-8_2x2.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 -> (none); Rating 1,71 a 3,6 V; -40 a +85 °C; LGA-8 -> (none); Specification (none) -> 1,71 a 3,6 V; -40 a +85 °C; LGA-8; Status_Ficha Conferido no catalogo em 2026-09-24; verificar estoque ao c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 -> (none); Verification (none) -> Conferido no catalogo em 2026-09-24; verificar estoque ao c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
Changed lines of the file:
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@@
 		(dnp no)
 		(fields_autoplaced yes)
-		(property "Reference" "U8"
+		(property "Reference" "U211"
 			(at 140.97 114.3 90)
 			(effects
@@
 			)
 		)
-		(property "LCSC Part" "C83291"
-			(at 139.7 106.68 0)
-			(effects
-				(font
-					(size 1.27 1.27)
-				)
-				(hide yes)
-			)
-		)
-		(property "Rating" "1,71 a 3,6 V; -40 a +85 °C; LGA-8"
+		(property "Specification" "1,71 a 3,6 V; -40 a +85 °C; LGA-8"
 			(at 139.7 106.68 0)
 			(effects
@@
 			)
 		)
-		(property "Modelo 3D" "${KICAD9_3DMODEL_DIR}/Package_LGA.3dshapes/Bosch_LGA-8_2x2.5mm_P0.65mm_ClockwisePinNumbering.step"
+		(property "Verification" "Conferido no catalogo em 2026-09-24; verificar estoque ao comprar"
 			(at 139.7 106.68 0)
-			(effects
-				(font
-					(size 1.27 1.27)
-				)
-				(hide yes)
-			)
-		)
-		(property "Status_Ficha" "Conferido no catalogo em 2026-09-24; verificar estoque ao comprar"
-			(at 139.7 106.68 0)
-			(effects
-				(font
-					(size 1.27 1.27)
-				)
-				(hide yes)
-			)
-		)
-		(property "CREATOR" ""
-			(at 139.7 106.68 90)
-			(effects
-				(font
-					(size 1.27 1.27)
-				)
-				(hide yes)
-			)
-		)
-		(property "VERIFIER" ""
-			(at 139.7 106.68 90)
 			(effects
 				(font
@@
 			(project ""
 				(path "/0c305a6e-f9cd-49a1-b146-c2956e5469b6/0abc4084-0cd9-43a4-88f9-87e0e6566acc"
-					(reference "U8")
+					(reference "U211")
 					(unit 1)
 				)
+			)
+		)
+		(property "Assembly" "SMT"
+			(at 0 0 0)
+			(effects
+				(font (size 1.27 1.27))
+				(hide yes)
 			)
 		)
@@
 		(on_board yes)
 		(dnp no)
-		(property "Reference" "R4"
+		(property "Reference" "R212"
 			(at 127.508 88.646 90)
 			(effects
@@
 			)
 		)
-		(property "Value" "10k"
+		(property "Value" "10 kΩ"
 			(at 127.508 91.186 90)
 			(effects
@@
 			)
 		)
-		(property "LCSC Part" "C25804"
-			(at 130.81 93.98 0)
-			(effects
-				(font
-					(size 1.27 1.27)
-				)
-				(hide yes)
-			)
-		)
-		(property "Rating" "10 kOhm; 1%; 0,1 W; 75 V; 0603"
+		(property "Specification" "10 kOhm; 1%; 0,1 W; 75 V; 0603"
 			(at 130.81 93.98 0)
 			(effects
@@
 			)
 		)
-		(property "Modelo 3D" "${KICAD9_3DMODEL_DIR}/Resistor_SMD.3dshapes/R_0603_1608Metric.step"
+		(property "Verification" "Conferido no catalogo em 2026-09-24; verificar estoque ao comprar"
 			(at 130.81 93.98 0)
-			(effects
-				(font
-					(size 1.27 1.27)
-				)
-				(hide yes)
-			)
-		)
-		(property "Status_Ficha" "Conferido no catalogo em 2026-09-24; verificar estoque ao comprar"
-			(at 130.81 93.98 0)
-			(effects
-				(font
-					(size 1.27 1.27)
-				)
-				(hide yes)
-			)
-		)
-		(property "CREATOR" ""
-			(at 130.81 93.98 90)
-			(effects
-				(font
-					(size 1.27 1.27)
-				)
-				(hide yes)
-			)
-		)
-		(property "VERIFIER" ""
-			(at 130.81 93.98 90)
 			(effects
 				(font
@@
 			(project "esquematico_V4"
 				(path "/0c305a6e-f9cd-49a1-b146-c2956e5469b6/0abc4084-0cd9-43a4-88f9-87e0e6566acc"
-					(reference "R4")
+					(reference "R212")
 					(unit 1)
 				)
+			)
+		)
+		(property "Assembly" "SMT"
+			(at 0 0 0)
+			(effects
+				(font (size 1.27 1.27))
+				(hide yes)
 			)
 		)
@@
 		(dnp no)
 		(fields_autoplaced yes)
-		(property "Reference" "C2"
+		(property "Reference" "C212"
 			(at 166.37 113.0299 0)
 			(effects
@@
 			)
 		)
-		(property "Value" "100n"
+		(property "Value" "100 nF"
 			(at 166.37 115.5699 0)
 			(effects
@@
 			)
 		)
-		(property "LCSC Part" "C14663"
-			(at 162.56 114.3 0)
-			(effects
-				(font
-					(size 1.27 1.27)
-				)
-				(hide yes)
-			)
-		)
-		(property "Rating" "100 nF; X7R; 50 V; 0603"
+		(property "Specification" "100 nF; X7R; 50 V; 0603"
 			(at 162.56 114.3 0)
 			(effects
@@
 			)
 		)
-		(property "Modelo 3D" "${KICAD9_3DMODEL_DIR}/Capacitor_SMD.3dshapes/C_0603_1608Metric.step"
-			(at 162.56 114.3 0)
-			(effects
-				(font
-					(size 1.27 1.27)
-				)
-				(hide yes)
-			)
-		)
-		(property "Status_Ficha" "Conferido no catalogo em 2026-09-24; verificar estoque ao comprar"
-			(at 162.56 114.3 0)
-			(effects
-				(font
-					(size 1.27 1.27)
-				)
-				(hide yes)
-			)
-		)
-		(property "CREATOR" ""
-			(at 162.56 114.3 0)
-			(effects
-				(font
-					(size 1.27 1.27)
-				)
-				(hide yes)
-			)
-		)
-		(property "VERIFIER" ""
+		(property "Verification" "Conferido no catalogo em 2026-09-24; verificar estoque ao comprar"
 			(at 162.56 114.3 0)
 			(effects
@@
 			(project "esquematico_V4"
 				(path "/0c305a6e-f9cd-49a1-b146-c2956e5469b6/0abc4084-0cd9-43a4-88f9-87e0e6566acc"
-					(reference "C2")
+					(reference "C212")
 					(unit 1)
 				)
+			)
+		)
+		(property "Assembly" "SMT"
+			(at 0 0 0)
+			(effects
+				(font (size 1.27 1.27))
+				(hide yes)
 			)
 		)
@@
 		(on_board yes)
 		(dnp no)
-		(property "Reference" "C1"
+		(property "Reference" "C211"
 			(at 155.956 114.046 0)
 			(effects
@@
 			)
 		)
-		(property "Value" "100n"
+		(property "Value" "100 nF"
 			(at 155.194 117.094 0)
 			(effects
@@
 			)
 		)
-		(property "LCSC Part" "C14663"
-			(at 152.4 114.3 0)
-			(effects
-				(font
-					(size 1.27 1.27)
-				)
-				(hide yes)
-			)
-		)
-		(property "Rating" "100 nF; X7R; 50 V; 0603"
+		(property "Specification" "100 nF; X7R; 50 V; 0603"
 			(at 152.4 114.3 0)
 			(effects
@@
 			)
 		)
-		(property "Modelo 3D" "${KICAD9_3DMODEL_DIR}/Capacitor_SMD.3dshapes/C_0603_1608Metric.step"
-			(at 152.4 114.3 0)
-			(effects
-				(font
-					(size 1.27 1.27)
-				)
-				(hide yes)
-			)
-		)
-		(property "Status_Ficha" "Conferido no catalogo em 2026-09-24; verificar estoque ao comprar"
-			(at 152.4 114.3 0)
-			(effects
-				(font
-					(size 1.27 1.27)
-				)
-				(hide yes)
-			)
-		)
-		(property "CREATOR" ""
-			(at 152.4 114.3 0)
-			(effects
-				(font
-					(size 1.27 1.27)
-				)
-				(hide yes)
-			)
-		)
-		(property "VERIFIER" ""
+		(property "Verification" "Conferido no catalogo em 2026-09-24; verificar estoque ao comprar"
 			(at 152.4 114.3 0)
 			(effects
@@
 			(project ""
 				(path "/0c305a6e-f9cd-49a1-b146-c2956e5469b6/0abc4084-0cd9-43a4-88f9-87e0e6566acc"
-					(reference "C1")
+					(reference "C211")
 					(unit 1)
 				)
+			)
+		)
+		(property "Assembly" "SMT"
+			(at 0 0 0)
+			(effects
+				(font (size 1.27 1.27))
+				(hide yes)
 			)
 		)
@@
 		(on_board yes)
 		(dnp no)
-		(property "Reference" "R3"
+		(property "Reference" "R211"
 			(at 124.968 78.486 90)
 			(effects
@@
 			)
 		)
-		(property "Value" "10k"
+		(property "Value" "10 kΩ"
 			(at 124.968 81.026 90)
 			(effects
@@
 			)
 		)
-		(property "LCSC Part" "C25804"
-			(at 128.27 83.82 0)
-			(effects
-				(font
-					(size 1.27 1.27)
-				)
-				(hide yes)
-			)
-		)
-		(property "Rating" "10 kOhm; 1%; 0,1 W; 75 V; 0603"
+		(property "Specification" "10 kOhm; 1%; 0,1 W; 75 V; 0603"
 			(at 128.27 83.82 0)
 			(effects
@@
 			)
 		)
-		(property "Modelo 3D" "${KICAD9_3DMODEL_DIR}/Resistor_SMD.3dshapes/R_0603_1608Metric.step"
+		(property "Verification" "Conferido no catalogo em 2026-09-24; verificar estoque ao comprar"
 			(at 128.27 83.82 0)
-			(effects
-				(font
-					(size 1.27 1.27)
-				)
-				(hide yes)
-			)
-		)
-		(property "Status_Ficha" "Conferido no catalogo em 2026-09-24; verificar estoque ao comprar"
-			(at 128.27 83.82 0)
-			(effects
-				(font
-					(size 1.27 1.27)
-				)
-				(hide yes)
-			)
-		)
-		(property "CREATOR" ""
-			(at 128.27 83.82 90)
-			(effects
-				(font
-					(size 1.27 1.27)
-				)
-				(hide yes)
-			)
-		)
-		(property "VERIFIER" ""
-			(at 128.27 83.82 90)
 			(effects
 				(font
@@
 			(project "esquematico_V4"
 				(path "/0c305a6e-f9cd-49a1-b146-c2956e5469b6/0abc4084-0cd9-43a4-88f9-87e0e6566acc"
-					(reference "R3")
+					(reference "R211")
 					(unit 1)
 				)
 			)
 		)
+		(property "Assembly" "SMT"
+			(at 0 0 0)
+			(effects
+				(font (size 1.27 1.27))
+				(hide yes)
+			)
+		)

Commit message: Add test points necessarios para debug
Parts:
- added TP211: I2C1_SCL, TestPoint:TestPoint_Pad_D1.0mm, symbol Connector:TestPoint
- added TP212: I2C1_SDA, TestPoint:TestPoint_Pad_D1.0mm, symbol Connector:TestPoint
- added TP213: GND, TestPoint:TestPoint_Pad_D1.0mm, symbol Connector:TestPoint
Connections:
- net GND: now also TP213.1
- net I2C1_SCL: now also TP211.1
- net I2C1_SDA: now also TP212.1
