File: hardware/kicad/estacao-meteorologica/sheets/alimentacao.kicad_sch (KiCad schematic)
At the start: 30 parts, among them J60 P4 / DC-005-2.0, J61 J_PWR / JST-XH, Q60 DMP6023LE-13, U60 AP63205WU-7, U61 TLV62569DBVR

Commit message: refatoracao: atualizacoes de hardware e falta revisao LoRa
Parts:
- removed R61: 300k / 1%, Resistor_SMD:R_0603_1608Metric, symbol Device:R
- C67: value 10u / 25V -> 4.7u / 25V; Function Entrada local U61; alem dos capacitores da saida5V -> Entrada local de U61; manter junto aos pinos VIN/GND; LCSC C15850 -> C7307475; LCSC Part C15850 -> C7307475; MPN CL21A106KAYNNNE -> MSAST21GAB5475MTNA01; Manufacturer Samsung Electro-Mechanics -> Taiyo Yuden; Rating X5R; 10%; considerar perda por bias DC -> X5R; 4.7uF/25V; Ceff 3.7uF conforme WEBENCH
- C68: value 10u / 25V -> 10u / 6.3V; footprint Capacitor_SMD:C_0805_2012Metric -> Capacitor_SMD:C_0402_1005Metric; Function Saida3V3 local; mais30.5uF das folhas existentes =40.5uF no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 -> Saida local +3V3; 1 de 3 capacitores em paralelo; LCSC C15850 -> C469527; LCSC Part C15850 -> C469527; MPN CL21A106KAYNNNE -> GRJ155R60J106ME11D; Manufacturer Samsung Electro-Mechanics -> Murata Manufacturing; Rating X5R; 10%; considerar perda por bias DC -> X5R; 10uF/6.3V; 1 de 3, Ceff total 11uF conforme WEBENCH
- C69: value 22u / 25V -> 10u / 6.3V; footprint Capacitor_SMD:C_1206_3216Metric -> Capacitor_SMD:C_0402_1005Metric; Function DNP: reserva, nao montar sem rever estabilidade e capacitan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 -> Saida local +3V3; 1 de 3 capacitores em paralelo; LCSC C12891 -> C469527; LCSC Part C12891 -> C469527; MPN CL31A226KAHNNNE -> GRJ155R60J106ME11D; Manufacturer Samsung Electro-Mechanics -> Murata Manufacturing; Rating X5R; 10%; considerar perda por bias DC -> X5R; 10uF/6.3V; 1 de 3, Ceff total 11uF conforme WEBENCH; now fitted
- C70: value 6p8 / 50V -> 10u / 6.3V; footprint Capacitor_SMD:C_0603_1608Metric -> Capacitor_SMD:C_0402_1005Metric; Function Feed-forward em paralelo comR61+R62; resposta de transientes -> Saida local +3V3; 1 de 3 capacitores em paralelo; LCSC C1679 -> C469527; LCSC Part C1679 -> C469527; MPN 0603CG6R8C500NT -> GRJ155R60J106ME11D; Manufacturer FH (Guangdong Fenghua Advanced Tech) -> Murata Manufacturing; Rating C0G; +/-0.25pF; feed-forward -> X5R; 10uF/6.3V; 1 de 3, Ceff total 11uF conforme WEBENCH
- L61: value 2u2 / MWSA0402S -> 2u2 / ASPI-0530HI; footprint Inductor_SMD:L_Sunlord_MWSA0402S -> Hardware_Power:L_Abracon_ASPI-0530HI; Function 2.2uH blindado; LC aprovado pela matriz do datasheetTI -> Indutor blindado do WEBENCH; pad recomendado 7.0x3.0, pads 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; LCSC C408335 -> C7217567; LCSC Part C408335 -> C7217567; MPN MWSA0402S-2R2MT -> ASPI-0530HI-2R2M-T2; Manufacturer Sunlord -> Abracon Corporation; Rating Isat min4A/tip5A; Irms min3.8A; DCRmax58mOhm -> L=2.2uH +/-20%; DCRmax35mOhm; Isat9A; Irms5.5A
- R62: value 150k / 1% -> 453k / 1%; Function Serie com300k; resistoresBasic para reduzir taxa de montagem -> Braço superior do divisor de FB; Vout nominal 3.318V; LCSC C22807 -> C2079749; LCSC Part C22807 -> C2079749; MPN 0603WAF1503T5E -> CRCW0603453KFKEA; Manufacturer UNI-ROYAL(Uniroyal Elec) -> Vishay-Dale
- R63: footprint Resistor_SMD:R_0603_1608Metric -> Resistor_SMD:R_0402_1005Metric; Function Perna inferior do divisor; Vout0.6*(1+450k/100k)=3.3V -> Braço inferior do divisor de FB; Vout nominal 3.318V; LCSC C25803 -> C481918; LCSC Part C25803 -> C481918; MPN 0603WAF1003T5E -> CRCW0402100KFKED; Manufacturer UNI-ROYAL(Uniroyal Elec) -> Vishay-Dale; Rating 0.1W; 75V -> 0.063W; 50V
- U61: Function Buck5V->3V3; R61+R62=450k, R63=100k; EN sempre ligado -> Buck5V->3V3; R62=453k, R63=100k; EN sempre ligado
Connections:
- net +3V3: now also R62.1
- net FB_3V3: no longer C70.2
- net GND: now also C70.2
Other:
- note added: "WEBENCH U61: C67=4,7uF (Ceff 3,7uF); C68+C69+C70=11uF Ceff total. Alvo3V3 <=1A; validar carga/termica. Sem LED permanente. NAO unir +3V3 a fonte externa/USB sem analisar retorno."
- note removed: "C68=10uF +30,5uF existentes =40,5uF; C69 DNP. Alvo3V3 <=1A; validar carga/termica. Sem LED permanente. NAO unir3V3 ao regulador3V3 da Nucleo; evitar retorno porUSB."
- moved on the sheet: C64, C68

Commit message: refatoracao: lora + Verificacao projeto inteiro
Parts:
- C60: Modelo 3D (none) -> ${KICAD9_3DMODEL_DIR}/Capacitor_SMD.3dshapes/CP_Elec_6.3x5.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; Status_Ficha (none) -> Conferido no catalogo em 2026-09-24; verificar estoque ao c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
- C61, C62, C65, C66: Modelo 3D (none) -> ${KICAD9_3DMODEL_DIR}/Capacitor_SMD.3dshapes/C_1206_3216Met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; Status_Ficha (none) -> Conferido no catalogo em 2026-09-24; verificar estoque ao c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
- C63, C64: Modelo 3D (none) -> ${KICAD9_3DMODEL_DIR}/Capacitor_SMD.3dshapes/C_0603_1608Met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; Status_Ficha (none) -> Conferido no catalogo em 2026-09-24; verificar estoque ao c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
- C67: Modelo 3D (none) -> ${KICAD9_3DMODEL_DIR}/Capacitor_SMD.3dshapes/C_0805_2012Met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; Status_Ficha (none) -> Conferido no catalogo em 2026-09-24; verificar estoque ao c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
- C68, C69, C70: Manufacturer Murata Manufacturing -> Murata Electronics; Modelo 3D (none) -> ${KICAD9_3DMODEL_DIR}/Capacitor_SMD.3dshapes/C_0402_1005Met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; Status_Ficha (none) -> Conferido no catalogo em 2026-09-24; verificar estoque ao c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
- D60: Modelo 3D (none) -> ${KICAD9_3DMODEL_DIR}/Diode_SMD.3dshapes/D_SMB.step; Status_Ficha (none) -> Conferido no catalogo em 2026-09-24; verificar estoque ao c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
- D61: Modelo 3D (none) -> ${KICAD9_3DMODEL_DIR}/Diode_SMD.3dshapes/D_SOD-123.step; Status_Ficha (none) -> Conferido no catalogo em 2026-09-24; verificar estoque ao c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
- F60: Modelo 3D (none) -> ${KICAD9_3DMODEL_DIR}/Fuse.3dshapes/Fuse_1206_3216Metric.st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; Status_Ficha (none) -> Conferido no catalogo em 2026-09-24; verificar estoque ao c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
- J60, Q60: Modelo 3D (none) -> ${KIPRJMOD}/../../libraries/Hardware_Power/Hardware_Power.3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; Status_Ficha (none) -> Conferido no catalogo em 2026-09-24; verificar estoque ao c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
- J61: Modelo 3D (none) -> ${KICAD9_3DMODEL_DIR}/Connector_JST.3dshapes/JST_XH_B2B-XH-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; Status_Ficha (none) -> Conferido no catalogo em 2026-09-24; verificar estoque ao c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
- JP60, TP60, TP61, TP62, TP63: LCSC (none) -> N/A; LCSC Part (none) -> N/A; MPN (none) -> N/A - elemento de cobre da PCB; Manufacturer (none) -> N/A; Modelo 3D (none) -> N/A - geometria de cobre, sem corpo
- L60: Modelo 3D (none) -> ${KICAD9_3DMODEL_DIR}/Inductor_SMD.3dshapes/L_Sunlord_MWSA0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; Status_Ficha (none) -> Conferido no catalogo em 2026-09-24; verificar estoque ao c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
- L61: Manufacturer Abracon Corporation -> Abracon LLC; Modelo 3D (none) -> ${KIPRJMOD}/../../libraries/Hardware_Power/Hardware_Power.3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; Status_Ficha (none) -> Conferido no catalogo em 2026-09-24; verificar estoque ao c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
- R60: Modelo 3D (none) -> ${KICAD9_3DMODEL_DIR}/Resistor_SMD.3dshapes/R_0603_1608Metr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; Status_Ficha (none) -> Conferido no catalogo em 2026-09-24; verificar estoque ao c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
- R62: Manufacturer Vishay-Dale -> Vishay Intertech; Modelo 3D (none) -> ${KICAD9_3DMODEL_DIR}/Resistor_SMD.3dshapes/R_0603_1608Metr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; Status_Ficha (none) -> Conferido no catalogo em 2026-09-24; verificar estoque ao c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
- R63: Manufacturer Vishay-Dale -> Vishay Intertech; Modelo 3D (none) -> ${KICAD9_3DMODEL_DIR}/Resistor_SMD.3dshapes/R_0402_1005Metr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; Status_Ficha (none) -> Conferido no catalogo em 2026-09-24; verificar estoque ao c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
- U60: Modelo 3D (none) -> ${KICAD9_3DMODEL_DIR}/Package_TO_SOT_SMD.3dshapes/TSOT-23-6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; Status_Ficha (none) -> Conferido no catalogo em 2026-09-24; verificar estoque ao c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
- U61: Modelo 3D (none) -> ${KICAD9_3DMODEL_DIR}/Package_TO_SOT_SMD.3dshapes/SOT-23-5.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; Status_Ficha (none) -> Conferido no catalogo em 2026-09-24; verificar estoque ao c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

Commit message: Padronizacao de nomes e numero de componentes
Parts:
- C601: renamed from C60; value 47u / 35V -> 47 µF, 35 V; Assembly (none) -> SMT; LCSC Part C87068 -> (none); Modelo 3D ${KICAD9_3DMODEL_DIR}/Capacitor_SMD.3dshapes/CP_Elec_6.3x5.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 -> (none); Rating 20%; -55..105C; 1000h@105C; bulk de cabo, nao substitui MLCC -> (none); Specification (none) -> 20%; -55..105C; 1000h@105C; bulk de cabo, nao substitui MLCC; Status_Ficha Conferido no catalogo em 2026-09-24; verificar estoque ao c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 -> (none); Verification (none) -> Conferido no catalogo em 2026-09-24; verificar estoque ao c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
- C602: renamed from C61; value 10u / 50V -> 10 µF, 50 V; Assembly (none) -> SMT; LCSC Part C13585 -> (none); Modelo 3D ${KICAD9_3DMODEL_DIR}/Capacitor_SMD.3dshapes/C_1206_3216Met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 -> (none); Rating X5R; 10%; considerar perda por bias DC -> (none); Specification (none) -> X5R; 10%; considerar perda por bias DC; Status_Ficha Conferido no catalogo em 2026-09-24; verificar estoque ao c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 -> (none); Verification (none) -> Conferido no catalogo em 2026-09-24; verificar estoque ao c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
- C603: renamed from C62; value 10u / 50V -> 10 µF, 50 V; Assembly (none) -> SMT; LCSC Part C13585 -> (none); Modelo 3D ${KICAD9_3DMODEL_DIR}/Capacitor_SMD.3dshapes/C_1206_3216Met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 -> (none); Rating X5R; 10%; considerar perda por bias DC -> (none); Specification (none) -> X5R; 10%; considerar perda por bias DC; Status_Ficha Conferido no catalogo em 2026-09-24; verificar estoque ao c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 -> (none); Verification (none) -> Conferido no catalogo em 2026-09-24; verificar estoque ao c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
- C604: renamed from C63; Assembly (none) -> SMT; LCSC Part C14663 -> (none); Modelo 3D ${KICAD9_3DMODEL_DIR}/Capacitor_SMD.3dshapes/C_0603_1608Met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 -> (none); Rating X7R; 10% -> (none); Specification (none) -> X7R; 10%; Status_Ficha Conferido no catalogo em 2026-09-24; verificar estoque ao c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 -> (none); Verification (none) -> Conferido no catalogo em 2026-09-24; verificar estoque ao c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
- C605: renamed from C64; Assembly (none) -> SMT; LCSC Part C14663 -> (none); Modelo 3D ${KICAD9_3DMODEL_DIR}/Capacitor_SMD.3dshapes/C_0603_1608Met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 -> (none); Rating X7R; 10% -> (none); Specification (none) -> X7R; 10%; Status_Ficha Conferido no catalogo em 2026-09-24; verificar estoque ao c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 -> (none); Verification (none) -> Conferido no catalogo em 2026-09-24; verificar estoque ao c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
- C606: renamed from C65; value 22u / 25V -> 22 µF, 25 V; Assembly (none) -> SMT; LCSC Part C12891 -> (none); Modelo 3D ${KICAD9_3DMODEL_DIR}/Capacitor_SMD.3dshapes/C_1206_3216Met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 -> (none); Rating X5R; 10%; considerar perda por bias DC -> (none); Specification (none) -> X5R; 10%; considerar perda por bias DC; Status_Ficha Conferido no catalogo em 2026-09-24; verificar estoque ao c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 -> (none); Verification (none) -> Conferido no catalogo em 2026-09-24; verificar estoque ao c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
- C607: renamed from C66; value 22u / 25V -> 22 µF, 25 V; Assembly (none) -> SMT; LCSC Part C12891 -> (none); Modelo 3D ${KICAD9_3DMODEL_DIR}/Capacitor_SMD.3dshapes/C_1206_3216Met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 -> (none); Rating X5R; 10%; considerar perda por bias DC -> (none); Specification (none) -> X5R; 10%; considerar perda por bias DC; Status_Ficha Conferido no catalogo em 2026-09-24; verificar estoque ao c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 -> (none); Verification (none) -> Conferido no catalogo em 2026-09-24; verificar estoque ao c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
- C608: renamed from C67; value 4.7u / 25V -> 4.7 µF, 25 V; Assembly (none) -> SMT; LCSC Part C7307475 -> (none); Modelo 3D ${KICAD9_3DMODEL_DIR}/Capacitor_SMD.3dshapes/C_0805_2012Met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 -> (none); Rating X5R; 4.7uF/25V; Ceff 3.7uF conforme WEBENCH -> (none); Specification (none) -> X5R; 4.7uF/25V; Ceff 3.7uF conforme WEBENCH; Status_Ficha Conferido no catalogo em 2026-09-24; verificar estoque ao c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 -> (none); Verification (none) -> Conferido no catalogo em 2026-09-24; verificar estoque ao c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
- C609: renamed from C68; value 10u / 6.3V -> 10 µF, 6.3 V; Assembly (none) -> SMT; LCSC Part C469527 -> (none); Modelo 3D ${KICAD9_3DMODEL_DIR}/Capacitor_SMD.3dshapes/C_0402_1005Met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 -> (none); Rating X5R; 10uF/6.3V; 1 de 3, Ceff total 11uF conforme WEBENCH -> (none); Specification (none) -> X5R; 10uF/6.3V; 1 de 3, Ceff total 11uF conforme WEBENCH; Status_Ficha Conferido no catalogo em 2026-09-24; verificar estoque ao c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 -> (none); Verification (none) -> Conferido no catalogo em 2026-09-24; verificar estoque ao c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
- C610: renamed from C69; value 10u / 6.3V -> 10 µF, 6.3 V; Assembly (none) -> SMT; LCSC Part C469527 -> (none); Modelo 3D ${KICAD9_3DMODEL_DIR}/Capacitor_SMD.3dshapes/C_0402_1005Met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 -> (none); Rating X5R; 10uF/6.3V; 1 de 3, Ceff total 11uF conforme WEBENCH -> (none); Specification (none) -> X5R; 10uF/6.3V; 1 de 3, Ceff total 11uF conforme WEBENCH; Status_Ficha Conferido no catalogo em 2026-09-24; verificar estoque ao c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 -> (none); Verification (none) -> Conferido no catalogo em 2026-09-24; verificar estoque ao c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
- C611: renamed from C70; value 10u / 6.3V -> 10 µF, 6.3 V; Assembly (none) -> SMT; LCSC Part C469527 -> (none); Modelo 3D ${KICAD9_3DMODEL_DIR}/Capacitor_SMD.3dshapes/C_0402_1005Met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 -> (none); Rating X5R; 10uF/6.3V; 1 de 3, Ceff total 11uF conforme WEBENCH -> (none); Specification (none) -> X5R; 10uF/6.3V; 1 de 3, Ceff total 11uF conforme WEBENCH; Status_Ficha Conferido no catalogo em 2026-09-24; verificar estoque ao c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 -> (none); Verification (none) -> Conferido no catalogo em 2026-09-24; verificar estoque ao c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
- D601: renamed from D60; Assembly (none) -> SMT; LCSC Part C3001977 -> (none); Modelo 3D ${KICAD9_3DMODEL_DIR}/Diode_SMD.3dshapes/D_SMB.step -> (none); Rating Bidirecional; VRWM16V; VC26V a23.1A; 600W 10/1000us -> (none); Specification (none) -> Bidirecional; VRWM16V; VC26V a23.1A; 600W 10/1000us; Status_Ficha Conferido no catalogo em 2026-09-24; verificar estoque ao c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 -> (none); Verification (none) -> Conferido no catalogo em 2026-09-24; verificar estoque ao c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
- D602: renamed from D61; Assembly (none) -> SMT; LCSC Part C19077408 -> (none); Modelo 3D ${KICAD9_3DMODEL_DIR}/Diode_SMD.3dshapes/D_SOD-123.step -> (none); Rating 350mW; VZ9.5-10.5V @5mA; K=source, A=gate -> (none); Specification (none) -> 350mW; VZ9.5-10.5V @5mA; K=source, A=gate; Status_Ficha Conferido no catalogo em 2026-09-24; verificar estoque ao c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 -> (none); Verification (none) -> Conferido no catalogo em 2026-09-24; verificar estoque ao c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
- F601: renamed from F60; value 1.5A / 32V lento -> 1.5 A, 32 V, slow-blow; Assembly (none) -> SMT; LCSC Part C553929 -> (none); Modelo 3D ${KICAD9_3DMODEL_DIR}/Fuse.3dshapes/Fuse_1206_3216Metric.st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 -> (none); Rating I2t tip 0.4137 A2s; interrupcao 50A; DCR tip 140mOhm -> (none); Specification (none) -> I2t tip 0.4137 A2s; interrupcao 50A; DCR tip 140mOhm; Status_Ficha Conferido no catalogo em 2026-09-24; verificar estoque ao c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 -> (none); Verification (none) -> Conferido no catalogo em 2026-09-24; verificar estoque ao c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
- J601: renamed from J60; value P4 / DC-005-2.0 -> DC jack, 2.0 mm; Assembly (none) -> THT — montagem manual; LCSC Part C22459640 -> (none); Modelo 3D ${KIPRJMOD}/../../libraries/Hardware_Power/Hardware_Power.3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 -> (none); Rating 20V; 3A; centro positivo; confirmar plugue 5.5/2.1 -> (none); Specification (none) -> 20V; 3A; centro positivo; confirmar plugue 5.5/2.1; Status_Ficha Conferido no catalogo em 2026-09-24; verificar estoque ao c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 -> (none); Verification (none) -> Conferido no catalogo em 2026-09-24; verificar estoque ao c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
- J602: renamed from J61; value J_PWR / JST-XH -> JST-XH, 1x02, P2.50 mm; Assembly (none) -> THT — montagem manual; LCSC Part C158012 -> (none); Modelo 3D ${KICAD9_3DMODEL_DIR}/Connector_JST.3dshapes/JST_XH_B2B-XH-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 -> (none); Rating 3A; 250V; passo 2.50mm; p1 positivo, p2 GND -> (none); Specification (none) -> 3A; 250V; passo 2.50mm; p1 positivo, p2 GND; Status_Ficha Conferido no catalogo em 2026-09-24; verificar estoque ao c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 -> (none); Verification (none) -> Conferido no catalogo em 2026-09-24; verificar estoque ao c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
- JP601: renamed from JP60; value SEL_FONTE -> Solder jumper, 3 pads; Assembly (none) -> SMT; LCSC Part N/A -> (none); Modelo 3D N/A - geometria de cobre, sem corpo -> (none); Rating Pad de cobre; fechar apenas 1-2 OU 2-3 -> (none); Specification (none) -> Pad de cobre; fechar apenas 1-2 OU 2-3
- L601: renamed from L60; value 4u7 / MWSA0603S -> 4.7 µH; Assembly (none) -> SMT; LCSC Part C408447 -> (none); Modelo 3D ${KICAD9_3DMODEL_DIR}/Inductor_SMD.3dshapes/L_Sunlord_MWSA0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 -> (none); Rating Isat min7.2A/tip9A; Irms min5A; DCRmax33mOhm -> (none); Specification (none) -> Isat min7.2A/tip9A; Irms min5A; DCRmax33mOhm; Status_Ficha Conferido no catalogo em 2026-09-24; verificar estoque ao c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 -> (none); Verification (none) -> Conferido no catalogo em 2026-09-24; verificar estoque ao c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
- L602: renamed from L61; value 2u2 / ASPI-0530HI -> 2.2 µH; Assembly (none) -> SMT; LCSC Part C7217567 -> (none); Modelo 3D ${KIPRJMOD}/../../libraries/Hardware_Power/Hardware_Power.3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 -> (none); Rating L=2.2uH +/-20%; DCRmax35mOhm; Isat9A; Irms5.5A -> (none); Specification (none) -> L=2.2uH +/-20%; DCRmax35mOhm; Isat9A; Irms5.5A; Status_Ficha Conferido no catalogo em 2026-09-24; verificar estoque ao c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 -> (none); Verification (none) -> Conferido no catalogo em 2026-09-24; verificar estoque ao c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
- Q601: renamed from Q60; Assembly (none) -> SMT; LCSC Part C154901 -> (none); Modelo 3D ${KIPRJMOD}/../../libraries/Hardware_Power/Hardware_Power.3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 -> (none); Rating PMOS60V; VGS +/-20V; 28mOhm max @-10V; 1G 2D 3S 4D -> (none); Specification (none) -> PMOS60V; VGS +/-20V; 28mOhm max @-10V; 1G 2D 3S 4D; Status_Ficha Conferido no catalogo em 2026-09-24; verificar estoque ao c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 -> (none); Verification (none) -> Conferido no catalogo em 2026-09-24; verificar estoque ao c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
- R601: renamed from R60; value 100k / 1% -> 100 kΩ, 1 %; Assembly (none) -> SMT; LCSC Part C25803 -> (none); Modelo 3D ${KICAD9_3DMODEL_DIR}/Resistor_SMD.3dshapes/R_0603_1608Metr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 -> (none); Rating 0.1W; 75V -> (none); Specification (none) -> 0.1W; 75V; Status_Ficha Conferido no catalogo em 2026-09-24; verificar estoque ao c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 -> (none); Verification (none) -> Conferido no catalogo em 2026-09-24; verificar estoque ao c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
- R602: renamed from R62; value 453k / 1% -> 453 kΩ, 1 %; Assembly (none) -> SMT; LCSC Part C2079749 -> (none); Modelo 3D ${KICAD9_3DMODEL_DIR}/Resistor_SMD.3dshapes/R_0603_1608Metr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 -> (none); Rating 0.1W; 75V -> (none); Specification (none) -> 0.1W; 75V; Status_Ficha Conferido no catalogo em 2026-09-24; verificar estoque ao c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 -> (none); Verification (none) -> Conferido no catalogo em 2026-09-24; verificar estoque ao c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
- R603: renamed from R63; value 100k / 1% -> 100 kΩ, 1 %; Assembly (none) -> SMT; LCSC Part C481918 -> (none); Modelo 3D ${KICAD9_3DMODEL_DIR}/Resistor_SMD.3dshapes/R_0402_1005Metr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 -> (none); Rating 0.063W; 50V -> (none); Specification (none) -> 0.063W; 50V; Status_Ficha Conferido no catalogo em 2026-09-24; verificar estoque ao c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 -> (none); Verification (none) -> Conferido no catalogo em 2026-09-24; verificar estoque ao c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
- TP601: renamed from TP60; Assembly (none) -> PCB — sem compra; LCSC Part N/A -> (none); Modelo 3D N/A - geometria de cobre, sem corpo -> (none); Rating Cobre exposto; nao comprar -> (none); Specification (none) -> Cobre exposto; nao comprar
- TP602: renamed from TP61; Assembly (none) -> PCB — sem compra; LCSC Part N/A -> (none); Modelo 3D N/A - geometria de cobre, sem corpo -> (none); Rating Cobre exposto; nao comprar -> (none); Specification (none) -> Cobre exposto; nao comprar
- TP603: renamed from TP62; Assembly (none) -> PCB — sem compra; LCSC Part N/A -> (none); Modelo 3D N/A - geometria de cobre, sem corpo -> (none); Rating Cobre exposto; nao comprar -> (none); Specification (none) -> Cobre exposto; nao comprar
- TP604: renamed from TP63; Assembly (none) -> PCB — sem compra; LCSC Part N/A -> (none); Modelo 3D N/A - geometria de cobre, sem corpo -> (none); Rating Cobre exposto; nao comprar -> (none); Specification (none) -> Cobre exposto; nao comprar
- U601: renamed from U60; Assembly (none) -> SMT; LCSC Part C2071056 -> (none); Modelo 3D ${KICAD9_3DMODEL_DIR}/Package_TO_SOT_SMD.3dshapes/TSOT-23-6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 -> (none); Rating 5V fixos; 2A CI; VIN3.8-32V; 1.1MHz; IQtip22uA -> (none); Specification (none) -> 5V fixos; 2A CI; VIN3.8-32V; 1.1MHz; IQtip22uA; Status_Ficha Conferido no catalogo em 2026-09-24; verificar estoque ao c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 -> (none); Verification (none) -> Conferido no catalogo em 2026-09-24; verificar estoque ao c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
- U602: renamed from U61; Assembly (none) -> SMT; LCSC Part C141836 -> (none); Modelo 3D ${KICAD9_3DMODEL_DIR}/Package_TO_SOT_SMD.3dshapes/SOT-23-5.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 -> (none); Rating 2A CI; VIN2.5-5.5V; 1.5MHz; IQtip35uA; sem PG -> (none); Specification (none) -> 2A CI; VIN2.5-5.5V; 1.5MHz; IQtip35uA; sem PG; Status_Ficha Conferido no catalogo em 2026-09-24; verificar estoque ao c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 -> (none); Verification (none) -> Conferido no catalogo em 2026-09-24; verificar estoque ao c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
Connections:
- net ENERGIA_POS renamed VIN_EXTERNAL
- net P4_POS renamed VIN_JACK

Commit message: Refact: tirei estagio de 12V -> 5V e agora é direto 12V -> 3V
Parts:
- removed C608: 4.7 µF, 25 V, Capacitor_SMD:C_0805_2012Metric, symbol Device:C
- removed C609, C610, C611: 10 µF, 6.3 V, Capacitor_SMD:C_0402_1005Metric, symbol Device:C
- removed L602: 2.2 µH, Hardware_Power:L_Abracon_ASPI-0530HI, symbol Device:L
- removed R602: 453 kΩ, 1 %, Resistor_SMD:R_0603_1608Metric, symbol Device:R
- removed R603: 100 kΩ, 1 %, Resistor_SMD:R_0402_1005Metric, symbol Device:R
- removed TP602: +5V, TestPoint:TestPoint_Pad_D1.5mm, symbol Connector:TestPoint
- removed U602: TLV62569DBVR, Package_TO_SOT_SMD:SOT-23-5, symbol Regulator_Switching:TLV62569DBV
- C602: Function MLCC de entrada do AP63205; junto ao VIN/GND -> MLCC de entrada do AP63203; junto ao VIN/GND
- C606: Function Saida5V; 22uF25V em paralelo comC66 -> Saida +3V3; capacitor principal apos L601
- C607: Function Saida5V; Ctotal44uFnominal -> Saida +3V3; Ctotal 44uF nominal; capacitor principal apos L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
- L601: value 4.7 µH -> 3.9 µH; footprint Inductor_SMD:L_Sunlord_MWSA0603S -> Inductor_SMD:L_APV_ANR5040; LCSC C408447 -> C7427132; MPN MWSA0603S-4R7MT -> ANR5040T3R9M; Manufacturer Sunlord -> APV; Specification Isat min7.2A/tip9A; Irms min5A; DCRmax33mOhm -> L=3,9uH ±20%; Irms 3,7A; Isat 4,2A; indutor blindado; corpo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; Verification Conferido no catalogo em 2026-09-24; verificar estoque ao c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 -> Ficha do fabricante e catalogo LCSC conferidos em 2026-09-2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
- U601: value AP63205WU-7 -> AP63203WU-7; symbol Regulator_Switching:AP63205WU -> Regulator_Switching:AP63203WU; Function Converte VIN_MAIN para5V; EN ligado aVIN; FB direto na said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 -> Converte VIN_MAIN diretamente para +3V3; EN ligado a VIN; F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; LCSC C2071056 -> C780769; MPN AP63205WU-7 -> AP63203WU-7; Specification 5V fixos; 2A CI; VIN3.8-32V; 1.1MHz; IQtip22uA -> 3,3V fixos; 2A CI; VIN3,8-32V; 1,1MHz; IQ tipico 22uA; Verification Conferido no catalogo em 2026-09-24; verificar estoque ao c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 -> Ficha do fabricante e catalogo LCSC conferidos em 2026-09-2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
Connections:
- net +5V is gone; now on net +3V3: C606.1, C607.1, L601.2, U601.1 (FB)
Other:
- note added: "AP63203: VIN3,8-32V -> +3V3 fixos; CI ate 2A, validar limite termico da placa. C606+C607 sao os capacitores principais da saida; usar capacitancia efetiva, nao apenas nominal. NAO unir +3V3 a fonte externa/USB sem analisar retorno."
- note added: "BUCK UNICO 3V3 | CI 2 A / VALIDAR TERMICA"
- note added: "FB: medir apos L601"
- note added: "L601=3,9uH; C606+C607=44uF nominais na saida +3V3; FB ligado APOS L601. Cin e Cboot fisicamente junto a U601; manter a malha VIN-CIN-GND curta. Alvo inicial: +3V3 <=1A; validar ripple, partida e termica."
- note added: "REFERENCIAS: Diodes AP63203 DS41326 — configuracao tipica de 3,3V e layout recomendado. LAYOUT: malhas VIN-CIN-GND curtas; SW minimo; FB longe de SW; plano GND continuo. Decisao/BOM/LCSC e limites: docs/engineering/hardware/Desenvolvimento/ESTUDO_ALIMENTACAO_12V_PARA_3V3_SEM_ESTAGIO_5V.md"
- note removed: "2 BUCK 5 V | CI 2 A / VALIDAR TERMICA"
- note removed: "FB: medir apos L60"
- note removed: "L60=4,7uH; C65+C66=44uF nominais; FB ligado APOS L60. C61/C62/C63 fisicamente junto a U60, apesar de desenhados acima. Alvo inicial: 5V externo <=0,5A + carga do buck3V3; validar termica."
- note removed: "REFERENCIAS: Diodes AP63205 DS41326 Fig.21/Tab.3; TI TLV62569 SLVSDG1C sec.8.2/10. LAYOUT: malhas VIN-CIN-GND curtas; SW minimo; FB longe deSW; planoGND continuo. Detalhes, BOM/LCSC e limites: docs/alimentacao/README.md"
- note removed: "WEBENCH U61: C67=4,7uF (Ceff 3,7uF); C68+C69+C70=11uF Ceff total. Alvo3V3 <=1A; validar carga/termica. Sem LED permanente. NAO unir +3V3 a fonte externa/USB sem analisar retorno."
- moved on the sheet: TP603, TP604

Commit message: rotemento 3.0
Connections:
- net V_SW: now reaches C605.2, L601.1, U601.5 (SW)
Other:
- note removed: "3 BUCK 3,3 V | SEM MCU PARA PARTIDA"

Commit message: feat(hardware): consolida revisão PCB V2
Parts:
- TP601, TP603, TP604: footprint TestPoint:TestPoint_Pad_D1.5mm -> TestPoint:TestPoint_Pad_D1.0mm
Changed lines of the file:
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@@
 			)
 		)
-		(property "Footprint" "TestPoint:TestPoint_Pad_D1.5mm"
+		(property "Footprint" "TestPoint:TestPoint_Pad_D1.0mm"
 			(at 195.58 160.02 0)
 			(effects
@@
 			)
 		)
-		(property "Footprint" "TestPoint:TestPoint_Pad_D1.5mm"
+		(property "Footprint" "TestPoint:TestPoint_Pad_D1.0mm"
 			(at 195.58 220.98 0)
 			(effects
@@
 			)
 		)
-		(property "Footprint" "TestPoint:TestPoint_Pad_D1.5mm"
+		(property "Footprint" "TestPoint:TestPoint_Pad_D1.0mm"
 			(at 355.6 59.69 0)
 			(effects
