File: hardware/kicad/estacao-meteorologica/sheets/bh1750_interface.kicad_sch (KiCad schematic)
At the start: 3 parts, among them J221 JST-XH, 1x04, P2.50 mm

Commit message: Add test points necessarios para debug
Parts:
- added TP221: BH_I2C3_SCL, TestPoint:TestPoint_Pad_D1.0mm, symbol Connector:TestPoint
- added TP222: BH_I2C3_SDA, TestPoint:TestPoint_Pad_D1.0mm, symbol Connector:TestPoint
- added TP223: GND, TestPoint:TestPoint_Pad_D1.0mm, symbol Connector:TestPoint
Connections:
- net BH_I2C3_SCL: now also TP221.1
- net BH_I2C3_SDA: now also TP222.1
- net GND: now also TP223.1; no longer D222.1 (A1)

Commit message: rotemento 3.0
Connections:
- net +3V3: no longer J221.2 (Pin_2)
- net BH_I2C3_SDA: now also J221.2 (Pin_2); no longer J221.4 (Pin_4)
- net GND: now also D222.1 (A1)
Other:
- moved on the sheet: TP222
Changed lines of the file:
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@@
 	(paper "A4")
+	(junction
+		(at 100.33 72.39)
+		(diameter 0)
+		(color 0 0 0 0)
+	)
 	(junction
 		(at 115.57 74.93)
@@
 	)
 	(junction
-		(at 100.33 77.47)
+		(at 113.03 72.39)
 		(diameter 0)
 		(color 0 0 0 0)
 	)
-	(junction
-		(at 115.57 77.47)
-		(diameter 0)
-		(color 0 0 0 0)
+	(wire
+		(pts
+			(xy 113.03 62.23) (xy 113.03 72.39)
+		)
+		(stroke
+			(width 0)
+			(type default)
+		)
 	)
 	(wire
@@
 	(wire
 		(pts
-			(xy 115.57 77.47) (xy 115.57 82.55)
+			(xy 100.33 82.55) (xy 100.33 72.39)
 		)
 		(stroke
@@
 	(wire
 		(pts
-			(xy 100.33 77.47) (xy 93.98 77.47)
-		)
-		(stroke
-			(width 0)
-			(type default)
-		)
-	)
-	(wire
-		(pts
-			(xy 100.33 77.47) (xy 100.33 82.55)
-		)
-		(stroke
-			(width 0)
-			(type default)
-		)
-	)
-	(wire
-		(pts
 			(xy 105.41 59.69) (xy 105.41 62.23)
 		)
@@
 	(wire
 		(pts
-			(xy 99.06 72.39) (xy 93.98 72.39)
+			(xy 93.98 72.39) (xy 100.33 72.39)
 		)
 		(stroke
@@
 	(wire
 		(pts
-			(xy 121.92 77.47) (xy 115.57 77.47)
-		)
-		(stroke
-			(width 0)
-			(type default)
-		)
-	)
-	(wire
-		(pts
-			(xy 119.38 82.55) (xy 115.57 82.55)
-		)
-		(stroke
-			(width 0)
-			(type default)
-		)
-	)
-	(wire
-		(pts
-			(xy 115.57 77.47) (xy 100.33 77.47)
+			(xy 100.33 72.39) (xy 113.03 72.39)
+		)
+		(stroke
+			(width 0)
+			(type default)
+		)
+	)
+	(wire
+		(pts
+			(xy 113.03 72.39) (xy 121.92 72.39)
+		)
+		(stroke
+			(width 0)
+			(type default)
+		)
+	)
+	(wire
+		(pts
+			(xy 93.98 77.47) (xy 121.92 77.47)
 		)
 		(stroke
@@
 	(hierarchical_label "BH_I2C3_SDA"
 		(shape passive)
-		(at 121.92 77.47 0)
+		(at 121.92 72.39 0)
 		(effects
 			(font
@@
 	(symbol
 		(lib_id "Connector:TestPoint")
-		(at 119.38 82.55 270)
+		(at 113.03 62.23 0)
 		(unit 1)
 		(exclude_from_sim no)
@@
 		(dnp no)
 		(property "Reference" "TP222"
-			(at 128.778 81.534 90)
+			(at 112.014 52.832 90)
 			(effects
 				(font
@@
 		)
 		(property "Value" "BH_I2C3_SDA"
-			(at 128.778 84.074 90)
+			(at 114.554 52.832 90)
 			(effects
 				(font
@@
 		)
 		(property "Footprint" "TestPoint:TestPoint_Pad_D1.0mm"
-			(at 119.38 82.55 0)
+			(at 113.03 62.23 0)
 			(effects
 				(font
@@
 		)
 		(property "Datasheet" "N/A - geometria definida no footprint"
-			(at 119.38 82.55 0)
+			(at 113.03 62.23 0)
 			(effects
 				(font
@@
 		)
 		(property "Description" "Ponto de teste em cobre, pad circular de 1,0 mm; rede BH_I2C3_SDA"
-			(at 119.38 82.55 0)
+			(at 113.03 62.23 0)
 			(effects
 				(font
@@
 		)
 		(property "Manufacturer" "N/A"
-			(at 119.38 82.55 0)
+			(at 113.03 62.23 0)
 			(effects
 				(font
@@
 		)
 		(property "MPN" "N/A - elemento de cobre da PCB"
-			(at 119.38 82.55 0)
+			(at 113.03 62.23 0)
 			(effects
 				(font
@@
 		)
 		(property "LCSC" "N/A"
-			(at 119.38 82.55 0)
+			(at 113.03 62.23 0)
 			(effects
 				(font
@@
 		)
 		(property "Specification" "Copper pad; no purchased component"
-			(at 119.38 82.55 0)
+			(at 113.03 62.23 0)
 			(effects
 				(font
@@
 		)
 		(property "Function" "Ponto de teste do sinal BH_I2C3_SDA"
-			(at 119.38 82.55 0)
+			(at 113.03 62.23 0)
 			(effects
 				(font
@@
 		)
 		(property "Assembly" "PCB — sem compra"
-			(at 196.85 -33.02 0)
+			(at -2.54 -15.24 0)
 			(effects
 				(font
@@
 		)
 		(instances
-			(project "esquematico_V4"
+			(project "estacao-meteorologica"
 				(path "/0c305a6e-f9cd-49a1-b146-c2956e5469b6/ee5e162e-fef6-4e44-a551-c13cb2903f32"
 					(reference "TP222")
@@
 	(symbol
 		(lib_id "power:GND")
+		(at 100.33 93.98 0)
+		(mirror y)
+		(unit 1)
+		(exclude_from_sim no)
+		(in_bom yes)
+		(on_board yes)
+		(dnp no)
+		(fields_autoplaced yes)
+		(property "Reference" "#PWR080"
+			(at 100.33 100.33 0)
+			(effects
+				(font
+					(size 1.27 1.27)
+				)
+				(hide yes)
+			)
+		)
+		(property "Value" "GND"
+			(at 100.33 99.06 0)
+			(effects
+				(font
+					(size 1.27 1.27)
+				)
+			)
+		)
+		(property "Footprint" ""
+			(at 100.33 93.98 0)
+			(effects
+				(font
+					(size 1.27 1.27)
+				)
+				(hide yes)
+			)
+		)
+		(property "Datasheet" ""
+			(at 100.33 93.98 0)
+			(effects
+				(font
+					(size 1.27 1.27)
+				)
+				(hide yes)
+			)
+		)
+		(property "Description" "Power symbol creates a global label with name \"GND\" , ground"
+			(at 100.33 93.98 0)
+			(effects
+				(font
+					(size 1.27 1.27)
+				)
+				(hide yes)
+			)
+		)
+		(pin "1"
+		)
+		(instances
+			(project "estacao-meteorologica"
+				(path "/0c305a6e-f9cd-49a1-b146-c2956e5469b6/ee5e162e-fef6-4e44-a551-c13cb2903f32"
+					(reference "#PWR080")
+					(unit 1)
+				)
+			)
+		)
+	)
+	(symbol
+		(lib_id "power:GND")
 		(at 99.06 69.85 90)
 		(mirror x)
@@
 	(symbol
 		(lib_id "power:+3V3")
-		(at 99.06 72.39 270)
+		(at 137.16 77.47 270)
 		(mirror x)
 		(unit 1)
@@
 		(fields_autoplaced yes)
 		(property "Reference" "#PWR05"
-			(at 95.25 72.39 0)
+			(at 133.35 77.47 0)
 			(effects
 				(font
@@
 		)
 		(property "Value" "+3V3"
-			(at 102.87 72.3899 90)
+			(at 140.97 77.4699 90)
 			(effects
 				(font
@@
 		)
 		(property "Footprint" ""
-			(at 99.06 72.39 0)
+			(at 137.16 77.47 0)
 			(effects
 				(font
@@
 		)
 		(property "Datasheet" ""
-			(at 99.06 72.39 0)
+			(at 137.16 77.47 0)
 			(effects
 				(font
@@
 		)
 		(property "Description" "Power symbol creates a global label with name \"+3V3\""
-			(at 99.06 72.39 0)
+			(at 137.16 77.47 0)
 			(effects
 				(font
@@
 		)
 		(instances
-			(project ""
+			(project "estacao-meteorologica"
 				(path "/0c305a6e-f9cd-49a1-b146-c2956e5469b6/ee5e162e-fef6-4e44-a551-c13cb2903f32"
 					(reference "#PWR05")

Commit message: feat(hardware): consolida revisão PCB V2
Connections:
- net +3V3: now also J221.4 (Pin_4)
- net BH_I2C3_SCL: now also D222.2 (A2), J221.2 (Pin_2), TP222.1; no longer D221.2 (A2), J221.3 (Pin_3), TP221.1
- net BH_I2C3_SDA: now also D221.2 (A2), J221.3 (Pin_3), TP221.1; no longer D222.2 (A2), J221.2 (Pin_2), TP222.1
Changed lines of the file:
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@@
 	(hierarchical_label "BH_I2C3_SDA"
 		(shape passive)
-		(at 121.92 72.39 0)
+		(at 121.92 74.93 0)
 		(effects
 			(font
@@
 	(hierarchical_label "BH_I2C3_SCL"
 		(shape passive)
-		(at 121.92 74.93 0)
+		(at 121.92 72.39 0)
 		(effects
 			(font
@@
 	(symbol
 		(lib_id "power:+3V3")
-		(at 137.16 77.47 270)
+		(at 121.92 77.47 270)
 		(mirror x)
 		(unit 1)
@@
 		(fields_autoplaced yes)
 		(property "Reference" "#PWR05"
-			(at 133.35 77.47 0)
+			(at 118.11 77.47 0)
 			(effects
 				(font
@@
 		)
 		(property "Value" "+3V3"
-			(at 140.97 77.4699 90)
+			(at 125.73 77.4699 90)
 			(effects
 				(font
@@
 		)
 		(property "Footprint" ""
-			(at 137.16 77.47 0)
+			(at 121.92 77.47 0)
 			(effects
 				(font
@@
 		)
 		(property "Datasheet" ""
-			(at 137.16 77.47 0)
+			(at 121.92 77.47 0)
 			(effects
 				(font
@@
 		)
 		(property "Description" "Power symbol creates a global label with name \"+3V3\""
-			(at 137.16 77.47 0)
-			(effects
-				(font
+			(at 121.92 77.47 0)
+			(effects
+				(font
