File: hardware/kicad/estacao-meteorologica/sheets/biruta.kicad_sch (KiCad schematic)
At the start: 11 parts, among them J32 R-RJ11R06P-A800

Commit message: refatoracao: atualizacoes de hardware e falta revisao LoRa
Parts:
- C50: value 10n -> 100n
- J32: Function RJ11 individual; contatos centrais -> Conector da biruta; p3/p4 apenas passagem Anem/Pluv, sem co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; Rating 6P6C; p3=return; p4=signal; THT -> 6P6C; p2=direcao; p5=GND; p3=+3V3 e p4=passagem reservada; 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
- TP52: value VREF_SENSOR -> AVREF_SENSOR; Function VREF_SENSOR -> AVREF_SENSOR
Connections:
- net +3V3: now also J32.3
- net GND: now also J32.5; no longer J32.3
- net WIND_DIR_RAW: now also J32.2; no longer J32.4
- net VREF_SENSOR renamed AVREF_SENSOR
- new net Anem/Pluv_Sig: J32.4
- no-connect marks 4 -> 2
Other:
- note added: "AVREF_SENSOR deve vir de VDDA/AVDD do STM32, apos o filtro analogico; nao unir ao 3V3 digital por etiqueta. C50 junto ao PA0; retorno GND curto. Medir offsets por fuga e temperatura. A LUT ativa do firmware tem 16 entradas; 8 e o numero de amostras por leitura."
- note added: "MISOL WH-SP-WD: rede resistiva passiva; 8 chaves / ate 16 codigos; cabo ~2 m. J32: p2=direcao do vento; p5=GND. p3=+3V3 e p4=Anem/Pluv_Sig sao passagem reservada, sem conexao aos condicionamentos."
- note added: "R50=10k 1%; ADC ideal=4095*R_sensor/(10000+R_sensor). R51/R52 estao APOS o divisor: nao entram na relacao DC ideal. Rfonte maxima ~20,23k; C50=100n: tau maxima ~2,02 ms; validar tempo ADC (144 ciclos)."
- note removed: "MISOL WH-SP-WD: rede resistiva passiva; 8 chaves / ate 16 codigos; cabo ~2 m."
- note removed: "R50=10k 1%; ADC ideal=4095*R_sensor/(10000+R_sensor). R51/R52 estao APOS o divisor: nao entram na relacao DC ideal. Rfonte maxima ~20,23k; tau maxima ~202 us; validar tempo ADC (144 ciclos)."
- note removed: "VREF_SENSOR vem de U5 CN10_7 (AVDD). Nao unir ao 3V3 digital por etiqueta. C50 junto ao PA0; retorno GND curto. Medir offsets por fuga e temperatura. A LUT ativa do firmware tem 16 entradas; 8 e o numero de amostras por leitura."
- moved on the sheet: J32, TP51, TP52

Commit message: refatoracao: lora + Verificacao projeto inteiro
Parts:
- C50: LCSC C57112 -> C14663; LCSC Part C57112 -> C14663; MPN 0603B103K500NT -> CC0603KRX7R9BB104; Manufacturer FH -> YAGEO; Modelo 3D (none) -> ${KICAD9_3DMODEL_DIR}/Capacitor_SMD.3dshapes/C_0603_1608Met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; Status_Ficha (none) -> Conferido no catalogo em 2026-09-24; verificar estoque ao c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
- D50: Modelo 3D (none) -> ${KICAD9_3DMODEL_DIR}/Diode_SMD.3dshapes/D_SOD-882.step; Status_Ficha (none) -> Conferido no catalogo em 2026-09-24; verificar estoque ao c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
- D51: Modelo 3D (none) -> ${KICAD9_3DMODEL_DIR}/Package_TO_SOT_SMD.3dshapes/SOT-23.st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; Status_Ficha (none) -> Conferido no catalogo em 2026-09-24; verificar estoque ao c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
- J32: Function Conector da biruta; p3/p4 apenas passagem Anem/Pluv, sem co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 -> Conector da biruta; p4=WIND_DIR_RAW para o condicionamento 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; Manufacturer Ckmtw -> Ckmtw(Shenzhen Cankemeng); Modelo 3D (none) -> ${KIPRJMOD}/../../libraries/Sensores_Meteo/Sensores_Meteo.3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; Rating 6P6C; p2=direcao; p5=GND; p3=+3V3 e p4=passagem reservada; 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 -> 6P6C; p2=GND; p3=+3V3; p4=direcao do vento; p1/p5/p6=NC; THT; Status_Ficha (none) -> Conferido no catalogo em 2026-09-24; verificar estoque ao c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
- R50, R51, R52: Manufacturer UNI-ROYAL -> UNI-ROYAL(Uniroyal Elec); Modelo 3D (none) -> ${KICAD9_3DMODEL_DIR}/Resistor_SMD.3dshapes/R_0603_1608Metr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; Status_Ficha (none) -> Conferido no catalogo em 2026-09-24; verificar estoque ao c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
- TP50, TP51, TP52, TP53: LCSC (none) -> N/A; LCSC Part (none) -> N/A; MPN (none) -> N/A - elemento de cobre da PCB; Manufacturer (none) -> N/A; Modelo 3D (none) -> N/A - geometria de cobre, sem corpo
Connections:
- net Anem/Pluv_Sig renamed Sinal_2
- net WIND_DIR_RAW: no longer names the net of D50.1 (K), J32.2, R50.2, R51.1, TP50.1
Other:
- note added: "MISOL WH-SP-WD: rede resistiva passiva; 8 chaves / ate 16 codigos; cabo ~2 m. J32: p2=GND; p3=+3V3; p4=direcao do vento; p1/p5/p6=NC."
- note removed: "MISOL WH-SP-WD: rede resistiva passiva; 8 chaves / ate 16 codigos; cabo ~2 m. J32: p2=direcao do vento; p5=GND. p3=+3V3 e p4=Anem/Pluv_Sig sao passagem reservada, sem conexao aos condicionamentos."

Commit message: Padronizacao de nomes e numero de componentes
Parts:
- C501: renamed from C50; value 100n -> 100 nF; Assembly (none) -> SMT; LCSC Part C14663 -> (none); Modelo 3D ${KICAD9_3DMODEL_DIR}/Capacitor_SMD.3dshapes/C_0603_1608Met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 -> (none); Rating 10%; 50V; X7R -> (none); Specification (none) -> 10%; 50V; X7R; Status_Ficha Conferido no catalogo em 2026-09-24; verificar estoque ao c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 -> (none); Verification (none) -> Conferido no catalogo em 2026-09-24; verificar estoque ao c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
- D501: renamed from D50; Assembly (none) -> SMT; LCSC Part C85402 -> (none); Modelo 3D ${KICAD9_3DMODEL_DIR}/Diode_SMD.3dshapes/D_SOD-882.step -> (none); Rating VRWM=5V; IR max 1uA at 5V/25C; see datasheet -> (none); Specification (none) -> VRWM=5V; IR max 1uA at 5V/25C; see datasheet; Status_Ficha Conferido no catalogo em 2026-09-24; verificar estoque ao c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 -> (none); Verification (none) -> Conferido no catalogo em 2026-09-24; verificar estoque ao c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
- D502: renamed from D51; Assembly (none) -> SMT; LCSC Part C389351 -> (none); Modelo 3D ${KICAD9_3DMODEL_DIR}/Package_TO_SOT_SMD.3dshapes/SOT-23.st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 -> (none); Rating IR max 100nA at 50V/25C; 1=GND, 2=3V3, 3=signal -> (none); Specification (none) -> IR max 100nA at 50V/25C; 1=GND, 2=3V3, 3=signal; Status_Ficha Conferido no catalogo em 2026-09-24; verificar estoque ao c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 -> (none); Verification (none) -> Conferido no catalogo em 2026-09-24; verificar estoque ao c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
- J501: renamed from J32; value R-RJ11R06P-A800 -> RJ11 6P6C, 90°; Assembly (none) -> SMT; LCSC Part C189750 -> (none); Modelo 3D ${KIPRJMOD}/../../libraries/Sensores_Meteo/Sensores_Meteo.3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 -> (none); Rating 6P6C; p2=GND; p3=+3V3; p4=direcao do vento; p1/p5/p6=NC; THT -> (none); Specification (none) -> 6P6C; p2=GND; p3=+3V3; p4=direcao do vento; p1/p5/p6=NC; THT; Status_Ficha Conferido no catalogo em 2026-09-24; verificar estoque ao c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 -> (none); Verification (none) -> Conferido no catalogo em 2026-09-24; verificar estoque ao c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
- R501: renamed from R50; value 10k -> 10 kΩ; Assembly (none) -> SMT; LCSC Part C25804 -> (none); Modelo 3D ${KICAD9_3DMODEL_DIR}/Resistor_SMD.3dshapes/R_0603_1608Metr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 -> (none); Rating 1%; 0.1W; 75V -> (none); Specification (none) -> 1%; 0.1W; 75V; Status_Ficha Conferido no catalogo em 2026-09-24; verificar estoque ao c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 -> (none); Verification (none) -> Conferido no catalogo em 2026-09-24; verificar estoque ao c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
- R502: renamed from R51; value 10k -> 10 kΩ; Assembly (none) -> SMT; LCSC Part C25804 -> (none); Modelo 3D ${KICAD9_3DMODEL_DIR}/Resistor_SMD.3dshapes/R_0603_1608Metr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 -> (none); Rating 1%; 0.1W; 75V -> (none); Specification (none) -> 1%; 0.1W; 75V; Status_Ficha Conferido no catalogo em 2026-09-24; verificar estoque ao c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 -> (none); Verification (none) -> Conferido no catalogo em 2026-09-24; verificar estoque ao c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
- R503: renamed from R52; value 1k -> 1 kΩ; Assembly (none) -> SMT; LCSC Part C21190 -> (none); Modelo 3D ${KICAD9_3DMODEL_DIR}/Resistor_SMD.3dshapes/R_0603_1608Metr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 -> (none); Rating 1%; 0.1W; 75V -> (none); Specification (none) -> 1%; 0.1W; 75V; Status_Ficha Conferido no catalogo em 2026-09-24; verificar estoque ao c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 -> (none); Verification (none) -> Conferido no catalogo em 2026-09-24; verificar estoque ao c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
- TP501: renamed from TP50; value WIND_DIR_RAW -> SENS_WIND_DIR_RAW; Assembly (none) -> PCB — sem compra; Function WIND_DIR_RAW -> SENS_WIND_DIR_RAW; LCSC Part N/A -> (none); Modelo 3D N/A - geometria de cobre, sem corpo -> (none); Rating Copper pad; no purchased component -> (none); Specification (none) -> Copper pad; no purchased component
- TP502: renamed from TP51; Assembly (none) -> PCB — sem compra; LCSC Part N/A -> (none); Modelo 3D N/A - geometria de cobre, sem corpo -> (none); Rating Copper pad; no purchased component -> (none); Specification (none) -> Copper pad; no purchased component
- TP503: renamed from TP52; Assembly (none) -> PCB — sem compra; LCSC Part N/A -> (none); Modelo 3D N/A - geometria de cobre, sem corpo -> (none); Rating Copper pad; no purchased component -> (none); Specification (none) -> Copper pad; no purchased component
- TP504: renamed from TP53; Assembly (none) -> PCB — sem compra; LCSC Part N/A -> (none); Modelo 3D N/A - geometria de cobre, sem corpo -> (none); Rating Copper pad; no purchased component -> (none); Specification (none) -> Copper pad; no purchased component
Connections:
- net Sinal_2 renamed SENS_SPARE

Commit message: Ajuste de componentes por folha
Connections:
- net SENS_SPARE: no longer names the net of J501.4
- no-connect marks 2 -> 3
Changed lines of the file:
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@@
+	)
+	(no_connect
+		(at 45.72 77.47)
 	)
 	(no_connect
@@
 			(width 0)
 			(type default)
-		)
-	)
-	(global_label "SENS_SPARE"
-		(shape input)
-		(at 45.72 77.47 0)
-		(fields_autoplaced yes)
-		(effects
-			(font
-				(size 1.27 1.27)
-			)
-			(justify left)
-		)
-		(property "Intersheetrefs" "${INTERSHEET_REFS}"
-			(at 55.6598 77.47 0)
-			(effects
-				(font
-					(size 1.27 1.27)
-				)
-				(justify left)
-				(hide yes)
-			)
 		)
 	)
@@
 			)
 		)
+		(property "Assembly" "PCB — sem compra"
+			(at 0 0 0)
+			(effects
+				(font
+					(size 1.27 1.27)
+				)
+				(hide yes)
+			)
+		)
 		(pin "1"
 		)
@@
 					(unit 1)
 				)
-			)
-		)
-		(property "Assembly" "PCB — sem compra"
-			(at 0 0 0)
-			(effects
-				(font (size 1.27 1.27))
-				(hide yes)
 			)
 		)
@@
 			)
 		)
+		(property "Assembly" "SMT"
+			(at 0 0 0)
+			(effects
+				(font
+					(size 1.27 1.27)
+				)
+				(hide yes)
+			)
+		)
 		(pin "2"
 		)
@@
 					(unit 1)
 				)
-			)
-		)
-		(property "Assembly" "SMT"
-			(at 0 0 0)
-			(effects
-				(font (size 1.27 1.27))
-				(hide yes)
 			)
 		)
@@
 			)
 		)
+		(property "Assembly" "SMT"
+			(at 0 0 0)
+			(effects
+				(font
+					(size 1.27 1.27)
+				)
+				(hide yes)
+			)
+		)
 		(pin "1"
 		)
@@
 					(unit 1)
 				)
-			)
-		)
-		(property "Assembly" "SMT"
-			(at 0 0 0)
-			(effects
-				(font (size 1.27 1.27))
-				(hide yes)
 			)
 		)
@@
 			)
 		)
+		(property "Assembly" "PCB — sem compra"
+			(at 0 0 0)
+			(effects
+				(font
+					(size 1.27 1.27)
+				)
+				(hide yes)
+			)
+		)
 		(pin "1"
 		)
@@
 					(unit 1)
 				)
-			)
-		)
-		(property "Assembly" "PCB — sem compra"
-			(at 0 0 0)
-			(effects
-				(font (size 1.27 1.27))
-				(hide yes)
 			)
 		)
@@
 			)
 		)
+		(property "Assembly" "SMT"
+			(at 0 0 0)
+			(effects
+				(font
+					(size 1.27 1.27)
+				)
+				(hide yes)
+			)
+		)
 		(pin "1"
 		)
@@
 					(unit 1)
 				)
-			)
-		)
-		(property "Assembly" "SMT"
-			(at 0 0 0)
-			(effects
-				(font (size 1.27 1.27))
-				(hide yes)
 			)
 		)
@@
 			)
 		)
+		(property "Assembly" "SMT"
+			(at 0 0 0)
+			(effects
+				(font
+					(size 1.27 1.27)
+				)
+				(hide yes)
+			)
+		)
 		(pin "2"
 		)
@@
 					(unit 1)
 				)
-			)
-		)
-		(property "Assembly" "SMT"
-			(at 0 0 0)
-			(effects
-				(font (size 1.27 1.27))
-				(hide yes)
 			)
 		)
@@
 			)
 		)
+		(property "Assembly" "SMT"
+			(at 0 0 0)
+			(effects
+				(font
+					(size 1.27 1.27)
+				)
+				(hide yes)
+			)
+		)
 		(pin "1"
 		)
@@
 					(unit 1)
 				)
-			)
-		)
-		(property "Assembly" "SMT"
-			(at 0 0 0)
-			(effects
-				(font (size 1.27 1.27))
-				(hide yes)
 			)
 		)
@@
 			)
 		)
+		(property "Assembly" "PCB — sem compra"
+			(at 0 0 0)
+			(effects
+				(font
+					(size 1.27 1.27)
+				)
+				(hide yes)
+			)
+		)
 		(pin "1"
 		)
@@
 					(unit 1)
 				)
-			)
-		)
-		(property "Assembly" "PCB — sem compra"
-			(at 0 0 0)
-			(effects
-				(font (size 1.27 1.27))
-				(hide yes)
 			)
 		)
@@
 			)
 		)
+		(property "Assembly" "PCB — sem compra"
+			(at 0 0 0)
+			(effects
+				(font
+					(size 1.27 1.27)
+				)
+				(hide yes)
+			)
+		)
 		(pin "1"
 		)
@@
 					(unit 1)
 				)
-			)
-		)
-		(property "Assembly" "PCB — sem compra"
-			(at 0 0 0)
-			(effects
-				(font (size 1.27 1.27))
-				(hide yes)
 			)
 		)
@@
 			)
 		)
+		(property "Assembly" "SMT"
+			(at 0 0 0)
+			(effects
+				(font
+					(size 1.27 1.27)
+				)
+				(hide yes)
+			)
+		)
 		(pin "2"
 		)
@@
 					(unit 1)
 				)
-			)
-		)
-		(property "Assembly" "SMT"
-			(at 0 0 0)
-			(effects
-				(font (size 1.27 1.27))
-				(hide yes)
 			)
 		)
@@
 			)
 		)
+		(property "Assembly" "SMT"
+			(at 0 0 0)
+			(effects
+				(font
+					(size 1.27 1.27)
+				)
+				(hide yes)
+			)
+		)
 		(pin "6"
 		)
@@
 			)
 		)
-		(property "Assembly" "SMT"
-			(at 0 0 0)
-			(effects
-				(font (size 1.27 1.27))
-				(hide yes)
-			)
-		)

Commit message: Roteamento 2.0 - rj11 compartilhado biruta e anemometro
Parts:
- added R1: 1 kΩ, Resistor_SMD:R_0603_1608Metric, symbol Device:R
Connections:
- net +3V3: now also R1.2; no longer J501.3
- net SENS_WIND_SPEED_RAW: now reaches J501.4
- new net: J501.3, R1.1
- no-connect marks 3 -> 2
Changed lines of the file:
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@@
-	)
-	(no_connect
-		(at 45.72 77.47)
 	)
 	(no_connect
@@
 	(wire
 		(pts
+			(xy 49.53 99.06) (xy 50.8 99.06)
+		)
+		(stroke
+			(width 0)
+			(type default)
+		)
+	)
+	(wire
+		(pts
+			(xy 50.8 92.71) (xy 50.8 99.06)
+		)
+		(stroke
+			(width 0)
+			(type default)
+		)
+	)
+	(wire
+		(pts
+			(xy 45.72 80.01) (xy 50.8 80.01)
+		)
+		(stroke
+			(width 0)
+			(type default)
+		)
+	)
+	(wire
+		(pts
+			(xy 50.8 80.01) (xy 50.8 85.09)
+		)
+		(stroke
+			(width 0)
+			(type default)
+		)
+	)
+	(wire
+		(pts
 			(xy 157.48 63.5) (xy 157.48 80.01)
 		)
@@
 		)
 	)
-	(global_label "+3V3"
+	(global_label "SENS_WIND_SPEED_RAW"
 		(shape passive)
-		(at 45.72 80.01 0)
+		(at 45.72 77.47 0)
+		(fields_autoplaced yes)
 		(effects
 			(font
-				(size 1 1)
+				(size 1.27 1.27)
 			)
 			(justify left)
 		)
 		(property "Intersheetrefs" "${INTERSHEET_REFS}"
-			(at 45.72 80.01 0)
-			(effects
-				(font
-					(size 1.27 1.27)
-				)
+			(at 69.9094 77.47 0)
+			(effects
+				(font
+					(size 1.27 1.27)
+				)
+				(justify left)
 				(hide yes)
 			)
@@
 				(path "/0c305a6e-f9cd-49a1-b146-c2956e5469b6/058dce74-971b-49d7-82f0-384e20be985c/4ef75fdb-90eb-437a-af55-0afcbbe28aca"
 					(reference "D501")
+					(unit 1)
+				)
+			)
+		)
+	)
+	(symbol
+		(lib_id "Device:R")
+		(at 50.8 88.9 0)
+		(unit 1)
+		(exclude_from_sim no)
+		(in_bom yes)
+		(on_board yes)
+		(dnp no)
+		(property "Reference" "R1"
+			(at 54.61 86.36 0)
+			(effects
+				(font
+					(size 1 1)
+				)
+			)
+		)
+		(property "Value" "1 kΩ"
+			(at 54.61 88.9 0)
+			(effects
+				(font
+					(size 1 1)
+				)
+			)
+		)
+		(property "Footprint" "Resistor_SMD:R_0603_1608Metric"
+			(at 50.8 88.9 0)
+			(effects
+				(font
+					(size 1 1)
+				)
+				(hide yes)
+			)
+		)
+		(property "Datasheet" "https://www.lcsc.com/datasheet/lcsc_datasheet_2206010130_UNI-ROYAL-Uniroyal-Elec-0603WAF1001T5E_C21190.pdf"
+			(at 50.8 88.9 0)
+			(effects
+				(font
+					(size 1 1)
+				)
+				(hide yes)
+			)
+		)
+		(property "Description" "Resistor SMD 1 kohm, 1%, 0,1 W, 0603"
+			(at 50.8 88.9 0)
+			(effects
+				(font
+					(size 1.27 1.27)
+				)
+				(hide yes)
+			)
+		)
+		(property "Manufacturer" "UNI-ROYAL(Uniroyal Elec)"
+			(at 50.8 88.9 0)
+			(effects
+				(font
+					(size 1 1)
+				)
+				(hide yes)
+			)
+		)
+		(property "MPN" "0603WAF1001T5E"
+			(at 50.8 88.9 0)
+			(effects
+				(font
+					(size 1 1)
+				)
+				(hide yes)
+			)
+		)
+		(property "LCSC" "C21190"
+			(at 50.8 88.9 0)
+			(effects
+				(font
+					(size 1 1)
+				)
+				(hide yes)
+			)
+		)
+		(property "Specification" "1%; 0.1W; 75V"
+			(at 50.8 88.9 0)
+			(effects
+				(font
+					(size 1 1)
+				)
+				(hide yes)
+			)
+		)
+		(property "Function" "Resistor serie da alimentacao do cabo; limita corrente pelo reed e pelo TVS"
+			(at 50.8 88.9 0)
+			(effects
+				(font
+					(size 1 1)
+				)
+				(hide yes)
+			)
+		)
+		(property "Verification" "Conferido no catalogo em 2026-09-24; verificar estoque ao comprar"
+			(at 50.8 88.9 0)
+			(effects
+				(font
+					(size 1.27 1.27)
+				)
+				(hide yes)
+			)
+		)
+		(property "Assembly" "SMT"
+			(at 2.54 -8.89 0)
+			(effects
+				(font
+					(size 1.27 1.27)
+				)
+				(hide yes)
+			)
+		)
+		(pin "1"
+		)
+		(pin "2"
+		)
+		(instances
+			(project "estacao-meteorologica"
+				(path "/0c305a6e-f9cd-49a1-b146-c2956e5469b6/058dce74-971b-49d7-82f0-384e20be985c/4ef75fdb-90eb-437a-af55-0afcbbe28aca"
+					(reference "R1")
 					(unit 1)
 				)
@@
 					(unit 1)
 				)
+			)
+		)
+	)
+	(symbol
+		(lib_id "power:+3V3")
+		(at 49.53 99.06 90)
+		(unit 1)
+		(exclude_from_sim no)
+		(in_bom yes)
+		(on_board yes)
+		(dnp no)
+		(fields_autoplaced yes)
+		(property "Reference" "#PWR081"
+			(at 53.34 99.06 0)
+			(effects
+				(font
+					(size 1.27 1.27)
+				)
+				(hide yes)
+			)
+		)
+		(property "Value" "+3V3"
+			(at 45.72 99.0599 90)
+			(effects
+				(font
+					(size 1.27 1.27)
+				)
+				(justify left)
+			)
+		)
+		(property "Footprint" ""
+			(at 49.53 99.06 0)
+			(effects
+				(font
+					(size 1.27 1.27)
+				)
+				(hide yes)
+			)
+		)
+		(property "Datasheet" ""
+			(at 49.53 99.06 0)
+			(effects
+				(font
+					(size 1.27 1.27)
+				)
+				(hide yes)
+			)
+		)
+		(property "Description" "Power symbol creates a global label with name \"+3V3\""
+			(at 49.53 99.06 0)
+			(effects
+				(font
+					(size 1.27 1.27)
+				)
+				(hide yes)
+			)
+		)
+		(pin "1"
+		)
+		(instances
+			(project "estacao-meteorologica"
+				(path "/0c305a6e-f9cd-49a1-b146-c2956e5469b6/058dce74-971b-49d7-82f0-384e20be985c/4ef75fdb-90eb-437a-af55-0afcbbe28aca"
+					(reference "#PWR081")
+					(unit 1)
+				)

Commit message: Add test points necessarios para debug
Parts:
- TP501, TP502, TP503: footprint TestPoint:TestPoint_Pad_D1.5mm -> TestPoint:TestPoint_Pad_D1.0mm
Changed lines of the file:
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@@
 			)
 		)
-		(property "Footprint" "TestPoint:TestPoint_Pad_D1.5mm"
+		(property "Footprint" "TestPoint:TestPoint_Pad_D1.0mm"
 			(at 90.17 50.8 0)
 			(effects
@@
 			)
 		)
-		(property "Description" "Ponto de teste em cobre, pad circular de 1,5 mm; rede AVREF_SENSOR"
+		(property "Description" "Ponto de teste em cobre, pad circular de 1,0 mm; rede AVREF_SENSOR"
 			(at 90.17 50.8 0)
 			(effects
@@
 			)
 		)
-		(property "Footprint" "TestPoint:TestPoint_Pad_D1.5mm"
+		(property "Footprint" "TestPoint:TestPoint_Pad_D1.0mm"
 			(at 66.04 69.85 0)
 			(effects
@@
 			)
 		)
-		(property "Description" "Ponto de teste em cobre, pad circular de 1,5 mm; rede WIND_DIR_RAW"
+		(property "Description" "Ponto de teste em cobre, pad circular de 1,0 mm; rede WIND_DIR_RAW"
 			(at 66.04 69.85 0)
 			(effects
@@
 			)
 		)
-		(property "Footprint" "TestPoint:TestPoint_Pad_D1.5mm"
+		(property "Footprint" "TestPoint:TestPoint_Pad_D1.0mm"
 			(at 232.41 95.25 0)
 			(effects
@@
 			)
 		)
-		(property "Description" "Ponto de teste em cobre, pad circular de 1,5 mm; rede WIND_DIR_ADC"
+		(property "Description" "Ponto de teste em cobre, pad circular de 1,0 mm; rede WIND_DIR_ADC"
 			(at 232.41 95.25 0)
 			(effects

Commit message: feat(hardware): consolida revisão PCB V2
Parts:
- TP504: footprint TestPoint:TestPoint_Pad_D1.5mm -> TestPoint:TestPoint_Pad_D1.0mm
Changed lines of the file:
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@@
 			)
 		)
-		(property "Footprint" "TestPoint:TestPoint_Pad_D1.5mm"
+		(property "Footprint" "TestPoint:TestPoint_Pad_D1.0mm"
 			(at 81.28 111.76 0)
 			(effects
