File: hardware/kicad/estacao-meteorologica/sheets/cartao_sd.kicad_sch (KiCad schematic)
At the start: 9 parts, among them J801 microSD socket, TF-15x15, U801 SN74LVC125APWR, U802 EMIF06-MSD02N16

Commit message: feat(hardware): consolida revisão PCB V2
Connections:
- net SD_CS_BUF: now also U801.8; no longer U801.11
- net SD_MISO: now also U801.3; no longer U801.6
- net SD_MISO_BUF: now also U801.2; no longer U801.5
- net SD_MOSI_BUF: now also U801.11; no longer U801.3
- net SD_SCK: now also U801.5; no longer U801.9
- net SD_SCK_BUF: now also U801.6; no longer U801.8
- net SD_SPI_CS: now also U801.9; no longer R801.1, U801.12
- net SD_SPI_MOSI: now also R801.1, U801.12; no longer U801.2
Changed lines of the file:
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@@
-		)
-	)
-	(global_label "SD_SCK_BUF"
-		(shape output)
-		(at 78.74 100.33 0)
-		(fields_autoplaced yes)
-		(effects
-			(font
-				(size 1.27 1.27)
-			)
-			(justify left)
-		)
-		(property "Intersheetrefs" "${INTERSHEET_REFS}"
-			(at 89.708 100.33 0)
-			(effects
-				(font
-					(size 1.27 1.27)
-				)
-				(justify left)
-				(hide yes)
-			)
 		)
 	)
@@
 				)
 				(justify right)
-				(hide yes)
-			)
-		)
-	)
-	(global_label "SD_MOSI_BUF"
-		(shape output)
-		(at 78.74 62.23 0)
-		(fields_autoplaced yes)
-		(effects
-			(font
-				(size 1.27 1.27)
-			)
-			(justify left)
-		)
-		(property "Intersheetrefs" "${INTERSHEET_REFS}"
-			(at 87.8333 62.23 0)
-			(effects
-				(font
-					(size 1.27 1.27)
-				)
-				(justify left)
 				(hide yes)
 			)
@@
 		)
 	)
+	(global_label "SD_CS_BUF"
+		(shape output)
+		(at 78.74 100.33 0)
+		(fields_autoplaced yes)
+		(effects
+			(font
+				(size 1.27 1.27)
+			)
+			(justify left)
+		)
+		(property "Intersheetrefs" "${INTERSHEET_REFS}"
+			(at 92.3085 100.33 0)
+			(effects
+				(font
+					(size 1.27 1.27)
+				)
+				(justify left)
+				(hide yes)
+			)
+		)
+	)
 	(global_label "SD_CARD_CS"
 		(shape input)
@@
 		)
 	)
+	(global_label "SD_MISO_BUF"
+		(shape input)
+		(at 40.64 62.23 180)
+		(fields_autoplaced yes)
+		(effects
+			(font
+				(size 1.27 1.27)
+			)
+			(justify right)
+		)
+		(property "Intersheetrefs" "${INTERSHEET_REFS}"
+			(at 30.821 62.23 0)
+			(effects
+				(font
+					(size 1.27 1.27)
+				)
+				(justify right)
+				(hide yes)
+			)
+		)
+	)
 	(global_label "SD_SCK_BUF"
+		(shape output)
+		(at 72.39 82.55 0)
+		(fields_autoplaced yes)
+		(effects
+			(font
+				(size 1.27 1.27)
+			)
+			(justify left)
+		)
+		(property "Intersheetrefs" "${INTERSHEET_REFS}"
+			(at 83.358 82.55 0)
+			(effects
+				(font
+					(size 1.27 1.27)
+				)
+				(justify left)
+				(hide yes)
+			)
+		)
+	)
+	(global_label "SD_SCK_BUF"
 		(shape input)
 		(at 104.14 86.36 180)
@@
 				)
 				(justify right)
+				(hide yes)
+			)
+		)
+	)
+	(global_label "SD_MOSI_BUF"
+		(shape output)
+		(at 78.74 127 0)
+		(fields_autoplaced yes)
+		(effects
+			(font
+				(size 1.27 1.27)
+			)
+			(justify left)
+		)
+		(property "Intersheetrefs" "${INTERSHEET_REFS}"
+			(at 87.8333 127 0)
+			(effects
+				(font
+					(size 1.27 1.27)
+				)
+				(justify left)
 				(hide yes)
 			)
@@
 		)
 	)
-	(global_label "SD_CS_BUF"
-		(shape output)
-		(at 78.74 127 0)
-		(fields_autoplaced yes)
-		(effects
-			(font
-				(size 1.27 1.27)
-			)
-			(justify left)
-		)
-		(property "Intersheetrefs" "${INTERSHEET_REFS}"
-			(at 88.438 127 0)
-			(effects
-				(font
-					(size 1.27 1.27)
-				)
-				(justify left)
-				(hide yes)
-			)
-		)
-	)
-	(global_label "SD_MISO_BUF"
+	(hierarchical_label "SD_MISO"
+		(shape output)
+		(at 78.74 62.23 0)
+		(effects
+			(font
+				(size 1.27 1.27)
+			)
+			(justify left)
+		)
+	)
+	(hierarchical_label "SD_SCK"
 		(shape input)
 		(at 40.64 82.55 180)
-		(fields_autoplaced yes)
-		(effects
-			(font
-				(size 1.27 1.27)
-			)
-			(justify right)
-		)
-		(property "Intersheetrefs" "${INTERSHEET_REFS}"
-			(at 30.821 82.55 0)
-			(effects
-				(font
-					(size 1.27 1.27)
-				)
-				(justify right)
-				(hide yes)
-			)
-		)
-	)
-	(hierarchical_label "SD_MISO"
-		(shape output)
-		(at 72.39 82.55 0)
-		(effects
-			(font
-				(size 1.27 1.27)
-			)
-			(justify left)
-		)
-	)
-	(hierarchical_label "SD_SCK"
+		(effects
+			(font
+				(size 1.27 1.27)
+			)
+			(justify right)
+		)
+	)
+	(hierarchical_label "SD_SPI_CS"
 		(shape input)
 		(at 40.64 100.33 180)
@@
 		)
 	)
+	(hierarchical_label "SD_SPI_MOSI"
+		(shape input)
+		(at 40.64 127 180)
+		(effects
+			(font
+				(size 1.27 1.27)
+			)
+			(justify right)
+		)
+	)
 	(hierarchical_label "SD_CD"
 		(shape input)
@@
 		(effects
 			(font
-				(size 1.27 1.27)
-			)
-			(justify right)
-		)
-	)
-	(hierarchical_label "SD_SPI_MOSI"
-		(shape input)
-		(at 40.64 62.23 180)
-		(effects
-			(font
-				(size 1.27 1.27)
-			)
-			(justify right)
-		)
-	)
-	(hierarchical_label "SD_SPI_CS"
-		(shape input)
-		(at 40.64 127 180)
-		(effects
-			(font
