File: hardware/kicad/estacao-meteorologica/sheets/mcu.kicad_sch (KiCad schematic)
At the start: 27 parts, among them J101 Header, 1x02, P2.54 mm, J102 Header, 1x06, P2.54 mm, J103 Header, 1x03, P2.54 mm, SW101 Tactile switch, SPST, U101 STM32F446RET6, Y101 32.768 kHz, CL 7 pF, Y102 8 MHz, CL 10 pF

Commit message: Roteamento 2.0 - rj11 compartilhado biruta e anemometro
Parts:
- BT101: value CR2032 holder, vertical -> CR1225 holder, horizontal; footprint Hardware_MCU:BT_Holder_MPD_BS-5_Vertical -> Hardware_Battery:BT_Holder_MYOUNG_BS-12-B4AK025-R; Assembly Manual — suporte PTH vertical. -> SMT — montar o suporte vazio em reflow; inserir a CR1225 ap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; LCSC C6869743 -> C20606807; MPN BS-5 -> BS-12-B4AK025-R; Manufacturer MPD (Memory Protection Devices) -> MYOUNG; Specification CR2032/BR2032, 3 V; THT; 3 furos Ø0,9 mm; dois pads + e um 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 -> CR1225, 3 V; SMT; dois pads 3,15 x 4,00 mm em passo de 15,8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; Verification Conferido com desenho mecânico e STEP oficial do MPD BS-5. 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 -> Conferido com desenho mecânico MYOUNG WD-CP-0239. Item LCSC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
Changed lines of the file:
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@@
 			)
 		)
-		(property "Value" "CR2032 holder, vertical"
+		(property "Value" "CR1225 holder, horizontal"
 			(at 209.55 38.7984 0)
 			(effects
@@
 			)
 		)
-		(property "Footprint" "Hardware_MCU:BT_Holder_MPD_BS-5_Vertical"
+		(property "Footprint" "Hardware_Battery:BT_Holder_MYOUNG_BS-12-B4AK025-R"
 			(at 205.74 37.846 90)
 			(effects
@@
 			)
 		)
-		(property "Datasheet" "https://www.batteryholders.com/uploads/parts/BS-5/datasheets/BS-5-datasheet.pdf"
+		(property "Datasheet" "https://www.lcsc.com/datasheet/C20606807.pdf"
 			(at 205.74 37.846 90)
 			(effects
@@
 			)
 		)
-		(property "Description" "Suporte vertical THT para uma CR2032/BR2032; dois terminais positivos e um negativo; 17,8 mm acima da PCB."
+		(property "Description" "Suporte horizontal SMT completo para CR1225; dois terminais, positivo e negativo; 24,1 x 12,7 x 4,7 mm."
 			(at 205.74 39.37 0)
 			(effects
@@
 			)
 		)
-		(property "Verification" "Conferido com desenho mecânico e STEP oficial do MPD BS-5. Item LCSC C6869743 de montagem manual; confirmar estoque antes da compra."
+		(property "Verification" "Conferido com desenho mecânico MYOUNG WD-CP-0239. Item LCSC C20606807; confirmar estoque antes da compra."
 			(at 205.74 39.37 0)
 			(effects
@@
 			)
 		)
-		(property "MPN" "BS-5"
+		(property "MPN" "BS-12-B4AK025-R"
 			(at 205.74 39.37 0)
 			(effects
@@
 			)
 		)
-		(property "Manufacturer" "MPD (Memory Protection Devices)"
+		(property "Manufacturer" "MYOUNG"
 			(at 205.74 39.37 0)
 			(effects
@@
 			)
 		)
-		(property "LCSC" "C6869743"
+		(property "LCSC" "C20606807"
 			(at 205.74 39.37 0)
 			(effects
@@
 			)
 		)
-		(property "Specification" "CR2032/BR2032, 3 V; THT; 3 furos Ø0,9 mm; dois pads + e um pad −."
+		(property "Specification" "CR1225, 3 V; SMT; dois pads 3,15 x 4,00 mm em passo de 15,8 mm; perfil do suporte 4,7 mm."
 			(at 205.74 39.37 0)
 			(effects
@@
 			)
 		)
-		(property "Assembly" "Manual — suporte PTH vertical."
+		(property "Assembly" "SMT — montar o suporte vazio em reflow; inserir a CR1225 apenas após a montagem."
 			(at 205.74 39.37 0)
 			(effects

Commit message: Refact - mudança do sensor bh1750 para placa filha e conector jst + reposicionamento do sensor DHT22 para reduzir influencia de temperatura interna da placa
Parts:
- added R105, R106: 4.7k, Resistor_SMD:R_0603_1608Metric, symbol Device:R
Connections:
- net +3V3: now also R105.1, R106.1
- net DHT22_DATA: now also U101.42 (PA9); no longer U101.41 (PA8)
- net BH_I2C3_SDA: now reaches U101.40 (PC9)
- net BH_I2C3_SDA: now also R106.2
- new net BH_I2C3_SCL: R105.2, U101.41 (PA8)
- no-connect marks 23 -> 21
Other:
- moved on the sheet: J102

Commit message: rotemento 3.0
Parts:
- BT101: Specification CR1225, 3 V; SMT; dois pads 3,15 x 4,00 mm em passo de 15,8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 -> CR1225, 3 V; SMT; pads 3,15 x 4,00 mm em passo de 21,46 mm;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; Verification Conferido com desenho mecânico MYOUNG WD-CP-0239. Item LCSC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 -> Footprint e modelo STEP importados com easyeda2kicad v1.0.1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
Changed lines of the file:
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@@
 			)
 		)
-		(property "Verification" "Conferido com desenho mecânico MYOUNG WD-CP-0239. Item LCSC C20606807; confirmar estoque antes da compra."
+		(property "Verification" "Footprint e modelo STEP importados com easyeda2kicad v1.0.1 a partir do registro EasyEDA/LCSC C20606807 em 2026-09-28."
 			(at 205.74 39.37 0)
 			(effects
@@
 			)
 		)
-		(property "Specification" "CR1225, 3 V; SMT; dois pads 3,15 x 4,00 mm em passo de 15,8 mm; perfil do suporte 4,7 mm."
+		(property "Specification" "CR1225, 3 V; SMT; pads 3,15 x 4,00 mm em passo de 21,46 mm; altura do modelo importado 4,71 mm."
 			(at 205.74 39.37 0)
 			(effects

Commit message: feat(hardware): consolida revisão PCB V2
Connections:
- net GND: now also J102.6 (Pin_6); no longer J102.2 (Pin_2)
- net SWCLK: now also J102.3 (Pin_3); no longer J102.4 (Pin_4)
- net SWDIO: now also J102.2 (Pin_2); no longer J102.3 (Pin_3)
- net SWO: now also J102.4 (Pin_4); no longer J102.6 (Pin_6)
Changed lines of the file:
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@@
 		)
 	)
-	(global_label "TXD"
-		(shape bidirectional)
-		(at 177.8 73.66 0)
+	(global_label "NRST"
+		(shape passive)
+		(at 247.65 106.68 0)
 		(fields_autoplaced yes)
 		(effects
@@
 		)
 		(property "Intersheetrefs" "${INTERSHEET_REFS}"
-			(at 185.3436 73.66 0)
+			(at 254.3015 106.68 0)
 			(effects
 				(font
@@
 		)
 	)
-	(global_label "SWDIO"
-		(shape passive)
-		(at 247.65 101.6 0)
+	(global_label "TXD"
+		(shape bidirectional)
+		(at 177.8 73.66 0)
 		(fields_autoplaced yes)
 		(effects
@@
 		)
 		(property "Intersheetrefs" "${INTERSHEET_REFS}"
-			(at 255.3901 101.6 0)
+			(at 185.3436 73.66 0)
 			(effects
 				(font
@@
 		)
 	)
-	(global_label "SWO"
+	(global_label "VBAT"
 		(shape passive)
-		(at 247.65 109.22 0)
+		(at 147.32 55.88 90)
 		(fields_autoplaced yes)
 		(effects
@@
 		)
 		(property "Intersheetrefs" "${INTERSHEET_REFS}"
-			(at 253.5153 109.22 0)
+			(at 147.32 49.5913 90)
 			(effects
 				(font
@@
 	(global_label "SWCLK"
 		(shape passive)
-		(at 247.65 104.14 0)
+		(at 177.8 104.14 0)
 		(fields_autoplaced yes)
 		(effects
@@
 		)
 		(property "Intersheetrefs" "${INTERSHEET_REFS}"
-			(at 255.7529 104.14 0)
+			(at 185.9029 104.14 0)
 			(effects
 				(font
@@
 		)
 	)
-	(global_label "VBAT"
-		(shape passive)
-		(at 147.32 55.88 90)
+	(global_label "RXD"
+		(shape bidirectional)
+		(at 220.98 77.47 0)
 		(fields_autoplaced yes)
 		(effects
@@
 		)
 		(property "Intersheetrefs" "${INTERSHEET_REFS}"
-			(at 147.32 49.5913 90)
+			(at 228.826 77.47 0)
 			(effects
 				(font
@@
 		)
 	)
-	(global_label "SWCLK"
-		(shape passive)
-		(at 177.8 104.14 0)
+	(global_label "BOOT0"
+		(shape input)
+		(at 46.99 118.11 180)
 		(fields_autoplaced yes)
 		(effects
@@
 				(size 1.27 1.27)
 			)
-			(justify left)
+			(justify right)
 		)
 		(property "Intersheetrefs" "${INTERSHEET_REFS}"
-			(at 185.9029 104.14 0)
+			(at 37.8967 118.11 0)
 			(effects
 				(font
 					(size 1.27 1.27)
 				)
-				(justify left)
+				(justify right)
 				(hide yes)
 			)
 		)
 	)
-	(global_label "RXD"
-		(shape bidirectional)
-		(at 220.98 77.47 0)
+	(global_label "BOOT0"
+		(shape input)
+		(at 132.08 73.66 180)
 		(fields_autoplaced yes)
 		(effects
@@
 				(size 1.27 1.27)
 			)
-			(justify left)
+			(justify right)
 		)
 		(property "Intersheetrefs" "${INTERSHEET_REFS}"
-			(at 228.826 77.47 0)
+			(at 122.9867 73.66 0)
 			(effects
 				(font
 					(size 1.27 1.27)
 				)
-				(justify left)
+				(justify right)
 				(hide yes)
 			)
 		)
 	)
-	(global_label "BOOT0"
-		(shape input)
-		(at 46.99 118.11 180)
+	(global_label "SWCLK"
+		(shape passive)
+		(at 247.65 101.6 0)
 		(fields_autoplaced yes)
 		(effects
@@
 				(size 1.27 1.27)
 			)
-			(justify right)
+			(justify left)
 		)
 		(property "Intersheetrefs" "${INTERSHEET_REFS}"
-			(at 37.8967 118.11 0)
+			(at 255.7529 101.6 0)
 			(effects
 				(font
 					(size 1.27 1.27)
 				)
-				(justify right)
+				(justify left)
 				(hide yes)
 			)
 		)
 	)
-	(global_label "BOOT0"
-		(shape input)
-		(at 132.08 73.66 180)
+	(global_label "SWDIO"
+		(shape passive)
+		(at 247.65 99.06 0)
 		(fields_autoplaced yes)
 		(effects
@@
 				(size 1.27 1.27)
 			)
-			(justify right)
+			(justify left)
 		)
 		(property "Intersheetrefs" "${INTERSHEET_REFS}"
-			(at 122.9867 73.66 0)
+			(at 255.3901 99.06 0)
 			(effects
 				(font
 					(size 1.27 1.27)
 				)
-				(justify right)
+				(justify left)
 				(hide yes)
 			)
 		)
 	)
-	(global_label "VBAT"
+	(global_label "SWO"
 		(shape passive)
-		(at 205.74 30.48 90)
+		(at 247.65 104.14 0)
 		(fields_autoplaced yes)
 		(effects
@@
 		)
 		(property "Intersheetrefs" "${INTERSHEET_REFS}"
-			(at 205.74 24.1913 90)
+			(at 253.5153 104.14 0)
 			(effects
 				(font
@@
 		)
 	)
-	(global_label "TXD"
-		(shape bidirectional)
-		(at 220.98 74.93 0)
+	(global_label "VBAT"
+		(shape passive)
+		(at 205.74 30.48 90)
 		(fields_autoplaced yes)
 		(effects
@@
 		)
 		(property "Intersheetrefs" "${INTERSHEET_REFS}"
-			(at 228.5236 74.93 0)
+			(at 205.74 24.1913 90)
 			(effects
 				(font
@@
 		)
 	)
-	(global_label "NRST"
-		(shape passive)
-		(at 247.65 106.68 0)
+	(global_label "TXD"
+		(shape bidirectional)
+		(at 220.98 74.93 0)
 		(fields_autoplaced yes)
 		(effects
@@
 		)
 		(property "Intersheetrefs" "${INTERSHEET_REFS}"
-			(at 254.3015 106.68 0)
+			(at 228.5236 74.93 0)
 			(effects
 				(font
@@
 	(symbol
 		(lib_id "power:GND")
-		(at 247.65 99.06 90)
+		(at 247.65 109.22 90)
 		(unit 1)
 		(exclude_from_sim no)
@@
 		(fields_autoplaced yes)
 		(property "Reference" "#PWR050"
-			(at 254 99.06 0)
+			(at 254 109.22 0)
 			(effects
 				(font
@@
 		)
 		(property "Value" "GND"
-			(at 251.46 99.0599 90)
+			(at 251.46 109.2199 90)
 			(effects
 				(font
@@
 		)
 		(property "Footprint" ""
-			(at 247.65 99.06 0)
+			(at 247.65 109.22 0)
 			(effects
 				(font
@@
 		)
 		(property "Datasheet" ""
-			(at 247.65 99.06 0)
+			(at 247.65 109.22 0)
 			(effects
 				(font
@@
 		)
 		(property "Description" "Power symbol creates a global label with name \"GND\" , ground"
-			(at 247.65 99.06 0)
+			(at 247.65 109.22 0)
 			(effects
 				(font
