File: hardware/kicad/estacao-meteorologica/estacao-meteorologica.kicad_pcb (KiCad board)
At the start: 2 copper layers, 200 x 100 mm, 101 parts, among them J10 Conn_GND, J11 Conn_01x02_Socket, J13 Conn_+5V, J14 Conn_01x02_Socket, J15 Conn_01x02_Socket, J16 Conn_01x02_Socket, J17 Micro_SD_Card, J2 Conn_DHT, J23 RJ45, J24 RJ45, J25 RJ45, J30 R-RJ11R06P-A800, J31 R-RJ11R06P-A800, J32 R-RJ11R06P-A800, J4 Conn_cartao_SD, J5 Conn_BH1750, J6 Conn_BMP, J60 P4 / DC-005-2.0, J61 J_PWR / JST-XH, J7 Conn_Lora_4, J8 Conn_02x06_Row_Letter_Last, J9 Conn_+3v3, Q60 DMP6023LE-13, U1 DHT22, U11 74LVC125, U12 LORA1276-C1-915MHZ, U2 module_bh1750, U3 module_bme280, U30 SN74LVC1G17DBVR, U4 Lora_Sx1276, U40 SN74LVC1G17DBVR, U5 NUCLEO-F446RE, U6 MicroSD Card Adapter, U60 AP63205WU-7, U61 TLV62569DBVR, U7 NUCLEO-F446RE, U8 BMP280, U9 BH1750FVI-TR

Commit message: refatoracao: atualizacoes de hardware e falta revisao LoRa
Parts:
- removed C4, C5: 100n, Capacitor_THT:C_Disc_D3.8mm_W2.6mm_P2.50mm
- removed J10: Conn_GND, Connector_PinSocket_2.54mm:PinSocket_1x10_P2.54mm_Vertical
- removed J11: Conn_01x02_Socket, Connector_PinSocket_2.54mm:PinSocket_2x03_P2.54mm_Vertical
- removed J13: Conn_+5V, Connector_PinSocket_2.54mm:PinSocket_1x10_P2.54mm_Vertical
- removed J14, J15, J16: Conn_01x02_Socket, Connector_PinSocket_2.54mm:PinSocket_1x02_P2.54mm_Vertical
- removed J2: Conn_DHT, Connector_PinSocket_2.54mm:PinSocket_1x04_P2.54mm_Vertical
- removed J23, J24, J25: RJ45, Connector_RJ:RJ45_RCH_RC01937
- removed J4: Conn_cartao_SD, Connector_PinSocket_2.54mm:PinSocket_1x06_P2.54mm_Vertical
- removed J5: Conn_BH1750, Connector_PinSocket_2.54mm:PinSocket_1x05_P2.54mm_Vertical
- removed J6: Conn_BMP, Connector_PinSocket_2.54mm:PinSocket_1x06_P2.54mm_Vertical
- removed J7: Conn_Lora_4, Connector_PinSocket_2.54mm:PinSocket_2x04_P2.54mm_Vertical
- removed J8: Conn_02x06_Row_Letter_Last, Connector_PinSocket_2.54mm:PinSocket_2x06_P2.54mm_Vertical
- removed J9: Conn_+3v3, Connector_PinSocket_2.54mm:PinSocket_1x10_P2.54mm_Vertical
- removed PS1: Lm2596, myLibrary:LM2596_modulo
- removed R10, R11, R8: 10k, Resistor_THT:R_Axial_DIN0204_L3.6mm_D1.6mm_P7.62mm_Horizontal
- removed R61: 300k / 1%, Resistor_SMD:R_0603_1608Metric
- removed the U1 at (194.3, 116.8)
- removed the U1 at (-74.4, 50.2)
- removed U2: module_bh1750, myLibrary:bh1750_modulo
- removed U3: module_bme280, myLibrary:bme280_modulo
- removed U5, U7: NUCLEO-F446RE, myLibrary:MODULE_NUCLEO-F446RE
- removed U6: MicroSD Card Adapter, myLibrary:Micro_SD_Card_Adapter
- added C1: 100n, Capacitor_SMD:C_0603_1608Metric, F.Cu at (-42.6, 17.5)
- added C10: 100n, Capacitor_SMD:C_0603_1608Metric, F.Cu at (-97.2, 61.1)
- added C2: 100n, Capacitor_SMD:C_0603_1608Metric, F.Cu at (-42.6, 19.0)
- added C25: 100n, Capacitor_SMD:C_0603_1608Metric, F.Cu at (-46.2, 31.1)
- added C3: 100n, Capacitor_SMD:C_0603_1608Metric, F.Cu at (-66.4, 5.60)
- added C6: 1u, Capacitor_SMD:C_0603_1608Metric, F.Cu at (-38.2, 32.4)
- added C7: 10u / 50V, Capacitor_SMD:C_1206_3216Metric, F.Cu at (-111.1, 73.8)
- added C8: 100n, Capacitor_SMD:C_0603_1608Metric, F.Cu at (-97.2, 56.0)
- added C9: 100n, Capacitor_SMD:C_0603_1608Metric, F.Cu at (-97.2, 58.6)
- added R17: 10k, Resistor_SMD:R_0603_1608Metric, F.Cu at (-97.2, 63.6)
- added R18: 10k, Resistor_SMD:R_0603_1608Metric, F.Cu at (-97.2, 66.1)
- added R3: 10k, Resistor_SMD:R_0603_1608Metric, F.Cu at (-35.6, 18.2)
- added R32: 1k, Resistor_SMD:R_0603_1608Metric, F.Cu at (-80.7, 106.5)
- added R4: 10k, Resistor_SMD:R_0603_1608Metric, F.Cu at (-42.6, 20.5)
- added R42: 1k, Resistor_SMD:R_0603_1608Metric, F.Cu at (-67.5, 66.1)
- added R5: 10k, Resistor_SMD:R_0603_1608Metric, F.Cu at (-46.2, 32.6)
- added R9: 1k, Resistor_SMD:R_0603_1608Metric, F.Cu at (-38.2, 30.9)
- added U1: DHT22, DHT22:DHT22_THT_P2.54mm_Vertical, F.Cu at (-60.7, -11.3)
- added U39: EMIF06-MSD02N16, Hardware_SD:QFN-16L_L3.5-W1.2-P0.40_EMIF06-MSD02N16, F.Cu at (-105.9, 73.4)
- C40, C50: value 10n -> 100n
- C67: value 10u / 25V -> 4.7u / 25V
- C68: value 10u / 25V -> 10u / 6.3V; footprint Capacitor_SMD:C_0805_2012Metric -> Capacitor_SMD:C_0402_1005Metric
- C69: value 22u / 25V -> 10u / 6.3V; footprint Capacitor_SMD:C_1206_3216Metric -> Capacitor_SMD:C_0402_1005Metric
- C70: value 6p8 / 50V -> 10u / 6.3V; footprint Capacitor_SMD:C_0603_1608Metric -> Capacitor_SMD:C_0402_1005Metric
- J17: value Micro_SD_Card -> 104031-0811
- L61: value 2u2 / MWSA0402S -> 2u2 / ASPI-0530HI; footprint Inductor_SMD:L_Sunlord_MWSA0402S -> Hardware_Power:L_Abracon_ASPI-0530HI
- R62: value 150k / 1% -> 453k / 1%
- R63: footprint Resistor_SMD:R_0603_1608Metric -> Resistor_SMD:R_0402_1005Metric
- R7: footprint Resistor_THT:R_Axial_DIN0204_L3.6mm_D1.6mm_P7.62mm_Horizontal -> Resistor_SMD:R_0603_1608Metric
- TP52: value VREF_SENSOR -> AVREF_SENSOR
- U11: value 74LVC125 -> SN74LVC125APWR
- U4: value Lora_Sx1276 -> STM32F446RET6; footprint myLibrary:SX1276_modulo -> Package_QFP:LQFP-64_10x10mm_P0.5mm
- U9: footprint myLibrary:BH1750FVI-TR_sensor -> Hardware_Sensors:BH1750FVI-TR_WSOF-6
- moved U9 270.2 mm to (-42.2, 31.5)
- moved U8 269.5 mm to (-39.1, 18.6), turned to -90 degrees
- moved J17 212.6 mm to (-106.5, 65.0)
- moved U11 176.5 mm to (-94.8, 70.8)
- moved TP50 144.1 mm to (44.9, 162.7)
- moved TP51 143.3 mm to (52.6, 154.7), turned to 180 degrees
- moved TP52 141.2 mm to (50.1, 158.1)
- moved J32 140.7 mm to (35.9, 158.9)
- moved C50 139.6 mm to (48.9, 154.6), turned to 90 degrees
- moved R50 136.6 mm to (44.1, 158.4), turned to 180 degrees
- moved R51 134.1 mm to (44.1, 156.9)
- moved R52 133.6 mm to (46.5, 155.3)
- moved D50 133.4 mm to (43.9, 160.1)
- moved D51 128.3 mm to (43.2, 153.9), turned to -90 degrees
- moved U12 118.0 mm to (-53.2, 84.4)
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Connections:
- C50 pad 1: WIND_DIR_ADC -> /METEOROLOGIA/WIND_DIR_ADC
- C70 pad 2: /alimentacao/FB_3V3 -> GND
- J17 pad 1: unconnected-(J17-DAT2-Pad1) -> DAT2
- J17 pad 2: CS_LLS -> SD_CS_CARD
- J17 pad 3: DI_LLS -> D_CMD_CARD
- J17 pad 5: SCK_LLS -> SD_CLK_CARD
- J17 pad 7: DO_LLS -> SD_DO_CARD
- J17 pad 8: unconnected-(J17-DAT1-Pad8) -> DAT1
- J30 pad 3: GND -> Net-(J30-Pad3)
- J31 pad 3: GND -> Net-(J31-Pad3)
- J32 pad 2: unconnected-(J32-Pad2) -> /METEOROLOGIA/BIRUTA/WIND_DIR_RAW
- J32 pad 3: GND -> +3V3
- J32 pad 4: /METEOROLOGIA/BIRUTA/WIND_DIR_RAW -> Anem/Pluv_Sig
- J32 pad 5: unconnected-(J32-Pad5) -> GND
- R30 pad 1: +3V3 -> GND
- R40 pad 1: +3V3 -> GND
- R50 pad 1: VREF_SENSOR -> AVREF_SENSOR
- R52 pad 2: WIND_DIR_ADC -> /METEOROLOGIA/WIND_DIR_ADC
- R62 pad 1: Net-(R61-Pad2) -> +3V3
- R7 pad 1: /DHT22/PA8 -> /DHT22/DHT_SIG
- R7 pad 2: +5V -> +3V3
- TP32 pad 1: RAIN_PULSE -> /METEOROLOGIA/RAIN_PULSE
- TP42 pad 1: WIND_SPEED_PULSE -> /METEOROLOGIA/WIND_SPEED_PULSE
- TP51 pad 1: WIND_DIR_ADC -> /METEOROLOGIA/WIND_DIR_ADC
- TP52 pad 1: VREF_SENSOR -> AVREF_SENSOR
- U11 pad 14: +5V -> +3V3
- U11 pad 7: +3V3 -> GND
- U30 pad 4: RAIN_PULSE -> /METEOROLOGIA/RAIN_PULSE
- U4 pad 1: ANT_EXT -> VBAT
- U4 pad 12: PB13 -> GND
- U4 pad 13: PB14 -> AVREF_SENSOR
- U4 pad 14: PB15 -> /METEOROLOGIA/WIND_DIR_ADC
- U4 pad 15: PB12 -> /METEOROLOGIA/RAIN_PULSE
- U4 pad 16: Gnd -> TXD
- U4 pad 2: Gnd -> unconnected-(U4-PC13-Pad2)
- U4 pad 3: +3V3 -> Net-(U4-PC14)
- U4 pad 4: PC4 -> Net-(U4-PC15)
- U4 pad 5: PA11 -> Net-(U4-PH0)
- U4 pad 6: PA12 -> Net-(U4-PH1)
- U4 pad 7: unconnected-(U4-DIO2-Pad7) -> NRST
- U4 pad 9: Gnd -> unconnected-(U4-PC1-Pad9)
- U40 pad 4: WIND_SPEED_PULSE -> /METEOROLOGIA/WIND_SPEED_PULSE
- U8 pad 2: /BMP280/BMP_CSB -> BMP_CSB
- U8 pad 3: /BMP280/BMP_SDA -> /BH1750/I2C1_SDA
- U8 pad 4: /BMP280/BMP_SCK -> /BH1750/I2C1_SCL
- U8 pad 5: /BMP280/BMP_SDO -> BMP_SDO
- U8 pad 8: Net-(U8-VDD) -> +3V3
- U9 pad 2: /BH1750/BH_ADDR -> BH_ADDR
- U9 pad 4: Net-(Q1-S) -> /BH1750/I2C1_SDA
- U9 pad 6: Net-(D1-A) -> /BH1750/I2C1_SCL
Routing:
- net +3V3: track 357.8 -> 3.98 mm
- net Gnd: track 137.8 -> 0.00 mm
- net PB6: track 115.5 -> 0.00 mm
- net PA7: track 85.2 -> 0.00 mm
- net PA6: track 74.0 -> 0.00 mm
- net PC7: track 69.9 -> 0.00 mm
- net PB12: track 69.6 -> 0.00 mm
- net PC4: track 69.2 -> 0.00 mm
- net PA8: track 65.0 -> 0.00 mm
- net PA1: track 64.3 -> 0.00 mm
- net PA5: track 63.7 -> 0.00 mm
- net PB7: track 61.7 -> 0.00 mm
- net PA11: track 57.5 -> 0.00 mm
- net PB13: track 56.7 -> 0.00 mm
- net PA12: track 54.2 -> 0.00 mm
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Other:
- board outline removed

Commit message: refatoracao: lora + Verificacao projeto inteiro
Parts:
- added BT1: Battery_Cell, Battery:BatteryHolder_MYOUNG_BS-07-A1BJ001_CR2032, F.Cu at (-186.9, 50.5)
- added C11: 100n, Capacitor_SMD:C_0603_1608Metric, F.Cu at (-153.2, 39.1)
- added C12: 10u, Capacitor_SMD:C_1206_3216Metric, F.Cu at (-148.3, 45.5)
- added C13: 100n, Capacitor_SMD:C_0603_1608Metric, F.Cu at (-188.2, 69.5)
- added C14: 100n, Capacitor_SMD:C_0603_1608Metric, F.Cu at (-188.2, 72.0)
- added C15: 4.7u, Capacitor_SMD:C_0805_2012Metric, F.Cu at (-166.8, 71.8)
- added C16: 4.7u, Capacitor_SMD:C_0805_2012Metric, F.Cu at (-166.8, 74.8)
- added C17: 1u, Capacitor_SMD:C_0603_1608Metric, F.Cu at (-188.2, 74.5)
- added C18: 10n, Capacitor_SMD:C_0603_1608Metric, F.Cu at (-188.2, 77.0)
- added C19: 15pF, Capacitor_SMD:C_0603_1608Metric, F.Cu at (-184.2, 64.5)
- added C20: 15pF, Capacitor_SMD:C_0603_1608Metric, F.Cu at (-184.2, 67.0)
- added C21: 15pF, Capacitor_SMD:C_0603_1608Metric, F.Cu at (-184.2, 69.5)
- added C22: 15pF, Capacitor_SMD:C_0603_1608Metric, F.Cu at (-184.2, 72.0)
- added C23: 100n, Capacitor_SMD:C_0603_1608Metric, F.Cu at (-184.2, 74.5)
- added C24: 100n, Capacitor_SMD:C_0603_1608Metric, F.Cu at (-184.2, 77.0)
- added C4: 100n, Capacitor_SMD:C_0603_1608Metric, F.Cu at (-188.2, 64.5)
- added C5: 100n, Capacitor_SMD:C_0603_1608Metric, F.Cu at (-188.2, 67.0)
- added D70: PESD5V0R1BSFYL, Hardware_LoRa:SOD-962_L0.6-W0.3-BI, F.Cu at (-150.2, 48.0)
- added FB1: FerriteBead, Inductor_SMD:L_0603_1608Metric, F.Cu at (-180.2, 64.5)
- added FB70: 120R @100MHz / 2A, Inductor_SMD:L_0603_1608Metric, F.Cu at (-153.2, 41.6)
- added J1: Conn_01x02_Pin, Connector_PinHeader_2.54mm:PinHeader_1x02_P2.54mm_Vertical, F.Cu at (-171.3, 72.5)
- added J2: Conn_01x06_Pin, Connector_PinHeader_2.54mm:PinHeader_1x06_P2.54mm_Vertical, F.Cu at (-159.5, 40.1)
- added J3: UART DEBUG 3V3, Connector_PinHeader_2.54mm:PinHeader_1x03_P2.54mm_Vertical, F.Cu at (-175.9, 65.5)
- added J70: U.FL / 50 ohm, Hardware_LoRa:U.FL_Hirose_U.FL-R-SMT-1_Vertical, F.Cu at (-148.6, 40.9)
- added R10: 10k, Resistor_SMD:R_0603_1608Metric, F.Cu at (-180.2, 72.0)
- added R11: 4.7k, Resistor_SMD:R_0603_1608Metric, F.Cu at (-180.2, 74.5)
- added R14: 10k, Resistor_SMD:R_0603_1608Metric, F.Cu at (-153.2, 44.1)
- added R15: 10k, Resistor_SMD:R_0603_1608Metric, F.Cu at (-153.2, 46.6)
- added R6: 4.7k, Resistor_SMD:R_0603_1608Metric, F.Cu at (-180.2, 67.0)
- added R8: 10k, Resistor_SMD:R_0603_1608Metric, F.Cu at (-180.2, 69.5)
- added SW1: SW_Push, Button_Switch_SMD:SW_SPST_TL3342, F.Cu at (-168.8, 66.7)
- added Y2: 32,768 kHz, Crystal:Crystal_SMD_3215-2Pin_3.2x1.5mm, F.Cu at (-162.0, 76.5)
- added Y3: 8 MHz, Crystal:Crystal_SMD_3225-4Pin_3.2x2.5mm, F.Cu at (-161.9, 72.5)
- U12: footprint LoRa1276_C1:COMM-SMD_LORA1276-C1-915MHZ -> Hardware_LoRa:COMM-SMD_LORA1276-C1-915MHZ
Connections:
- D50 pad 1: /METEOROLOGIA/BIRUTA/WIND_DIR_RAW -> GND
- J32 pad 4: Anem/Pluv_Sig -> /METEOROLOGIA/BIRUTA/WIND_DIR_RAW
- J32 pad 5: GND -> unconnected-(J32-Pad5)
- U12 pad 13: +3V3 -> /LORA Module/VCC_LORA
- U12 pad 9: ANT_EXT -> /LORA Module/RF_ANT_915
- U4 pad 26: unconnected-(U4-PB0-Pad26) -> /LORA Module/Lora_DIO2

Commit message: Padronizacao de nomes e numero de componentes
Parts:
- added H901: M3 NPTH, Ø3.2 mm, MountingHole:MountingHole_3.2mm_M3, F.Cu at (-152.5, 120.7)
- added H902: M3 NPTH, Ø3.2 mm, MountingHole:MountingHole_3.2mm_M3, F.Cu at (-152.5, 128.6)
- added H903: M3 NPTH, Ø3.2 mm, MountingHole:MountingHole_3.2mm_M3, F.Cu at (-152.5, 136.6)
- added H904: M3 NPTH, Ø3.2 mm, MountingHole:MountingHole_3.2mm_M3, F.Cu at (-152.5, 144.5)
- BT101: renamed from BT1; value Battery_Cell -> CR2032 holder, vertical; footprint Battery:BatteryHolder_MYOUNG_BS-07-A1BJ001_CR2032 -> Hardware_MCU:BT_Holder_MPD_BS-5_Vertical
- C101: renamed from C4; value 100n -> 100 nF
- C102: renamed from C5; value 100n -> 100 nF
- C103: renamed from C13; value 100n -> 100 nF
- C104: renamed from C14; value 100n -> 100 nF
- C105: renamed from C15; value 4.7u -> 4.7 µF
- C106: renamed from C16; value 4.7u -> 4.7 µF
- C107: renamed from C17; value 1u -> 1 µF
- C108: renamed from C18; value 10n -> 10 nF
- C111: renamed from C21; value 15pF -> 9pF
- C112: renamed from C22; value 15pF -> 9pF
- C113: renamed from C23; value 100n -> 100 nF
- C114: renamed from C24; value 100n -> 100 nF
- C211: renamed from C1; value 100n -> 100 nF
- C212: renamed from C2; value 100n -> 100 nF
- C221: renamed from C6; value 1u -> 1 µF
- C222: renamed from C25; value 100n -> 100 nF
- C231: renamed from C3; value 100n -> 100 nF
- C301: renamed from C30; value 100n -> 100 nF
- C302: renamed from C31; value 100n -> 100 nF
- C401: renamed from C40; value 100n -> 100 nF
- C402: renamed from C41; value 100n -> 100 nF
- C501: renamed from C50; value 100n -> 100 nF
- C601: renamed from C60; value 47u / 35V -> 47 µF, 35 V
- C602: renamed from C61; value 10u / 50V -> 10 µF, 50 V
- C603: renamed from C62; value 10u / 50V -> 10 µF, 50 V
- C606: renamed from C65; value 22u / 25V -> 22 µF, 25 V
- C607: renamed from C66; value 22u / 25V -> 22 µF, 25 V
- C608: renamed from C67; value 4.7u / 25V -> 4.7 µF, 25 V
- C609: renamed from C68; value 10u / 6.3V -> 10 µF, 6.3 V
- C610: renamed from C69; value 10u / 6.3V -> 10 µF, 6.3 V
- C611: renamed from C70; value 10u / 6.3V -> 10 µF, 6.3 V
- C701: renamed from C11; value 100n -> 100 nF
- C702: renamed from C12; value 10u -> 10 µF
- C801: renamed from C7; value 10u / 50V -> 10 µF, 50 V
- C802: renamed from C8; value 100n -> 100 nF
- C803: renamed from C9; value 100n -> 100 nF
- C804: renamed from C10; value 100n -> 100 nF
- F601: renamed from F60; value 1.5A / 32V lento -> 1.5 A, 32 V, slow-blow
- FB101: renamed from FB1; value FerriteBead -> Ferrite bead
- FB701: renamed from FB70; value 120R @100MHz / 2A -> 120 Ω @ 100 MHz, 2 A
- J101: renamed from J1; value Conn_01x02_Pin -> Header, 1x02, P2.54 mm
- J102: renamed from J2; value Conn_01x06_Pin -> Header, 1x06, P2.54 mm
- J103: renamed from J3; value UART DEBUG 3V3 -> Header, 1x03, P2.54 mm
- J301: renamed from J30; value R-RJ11R06P-A800 -> RJ11 6P6C, 90°
- J401: renamed from J31; value R-RJ11R06P-A800 -> RJ11 6P6C, 90°
- J501: renamed from J32; value R-RJ11R06P-A800 -> RJ11 6P6C, 90°
- J601: renamed from J60; value P4 / DC-005-2.0 -> DC jack, 2.0 mm
- J602: renamed from J61; value J_PWR / JST-XH -> JST-XH, 1x02, P2.50 mm
- J701: renamed from J70; value U.FL / 50 ohm -> U.FL, 50 Ω
- J801: renamed from J17; value 104031-0811 -> microSD socket
- JP601: renamed from JP60; value SEL_FONTE -> Solder jumper, 3 pads
- L601: renamed from L60; value 4u7 / MWSA0603S -> 4.7 µH
- L602: renamed from L61; value 2u2 / ASPI-0530HI -> 2.2 µH
- R102: renamed from R8; value 10k -> 10 kΩ
- R103: renamed from R10; value 10k -> 10 kΩ
- R211: renamed from R3; value 10k -> 10 kΩ
- R212: renamed from R4; value 10k -> 10 kΩ
- R221: renamed from R5; value 10k -> 10 kΩ
- R222: renamed from R9; value 1k -> 1 kΩ
- R231: renamed from R7; value 10k -> 10 kΩ
- R301: renamed from R30; value 10k -> 10 kΩ
- R302: renamed from R31; value 4k7 -> 4.7 kΩ
- R303: renamed from R32; value 1k -> 1 kΩ
- R401: renamed from R40; value 10k -> 10 kΩ
- R402: renamed from R41; value 4k7 -> 4.7 kΩ
- R403: renamed from R42; value 1k -> 1 kΩ
- R501: renamed from R50; value 10k -> 10 kΩ
- R502: renamed from R51; value 10k -> 10 kΩ
- R503: renamed from R52; value 1k -> 1 kΩ
- R601: renamed from R60; value 100k / 1% -> 100 kΩ, 1 %
- R602: renamed from R62; value 453k / 1% -> 453 kΩ, 1 %
- R603: renamed from R63; value 100k / 1% -> 100 kΩ, 1 %
- R701: renamed from R14; value 10k -> 10 kΩ
- R702: renamed from R15; value 10k -> 10 kΩ
- R801: renamed from R17; value 10k -> 10 kΩ
- R802: renamed from R18; value 10k -> 10 kΩ
- SW101: renamed from SW1; value SW_Push -> Tactile switch, SPST
- TP301: renamed from TP30; value PLUVIOMETRO_RAW -> SENS_RAIN_RAW
- TP302: renamed from TP31; value PLUVIOMETRO_FILT -> SENS_RAIN_FILTERED
- TP401: renamed from TP40; value ANEMOMETRO_RAW -> SENS_WIND_SPEED_RAW
- TP402: renamed from TP41; value ANEMOMETRO_FILT -> SENS_WIND_SPEED_FILTERED
- TP501: renamed from TP50; value WIND_DIR_RAW -> SENS_WIND_DIR_RAW
- Y101: renamed from Y2; value 32,768 kHz -> 32.768 kHz, CL 7 pF
- Y102: renamed from Y3; value 8 MHz -> 8 MHz, CL 10 pF
- renumbered C19 to C109, C20 to C110, C63 to C604, C64 to C605, D30 to D301, D31 to D302, D40 to D401, D41 to D402, D50 to D501, D51 to D502, D60 to D601, D61 to D602, D70 to D701, Q60 to Q601, R6 to R101, R11 to R104, TP32 to TP303, TP33 to TP304, TP42 to TP403, TP43 to TP404, TP51 to TP502, TP52 to TP503, TP53 to TP504, TP60 to TP601, TP61 to TP602, TP62 to TP603, TP63 to TP604, U4 to U101, U8 to U211, U9 to U221, U1 to U231, U30 to U301, U40 to U401, U60 to U601, U61 to U602, U12 to U701, U11 to U801, U39 to U802
Connections:
- net /BH1750/I2C1_SCL renamed /MCU E DEPURAÇÃO/I2C1_SCL
- net /BH1750/I2C1_SDA renamed /MCU E DEPURAÇÃO/I2C1_SDA
- net /Cartao SD/MCU_MOSI renamed /CARTÃO microSD/SD_SPI_MOSI
- net /Cartao SD/SD_CD renamed /CARTÃO microSD/SD_CD
- net /Cartao SD/SD_CS renamed /CARTÃO microSD/SD_SPI_CS
- net /Cartao SD/SD_MISO renamed /CARTÃO microSD/SD_MISO
- net /Cartao SD/SD_SCK renamed /CARTÃO microSD/SD_SCK
- net /DHT22/DHT_SIG renamed /MCU E DEPURAÇÃO/DHT22_DATA
- net /LORA Module/Lora_DIO0 renamed /MCU E DEPURAÇÃO/LORA_DIO0
- net /LORA Module/Lora_DIO1 renamed /MCU E DEPURAÇÃO/LORA_DIO1
- net /LORA Module/Lora_DIO2 renamed /MCU E DEPURAÇÃO/LORA_DIO2
- net /LORA Module/Lora_MISO renamed /MCU E DEPURAÇÃO/LORA_SPI_MISO
- net /LORA Module/Lora_MOSI renamed /MCU E DEPURAÇÃO/LORA_SPI_MOSI
- net /LORA Module/Lora_NSS renamed /MCU E DEPURAÇÃO/LORA_NSS
- net /LORA Module/Lora_RST renamed /MCU E DEPURAÇÃO/LORA_RST
- net /LORA Module/Lora_SCK renamed /MCU E DEPURAÇÃO/LORA_SPI_SCK
- net /LORA Module/RF_ANT_915 renamed /RÁDIO LoRa/RF_ANT_915
- net /LORA Module/VCC_LORA renamed /RÁDIO LoRa/+3V3_LORA
- net /METEOROLOGIA/ANEMOMETRO/ANEMOMETRO_RAW renamed /INTERFACES METEOROLÓGICAS/ANEMÔMETRO/SENS_WIND_SPEED_RAW
- net /METEOROLOGIA/PLUVIOMETRO/PLUVIOMETRO_RAW renamed /INTERFACES METEOROLÓGICAS/PLUVIÔMETRO/SENS_RAIN_RAW
- net /METEOROLOGIA/RAIN_PULSE renamed /INTERFACES METEOROLÓGICAS/RAIN_PULSE
- net /METEOROLOGIA/WIND_DIR_ADC renamed /INTERFACES METEOROLÓGICAS/WIND_DIR_ADC
- net /METEOROLOGIA/WIND_SPEED_PULSE renamed /INTERFACES METEOROLÓGICAS/WIND_SPEED_PULSE
- net /alimentacao/ENERGIA_POS renamed /ALIMENTAÇÃO/VIN_EXTERNAL
- net /alimentacao/FB_3V3 renamed /ALIMENTAÇÃO/FB_3V3
- net /alimentacao/P4_POS renamed /ALIMENTAÇÃO/VIN_JACK
- net /alimentacao/VIN_MAIN renamed /ALIMENTAÇÃO/VIN_MAIN
- net CS_LLS renamed SD_CS_BUF
- net DAT1 renamed SD_CARD_DAT1
- net DAT2 renamed SD_CARD_DAT2
- net DI_LLS renamed SD_MOSI_BUF
- net DO_LLS renamed SD_MISO_BUF
- net D_CMD_CARD renamed SD_CARD_MOSI
- net SCK_LLS renamed SD_SCK_BUF
- net SD_CLK_CARD renamed SD_CARD_SCK
- net SD_CS_CARD renamed SD_CARD_CS
- net SD_DO_CARD renamed SD_CARD_MISO
- D501 pad 1: GND -> Net-(D501-K)
- J501 pad 2: /METEOROLOGIA/BIRUTA/WIND_DIR_RAW -> Net-(D501-K)
- J501 pad 4: /METEOROLOGIA/BIRUTA/WIND_DIR_RAW -> SENS_SPARE
- J501 pad 5: unconnected-(J32-Pad5) -> GND
- R501 pad 2: /METEOROLOGIA/BIRUTA/WIND_DIR_RAW -> Net-(D501-K)
- R502 pad 1: /METEOROLOGIA/BIRUTA/WIND_DIR_RAW -> Net-(D501-K)
- TP501 pad 1: /METEOROLOGIA/BIRUTA/WIND_DIR_RAW -> Net-(D501-K)

Commit message: Ajuste de componentes por folha
Parts:
- moved J701 302.2 mm to (152.4, 66.9), turned to 90 degrees
- moved D701 300.6 mm to (149.6, 69.3)
- moved C701 300.1 mm to (145.4, 68.8)
- moved FB701 294.6 mm to (140.4, 66.3)
- moved C702 294.6 mm to (145.5, 66.4)
- moved C101 289.5 mm to (101.1, 75.4), turned to -90 degrees
- moved C102 285.3 mm to (96.4, 87.0), turned to 180 degrees
- moved R701 283.8 mm to (128.9, 75.1), turned to -90 degrees
- moved R702 280.9 mm to (126.3, 75.1), turned to -90 degrees
- moved C103 278.2 mm to (89.5, 86.6), turned to 180 degrees
- moved C104 277.9 mm to (89.7, 70.9)
- moved R101 273.9 mm to (93.7, 70.4), turned to 180 degrees
- moved J101 273.4 mm to (97.0, 20.0)
- moved R104 273.4 mm to (93.1, 68.1), turned to 180 degrees
- moved C108 273.3 mm to (85.1, 80.5), turned to 90 degrees
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
Commit message: Roteamento 1
Parts:
- J801: value microSD socket -> microSD socket, TF-15x15; footprint Connector_Card:microSD_HC_Molex_104031-0811 -> Hardware_SD_Interface:microSD_SOFNG_TF-15x15
- moved H904 147.8 mm to (43.7, 29.7)
- moved H903 125.4 mm to (147.5, 38.4)
- moved J102 111.0 mm to (93.6, 50.5)
- moved BT101 75.8 mm to (73.6, 96.6), turned to -90 degrees
- moved H902 73.5 mm to (39.9, 113.9)
- moved J103 71.5 mm to (85.5, 85.3)
- moved C402 63.4 mm to (60.9, 48.0)
- moved J401 63.4 mm to (48.3, 45.0)
- moved R401 63.4 mm to (54.5, 46.5)
- moved R402 63.4 mm to (53.7, 43.8)
- moved TP401 63.4 mm to (54.1, 50.8)
- moved TP403 63.4 mm to (64.5, 48.3)
- moved C401 63.4 mm to (55.6, 41.9)
- moved D401 63.4 mm to (53.9, 48.4)
- moved D402 63.4 mm to (58.8, 41.4)
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Connections:
- J501 pad 4: SENS_SPARE -> unconnected-(J501-Pad4)
Routing:
- net +3V3: track 3.98 -> 0.00 mm
- net BMP_CSB: track 1.87 -> 0.00 mm
Other:
- board outline added: 124.6 x 97.9 mm

Commit message: Roteamento 1.1
Parts:
- moved H904 31.4 mm to (71.8, 43.8)
- moved H902 24.6 mm to (63.5, 107.1)
- moved H903 10.6 mm to (138.4, 43.9)
- moved H901 8.68 mm to (138.6, 107.2)
- moved C701 2.86 mm to (135.2, 76.1)
- moved FB701 2.86 mm to (130.2, 73.6)
- moved D701 2.86 mm to (139.4, 76.6)
- moved R702 2.86 mm to (142.6, 83.2)
- moved U701 2.86 mm to (133.0, 86.5)
- moved J701 2.86 mm to (142.2, 74.2)
- moved C702 2.86 mm to (135.3, 73.7)
- moved R701 2.86 mm to (142.6, 88.0)
- moved TP503 1.41 mm to (56.6, 107.7)
- moved TP501 0.20 mm to (53.7, 107.7)
Other:
- board size 124.6 x 97.9 mm -> 124.6 x 76.8 mm
Changed lines of the file:
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@@
 	(footprint "Capacitor_SMD:C_0603_1608Metric"
 		(layer "F.Cu")
-		(at 136.275 78.75)
+		(at 135.2 76.1)
 		(descr "Capacitor SMD 0603 (1608 Metric), square (rectangular) end terminal, IPC-7351 nominal, (Body size source: IPC-SM-782 page 76, https://www.pcb-3d.com/wordpress/wp-content/uploads/ipc-sm-782a_amendment_1_and_2.pdf), generated with kicad-footprint-generator")
 		(tags "capacitor")
@@
 	(footprint "Resistor_SMD:R_0603_1608Metric"
 		(layer "F.Cu")
-		(at 143.7 85.9 -90)
+		(at 142.625 83.25 -90)
 		(descr "Resistor SMD 0603 (1608 Metric), square (rectangular) end terminal, IPC-7351 nominal, (Body size source: IPC-SM-782 page 72, https://www.pcb-3d.com/wordpress/wp-content/uploads/ipc-sm-782a_amendment_1_and_2.pdf), generated with kicad-footprint-generator")
 		(tags "resistor")
@@
 	(footprint "Resistor_SMD:R_0603_1608Metric"
 		(layer "F.Cu")
-		(at 143.7 90.6 -90)
+		(at 142.625 87.95 -90)
 		(descr "Resistor SMD 0603 (1608 Metric), square (rectangular) end terminal, IPC-7351 nominal, (Body size source: IPC-SM-782 page 72, https://www.pcb-3d.com/wordpress/wp-content/uploads/ipc-sm-782a_amendment_1_and_2.pdf), generated with kicad-footprint-generator")
 		(tags "resistor")
@@
 	(footprint "TestPoint:TestPoint_Pad_D1.5mm"
 		(layer "F.Cu")
-		(at 58 107.9 -90)
+		(at 56.6 107.7 -90)
 		(descr "SMD pad as test Point, diameter 1.5mm")
 		(tags "test point SMD pad")
 		(property "Reference" "TP503"
-			(at 2.1 -2 180)
+			(at 0.5 -2.3 270)
 			(layer "F.SilkS")
 			(effects
@@
 	(footprint "Hardware_LoRa:COMM-SMD_LORA1276-C1-915MHZ"
 		(layer "F.Cu")
-		(at 134.1 89.2 90)
+		(at 133.025 86.55 90)
 		(property "Reference" "U701"
 			(at 0 -11 90)
@@
 	(footprint "TestPoint:TestPoint_Pad_D1.5mm"
 		(layer "F.Cu")
-		(at 53.7 107.9 180)
+		(at 53.7 107.7 180)
 		(descr "SMD pad as test Point, diameter 1.5mm")
 		(tags "test point SMD pad")
@@
 	(footprint "MountingHole:MountingHole_3.2mm_M3"
 		(layer "F.Cu")
-		(at 43.7 29.7)
+		(at 71.8 43.8)
 		(descr "Mounting Hole 3.2mm, M3, no annular, generated by kicad-footprint-generator mountinghole.py")
 		(tags "mountinghole M3")
@@
 	(footprint "Hardware_LoRa:U.FL_Hirose_U.FL-R-SMT-1_Vertical"
 		(layer "F.Cu")
-		(at 143.275 76.85 90)
+		(at 142.2 74.2 90)
 		(descr "Hirose U.FL Coaxial https://www.hirose.com/product/en/products/U.FL/U.FL-R-SMT-1%2810%29/")
 		(tags "Hirose U.FL Coaxial")
 		(property "Reference" "J701"
-			(at 3.1 -0.1 180)
+			(at 3 -0.1 180)
 			(layer "F.SilkS")
 			(effects
@@
 			(polygon
 				(pts
-					(xy 142.325 75.275) (xy 142.325 77.365) (xy 144.225 77.365) (xy 144.225 75.275)
+					(xy 141.25 72.625) (xy 141.25 74.715) (xy 143.15 74.715) (xy 143.15 72.625)
 				)
 			)
@@
 	(footprint "MountingHole:MountingHole_3.2mm_M3"
 		(layer "F.Cu")
-		(at 147.5 38.4)
+		(at 138.4 43.9)
 		(descr "Mounting Hole 3.2mm, M3, no annular, generated by kicad-footprint-generator mountinghole.py")
 		(tags "mountinghole M3")
@@
 		(model "${KIPRJMOD}/../../libraries/Hardware_MCU/Hardware_MCU.3dshapes/BT_Holder_MPD_BS-5_Vertical.step"
 			(offset
-				(xyz 0 0 0)
+				(xyz 0 -2 0)
 			)
 			(scale
@@
 			)
 			(rotate
-				(xyz 0 0 0)
+				(xyz -90 -0 -90)
 			)
 		)
@@
 	(footprint "Hardware_LoRa:SOD-962_L0.6-W0.3-BI"
 		(layer "F.Cu")
-		(at 140.475 79.25)
+		(at 139.4 76.6)
 		(descr "Nexperia DSN0603-2 SOD962-2; datasheet 2023-09-06 fig14; reflow stencil 0.1mm")
 		(property "Reference" "D701"
@@
 	(footprint "Inductor_SMD:L_0603_1608Metric"
 		(layer "F.Cu")
-		(at 131.275 76.25)
+		(at 130.2 73.6)
 		(descr "Inductor SMD 0603 (1608 Metric), square (rectangular) end terminal, IPC-7351 nominal, (Body size source: http://www.tortai-tech.com/upload/download/2011102023233369053.pdf), generated with kicad-footprint-generator")
 		(tags "inductor")
@@
 	(footprint "MountingHole:MountingHole_3.2mm_M3"
 		(layer "F.Cu")
-		(at 146.2 111.4)
+		(at 138.6 107.2)
 		(descr "Mounting Hole 3.2mm, M3, no annular, generated by kicad-footprint-generator mountinghole.py")
 		(tags "mountinghole M3")
@@
 	(footprint "Capacitor_SMD:C_1206_3216Metric"
 		(layer "F.Cu")
-		(at 136.375 76.35)
+		(at 135.3 73.7)
 		(descr "Capacitor SMD 1206 (3216 Metric), square (rectangular) end terminal, IPC-7351 nominal, (Body size source: IPC-SM-782 page 76, https://www.pcb-3d.com/wordpress/wp-content/uploads/ipc-sm-782a_amendment_1_and_2.pdf), generated with kicad-footprint-generator")
 		(tags "capacitor")
@@
 	(footprint "MountingHole:MountingHole_3.2mm_M3"
 		(layer "F.Cu")
-		(at 39.9 113.9)
+		(at 63.5 107.1)
 		(descr "Mounting Hole 3.2mm, M3, no annular, generated by kicad-footprint-generator mountinghole.py")
 		(tags "mountinghole M3")
@@
 	)
 	(gr_rect
-		(start 30.6 22.3)
-		(end 155.2 120.2)
+		(start 30.6 35)
+		(end 155.2 111.8)
 		(stroke
 			(width 0.05)
