File: hardware/kicad/estacao-meteorologica/estacao-meteorologica.kicad_pcb (KiCad board)
At the start: 2 copper layers, 96.9 x 56.3 mm, 125 parts, among them J101 Header, 1x02, P2.54 mm, J102 Header, 1x06, P2.54 mm, J103 Header, 1x03, P2.54 mm, J221 JST-XH, 1x04, P2.50 mm, J301 RJ11 6P6C, 90°, J501 RJ11 6P6C, 90°, J601 DC jack, 2.0 mm, J602 JST-XH, 1x02, P2.50 mm, J701 U.FL, 50 Ω, J801 microSD socket, TF-15x15, Q601 DMP6023LE-13, SW101 Tactile switch, SPST, U101 STM32F446RET6, U211 BMP280, U231 DHT22, U301 SN74LVC1G17DBVR, U401 SN74LVC1G17DBVR, U601 AP63203WU-7, U701 LORA1276-C1-915MHZ, U801 SN74LVC125APWR, U802 EMIF06-MSD02N16, Y101 32.768 kHz, CL 7 pF, Y102 8 MHz, CL 10 pF

Commit message: chore(hardware): inicia novo roteamento da PCB V2
Parts:
- removed BT101: CR1225 holder, horizontal, Hardware_Battery:BT_Holder_MYOUNG_BS-12-B4AK025-R
- removed C101, C102, C103, C104, C113, C114, C211, C212, C231, C301, C302, C401, C402, C501, C701, C802, C803, C804: 100 nF, Capacitor_SMD:C_0603_1608Metric
- removed C105, C106: 4.7 µF, Capacitor_SMD:C_0805_2012Metric
- removed C107: 1 µF, Capacitor_SMD:C_0603_1608Metric
- removed C108: 10 nF, Capacitor_SMD:C_0603_1608Metric
- removed C109, C110: 15pF, Capacitor_SMD:C_0603_1608Metric
- removed C111, C112: 9pF, Capacitor_SMD:C_0603_1608Metric
- removed C601: 47 µF, 35 V, Capacitor_SMD:CP_Elec_6.3x5.8
- removed C602, C603, C801: 10 µF, 50 V, Capacitor_SMD:C_1206_3216Metric
- removed C604, C605: 100n / 50V, Capacitor_SMD:C_0603_1608Metric
- removed C606, C607: 22 µF, 25 V, Capacitor_SMD:C_1206_3216Metric
- removed C702: 10 µF, Capacitor_SMD:C_1206_3216Metric
- removed D221, D222, D701: PESD5V0R1BSFYL, Hardware_LoRa:SOD-962_L0.6-W0.3-BI
- removed D301, D401, D501: PESD5V0S1UL, Diode_SMD:D_SOD-882
- removed D302, D402, D502: BAS70-04, Package_TO_SOT_SMD:SOT-23
- removed D601: SMBJ16CA, Diode_SMD:D_SMB
- removed D602: BZT52C10 / 10V, Diode_SMD:D_SOD-123
- removed F601: 1.5 A, 32 V, slow-blow, Fuse:Fuse_1206_3216Metric
- removed FB101: Ferrite bead, Inductor_SMD:L_0603_1608Metric
- removed FB701: 120 Ω @ 100 MHz, 2 A, Inductor_SMD:L_0603_1608Metric
- removed H901, H902, H903, H904: M3 NPTH, Ø3.2 mm, MountingHole:MountingHole_3.2mm_M3
- removed J101: Header, 1x02, P2.54 mm, Connector_PinHeader_2.54mm:PinHeader_1x02_P2.54mm_Vertical
- removed J102: Header, 1x06, P2.54 mm, Connector_PinHeader_2.54mm:PinHeader_1x06_P2.54mm_Vertical
- removed J103: Header, 1x03, P2.54 mm, Connector_PinHeader_2.54mm:PinHeader_1x03_P2.54mm_Vertical
- removed J221: JST-XH, 1x04, P2.50 mm, Connector_JST:JST_XH_B4B-XH-A_1x04_P2.50mm_Vertical
- removed J301, J501: RJ11 6P6C, 90°, Sensores_Meteo:RJ11-TH_PCB-6P6C-90
- removed J601: DC jack, 2.0 mm, Hardware_Power:DC-IN-TH_DC-005-2.0_C22459640
- removed J602: JST-XH, 1x02, P2.50 mm, Connector_JST:JST_XH_B2B-XH-A_1x02_P2.50mm_Vertical
- removed J701: U.FL, 50 Ω, Hardware_LoRa:U.FL_Hirose_U.FL-R-SMT-1_Vertical
- removed J801: microSD socket, TF-15x15, Hardware_SD_Interface:microSD_SOFNG_TF-15x15_C111196
- removed JP601: Solder jumper, 3 pads, Jumper:SolderJumper-3_P2.0mm_Open_TrianglePad1.0x1.5mm_NumberLabels
- removed L601: 3.9 µH, Inductor_SMD:L_APV_ANR5040
- removed Q601: DMP6023LE-13, Hardware_Power:SOT-223-4_L6.5-W3.5-P2.30-LS7.0-BR
- removed R1, R303, R503: 1 kΩ, Resistor_SMD:R_0603_1608Metric
- removed R101, R104, R105, R106: 4.7k, Resistor_SMD:R_0603_1608Metric
- removed R102, R103, R211, R212, R231, R301, R401, R501, R502, R701, R702, R801, R802: 10 kΩ, Resistor_SMD:R_0603_1608Metric
- removed R302, R402: 4.7 kΩ, Resistor_SMD:R_0603_1608Metric
- removed R601: 100 kΩ, 1 %, Resistor_SMD:R_0603_1608Metric
- removed SW101: Tactile switch, SPST, Button_Switch_SMD:SW_SPST_TL3342
- removed TP211: I2C1_SCL, TestPoint:TestPoint_Pad_D1.0mm
- removed TP212: I2C1_SDA, TestPoint:TestPoint_Pad_D1.0mm
- removed TP213, TP223, TP232, TP304, TP404, TP504, TP604: GND, TestPoint:TestPoint_Pad_D1.0mm
- removed TP221: BH_I2C3_SCL, TestPoint:TestPoint_Pad_D1.0mm
- removed TP222: BH_I2C3_SDA, TestPoint:TestPoint_Pad_D1.0mm
- removed TP231: DHT22_DATA, TestPoint:TestPoint_Pad_D1.0mm
- removed TP301: SENS_RAIN_RAW, TestPoint:TestPoint_Pad_D1.0mm
- removed TP302: SENS_RAIN_FILTERED, TestPoint:TestPoint_Pad_D1.0mm
- removed TP303: RAIN_PULSE, TestPoint:TestPoint_Pad_D1.0mm
- removed TP401: SENS_WIND_SPEED_RAW, TestPoint:TestPoint_Pad_D1.0mm
- removed TP402: SENS_WIND_SPEED_FILTERED, TestPoint:TestPoint_Pad_D1.0mm
- removed TP403: WIND_SPEED_PULSE, TestPoint:TestPoint_Pad_D1.0mm
- removed TP501: SENS_WIND_DIR_RAW, TestPoint:TestPoint_Pad_D1.0mm
- removed TP502: WIND_DIR_ADC, TestPoint:TestPoint_Pad_D1.0mm
- removed TP503: AVREF_SENSOR, TestPoint:TestPoint_Pad_D1.0mm
- removed TP601: VIN_MAIN, TestPoint:TestPoint_Pad_D1.0mm
- removed TP603: +3V3, TestPoint:TestPoint_Pad_D1.0mm
- removed U101: STM32F446RET6, Package_QFP:LQFP-64_10x10mm_P0.5mm
- removed U211: BMP280, Package_LGA:Bosch_LGA-8_2x2.5mm_P0.65mm_ClockwisePinNumbering
- removed U231: DHT22, DHT22:DHT22_THT_P2.54mm_Vertical
- removed U301, U401: SN74LVC1G17DBVR, Package_TO_SOT_SMD:SOT-23-5
- removed U601: AP63203WU-7, Package_TO_SOT_SMD:TSOT-23-6
- removed U701: LORA1276-C1-915MHZ, Hardware_LoRa:COMM-SMD_LORA1276-C1-915MHZ
- removed U801: SN74LVC125APWR, Package_SO:TSSOP-14_4.4x5mm_P0.65mm
- removed U802: EMIF06-MSD02N16, Hardware_SD:QFN-16L_L3.5-W1.2-P0.40_EMIF06-MSD02N16
- removed Y101: 32.768 kHz, CL 7 pF, Crystal:Crystal_SMD_3215-2Pin_3.2x1.5mm
- removed Y102: 8 MHz, CL 10 pF, Crystal:Crystal_SMD_3225-4Pin_3.2x2.5mm
Routing:
- net +3V3: track 404.9 -> 0.00 mm, vias 5 -> 0
- net GND: track 121.3 -> 0.00 mm, vias 95 -> 0
- net /INTERFACES METEOROLÓGICAS/WIND_SPEED_PULSE: track 59.1 -> 0.00 mm, vias 4 -> 0
- net NRST: track 56.1 -> 0.00 mm, vias 3 -> 0
- net AVREF_SENSOR: track 53.3 -> 0.00 mm, vias 2 -> 0
- net /INTERFACES METEOROLÓGICAS/WIND_DIR_ADC: track 48.7 -> 0.00 mm, vias 2 -> 0
- net /MCU E DEPURAÇÃO/LORA_RST: track 42.4 -> 0.00 mm, vias 2 -> 0
- net /MCU E DEPURAÇÃO/DHT22_DATA: track 39.0 -> 0.00 mm, vias 2 -> 0
- net /BH1750_INTERFACE/BH_I2C3_SDA: track 37.9 -> 0.00 mm, vias 4 -> 0
- net /INTERFACES METEOROLÓGICAS/RAIN_PULSE: track 36.3 -> 0.00 mm, vias 2 -> 0
- net /BH1750_INTERFACE/BH_I2C3_SCL: track 35.3 -> 0.00 mm, vias 4 -> 0
- net /MCU E DEPURAÇÃO/LORA_NSS: track 31.9 -> 0.00 mm, vias 2 -> 0
- net /RÁDIO LoRa/+3V3_LORA: track 25.5 -> 0.00 mm
- net /ALIMENTAÇÃO/VIN_MAIN: track 24.9 -> 0.00 mm
- net SWDIO: track 23.9 -> 0.00 mm, vias 1 -> 0
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- removed copper zone on F.Cu, net +3V3
- removed copper zone on F.Cu, net /ALIMENTAÇÃO/VIN_MAIN
- removed copper zone on F.Cu, net /ALIMENTAÇÃO/V_SW
- removed copper zone on B.Cu, net GND
- removed copper zone on F.Cu, net GND
Other:
- board outline removed
